File: hardware/cards/card_storage.kicad_sch (KiCad schematic)
At the start: 22 parts, among them J1 Conn_02x20_Odd_Even, J2 Conn_02x25_Odd_Even, U1 74HCT04, U10 74HCT573, U11 74HCT138, U2 74HCT08, U3 74HCT08, U4 74HCT32, U5 74HCT125, U6 74HCT138, U7 74HCT138, U8 74HCT245, U9 74HCT573

Commit message: JLCPCB sourcing pass: verify pinouts, LCSC part numbers, SMD build
Custom-symbol verification (open-questions Q5 resolved):
- MAX3241 symbol was wrong on nearly every pin and used MAX3243-style
  control names; regenerated to the real SSOP-28 pinout (SHDN#/EN#/
  R1OUTB/R2OUTB) and com_port rewired -- EN# must be GROUNDED (the old
  ~FORCEON-high would have disabled the receivers on real silicon)
- DS12C887 symbol wrong on 4 pins (DS=17, RESET#=18, IRQ#=19, SQW=23)

Sourcing (every part checked against the JLC DB; ~45 line items):
- New tools/parts.py maps (lib_id, value) -> LCSC; build.py applies it as
  an 'LCSC Part Num' property on every component (384 across the project)
- Sheets stay generic; stock-forced substitutions bound in the map:
  '374->'574 (parallel rewired), '163->'161, '157->HC157 (+HCT-buffered
  3.3V selects, I0/I1 swapped), '02->HC02, TCM809->MCP809, 2N3904->MMBT3904
- bus_mcu address counters moved to the 3.3V domain (HC161 on 3V3_BUS,
  loaded from MCU-side MD0-7; HCT244s read the 3.3V outputs at TTL Vih)
- 14.318 XOs are 3.3V-only parts: powered from 3V3, squared up via spare
  HCT gates (cpu_core U13, card_isatest U19)
- COM baud reference is now a 1.8432MHz crystal on the 16C550's XIN/XOUT
  (3.3V-only oscillators vs a 5V-only soft card)
- Supervisor QSPI header replaced with a real W25Q128JVSIQ
- Socket policy (fab installs sockets): V20 DIP-40, SRAM DIP-32 (no 5V
  512Kx8 SRAM at JLC at all), DS12C887 DIP-24, female headers for modules

Docs: CLAUDE.md fabrication-constraints section (SMD, 100x100mm, generic-
symbols rule, voltage-domain rule); README + hardware/README fab notes;
notes/jlcpcb-sourcing.md (decisions, thin-stock flags, not-at-JLC list);
stale questions-sidecar.md collapsed to its supersession record.

Rebuilt motherboard + cards: structural ERC 0, byte-identical rebuilds.

Co-Authored-By: Claude Fable 5 <noreply@anthropic.com>
Parts:
- C1, C2, C3, C4: LCSC Part Num (none) -> C14663
- J1, J_IN, J_OUT: LCSC Part Num (none) -> C2333
- J2: LCSC Part Num (none) -> C2962036
- R1, R2, R3: LCSC Part Num (none) -> C25804
- U1: LCSC Part Num (none) -> C672096
- U10, U9: LCSC Part Num (none) -> C5209384
- U11, U6, U7: LCSC Part Num (none) -> C5965
- U2, U3: LCSC Part Num (none) -> C5959
- U4: LCSC Part Num (none) -> C5985
- U5: LCSC Part Num (none) -> C5962
- U8: LCSC Part Num (none) -> C5979
Changed lines of the file:
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@@
+			)
+		)
+		(property "LCSC Part Num" "C2333"
+			(at 444.5 152.4 0)
+			(effects
+				(font
+					(size 1.27 1.27)
+				)
+				(hide yes)
 			)
 		)
@@
 			)
 		)
+		(property "LCSC Part Num" "C2333"
+			(at 508 152.4 0)
+			(effects
+				(font
+					(size 1.27 1.27)
+				)
+				(hide yes)
+			)
+		)
 		(pin "1"
 		)
@@
 			)
 		)
+		(property "LCSC Part Num" "C672096"
+			(at 38.1 76.2 0)
+			(effects
+				(font
+					(size 1.27 1.27)
+				)
+				(hide yes)
+			)
+		)
 		(pin "1"
 		)
@@
 			)
 		)
+		(property "LCSC Part Num" "C5959"
+			(at 38.1 142.24 0)
+			(effects
+				(font
+					(size 1.27 1.27)
+				)
+				(hide yes)
+			)
+		)
 		(pin "1"
 		)
@@
 			)
 		)
+		(property "LCSC Part Num" "C5959"
+			(at 38.1 205.74 0)
+			(effects
+				(font
+					(size 1.27 1.27)
+				)
+				(hide yes)
+			)
+		)
 		(pin "1"
 		)
@@
 			)
 		)
+		(property "LCSC Part Num" "C5985"
+			(at 114.3 210.82 0)
+			(effects
+				(font
+					(size 1.27 1.27)
+				)
+				(hide yes)
+			)
+		)
 		(pin "1"
 		)
@@
 			)
 		)
+		(property "LCSC Part Num" "C5962"
+			(at 38.1 256.54 0)
+			(effects
+				(font
+					(size 1.27 1.27)
+				)
+				(hide yes)
+			)
+		)
 		(pin "2"
 		)
@@
 			)
 		)
+		(property "LCSC Part Num" "C5965"
+			(at 114.3 63.5 0)
+			(effects
+				(font
+					(size 1.27 1.27)
+				)
+				(hide yes)
+			)
+		)
 		(pin "1"
 		)
@@
 			)
 		)
+		(property "LCSC Part Num" "C5965"
+			(at 114.3 142.24 0)
+			(effects
+				(font
+					(size 1.27 1.27)
+				)
+				(hide yes)
+			)
+		)
 		(pin "1"
 		)
@@
 			)
 		)
+		(property "LCSC Part Num" "C5965"
+			(at 152.4 63.5 0)
+			(effects
+				(font
+					(size 1.27 1.27)
+				)
+				(hide yes)
+			)
+		)
 		(pin "1"
 		)
@@
 			)
 		)
+		(property "LCSC Part Num" "C5979"
+			(at 190.5 63.5 0)
+			(effects
+				(font
+					(size 1.27 1.27)
+				)
+				(hide yes)
+			)
+		)
 		(pin "1"
 		)
@@
 			)
 		)
+		(property "LCSC Part Num" "C5209384"
+			(at 190.5 142.24 0)
+			(effects
+				(font
+					(size 1.27 1.27)
+				)
+				(hide yes)
+			)
+		)
 		(pin "2"
 		)
@@
 			)
 		)
+		(property "LCSC Part Num" "C5209384"
+			(at 190.5 215.9 0)
+			(effects
+				(font
+					(size 1.27 1.27)
+				)
+				(hide yes)
+			)
+		)
 		(pin "2"
 		)
@@
 			)
 		)
+		(property "LCSC Part Num" "C2333"
+			(at 292.1 127 0)
+			(effects
+				(font
+					(size 1.27 1.27)
+				)
+				(hide yes)
+			)
+		)
 		(pin "1"
 		)
@@
 			)
 		)
+		(property "LCSC Part Num" "C2962036"
+			(at 368.3 127 0)
+			(effects
+				(font
+					(size 1.27 1.27)
+				)
+				(hide yes)
+			)
+		)
 		(pin "1"
 		)
@@
 			)
 		)
+		(property "LCSC Part Num" "C25804"
+			(at 228.6 25.4 0)
+			(effects
+				(font
+					(size 1.27 1.27)
+				)
+				(hide yes)
+			)
+		)
 		(pin "1"
 		)
@@
 			)
 		)
+		(property "LCSC Part Num" "C25804"
+			(at 243.84 25.4 0)
+			(effects
+				(font
+					(size 1.27 1.27)
+				)
+				(hide yes)
+			)
+		)
 		(pin "1"
 		)
@@
 			)
 		)
+		(property "LCSC Part Num" "C25804"
+			(at 259.08 25.4 0)
+			(effects
+				(font
+					(size 1.27 1.27)
+				)
+				(hide yes)
+			)
+		)
 		(pin "1"
 		)
@@
 			)
 		)
+		(property "LCSC Part Num" "C14663"
+			(at 49.53 276.86 0)
+			(effects
+				(font
+					(size 1.27 1.27)
+				)
+				(hide yes)
+			)
+		)
 		(pin "1"
 		)
@@
 			)
 		)
+		(property "LCSC Part Num" "C14663"
+			(at 100.33 276.86 0)
+			(effects
+				(font
+					(size 1.27 1.27)
+				)
+				(hide yes)
+			)
+		)
 		(pin "1"
 		)
@@
 			)
 		)
+		(property "LCSC Part Num" "C14663"
+			(at 149.86 276.86 0)
+			(effects
+				(font
+					(size 1.27 1.27)
+				)
+				(hide yes)
+			)
+		)
 		(pin "1"
 		)
@@
 			(at 199.39 276.86 0)
 			(effects
+				(font
+					(size 1.27 1.27)
+				)
+				(hide yes)
+			)
+		)
+		(property "LCSC Part Num" "C14663"
+			(at 199.39 276.86 0)
+			(effects
