File: hardware/cards/card_com.kicad_sch (KiCad schematic)
At the start: 22 parts, among them J1 DE9_Pins, J2 Conn_01x03, J3 Conn_01x04, U1 16550, U2 MAX3241, U3 74HCT04, U4 74HCT08, U5 74HCT08, U6 74HCT125, Y1 1.8432MHz

Commit message: COM cards: socket the 16550s (SMD PLCC-44)
The fab reflows a Nextron SMD PLCC-44 socket (LCSC C2828044, ~$0.39) in
the normal SMD pass; the UART installs by hand. One footprint accepts the
active-production TL16C550CFNR (Mouser ~320 pcs), NOS tubes, and period
NS16550AFN pulls (same industry PLCC pinout), and a suspect UART is
diagnosed by swap. MaxLinear's PLCC ST16C550CJ44-F is EOL; TI's reel CFNR
is the active leg. Schematic unchanged (parts.py retarget + comments);
DB9s stay THT (C141880) -- SMD D-subs cost 5-9x and shear pads under
cable torque. Sourcing notes + CLAUDE.md socket policy updated.

Co-Authored-By: Claude Fable 5 <noreply@anthropic.com>
Parts:
- U1: LCSC Part Num C544406 -> C2828044
Changed lines of the file:
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@@
 			)
 		)
-		(property "LCSC Part Num" "C544406"
+		(property "LCSC Part Num" "C2828044"
 			(at 127 101.6 0)
 			(effects

Commit message: Design review 2026-07-11: rail protection, decoupling, wiring fixes
Protection:
- Sidecar +5V now feeds through a 2A polyfuse into +5V_ISA with an
  SMBJ5.0A clamp + 22uF bulk (a faulted ISA card trips its own fuse
  instead of dropping the board; back-fed voltage is clamped).
- USB-C VBUS enters through a 3A polyfuse with an SMBJ5.0A on +5V
  (backstop for the CFG1 9-20V failure mode). CH224K gains a 1uF VDD
  cap; its PG routes to Supervisor GPIO16 as PD_PG. Buck output
  doubled to 2x22uF, 10uF at VIN, extra rail bulk.
- Supervisor USB-A host port: 27R series termination (RP2040
  requirement), USBLC6-2SC6 ESD array, 100uF VBUS bulk.
- Video: HDMI +5V fused (500mA), HPD sensed on GPIO41, 100R series on
  VGA sync. TMDS ESD array deferred to layout (no symbol).
- card_isatest: V5RAW bulk, Q1 gate soft-start cap, TVS on DUT rail.

Wiring fixes:
- SPKR had no driver anywhere (netlist: 1 node). Bus MCU GPIO22
  reassigned from the diagnostics-only bus-CLK sense to SPKR; bus_mcu
  drops CLK from its interface. Doc 5.2 updated.
- bus_mcu C8 decoupled +3V3, a rail that sheet never uses -> 3V3_BUS.
- Storage IRQ5 was push-pull (permanently driven when idle) -> 2N7002
  + gated '125 tri-state, same convention as the LPT IRQ7 stage.
- MAX3241 pump caps resized to the 5V datasheet values (47nF/330nF).
- LPT DB25 status inputs get 4.7k pull-ups (floated with no printer).
- Audio line-out gets a 100R series isolator before the jack.

Best practices:
- Decoupling to ~1x100nF per IC on every sheet + bulk per board
  (cpu_core 7->16 incl. the naked 3.3V oscillator, storage 4->11,
  parallel 6->13, rtc/com/video/bus_mcu/card_isatest similar).
- All floating spare CMOS inputs tied ('00/'74/'157/'02/'04/'125
  sections across cpu_core, bus_mcu, rtc, storage, card_isatest).

Sourcing: new parts mapped in parts.py with JLC-verified LCSC numbers;
Power_Protection lib registered in the tools; TPS563200 stock alert
(4 pcs left at JLC) flagged in parts.py + jlcpcb-sourcing.md. All
decisi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
Parts:
- added C10, C11, C12, C9: 100nF, symbol Device:C
- added C13: 10uF, symbol Device:C
- C3: value 100nF -> 47nF; LCSC Part Num C14663 -> C1622
- C4, C5, C6: value 100nF -> 330nF; LCSC Part Num C14663 -> C1615
Connections:
- net +5V: now also C10.1, C11.1, C12.1, C13.1, C9.1
- net GND: now also C10.2, C11.2, C12.2, C13.2, C9.2
