File: hardware/cards/card_lpt.kicad_sch (KiCad schematic)
At the start: 22 parts, among them J1 DB25_Pins, U1 74HCT574, U10 74HCT32, U11 74HCT32, U12 74HCT00, U13 74HCT125, U2 74HCT574, U3 74HCT244, U4 74HCT245, U5 74HCT244, U6 74HCT138, U7 74HCT08, U8 74HCT08, U9 74HCT04

Commit message: Design review 2026-07-11: rail protection, decoupling, wiring fixes
Protection:
- Sidecar +5V now feeds through a 2A polyfuse into +5V_ISA with an
  SMBJ5.0A clamp + 22uF bulk (a faulted ISA card trips its own fuse
  instead of dropping the board; back-fed voltage is clamped).
- USB-C VBUS enters through a 3A polyfuse with an SMBJ5.0A on +5V
  (backstop for the CFG1 9-20V failure mode). CH224K gains a 1uF VDD
  cap; its PG routes to Supervisor GPIO16 as PD_PG. Buck output
  doubled to 2x22uF, 10uF at VIN, extra rail bulk.
- Supervisor USB-A host port: 27R series termination (RP2040
  requirement), USBLC6-2SC6 ESD array, 100uF VBUS bulk.
- Video: HDMI +5V fused (500mA), HPD sensed on GPIO41, 100R series on
  VGA sync. TMDS ESD array deferred to layout (no symbol).
- card_isatest: V5RAW bulk, Q1 gate soft-start cap, TVS on DUT rail.

Wiring fixes:
- SPKR had no driver anywhere (netlist: 1 node). Bus MCU GPIO22
  reassigned from the diagnostics-only bus-CLK sense to SPKR; bus_mcu
  drops CLK from its interface. Doc 5.2 updated.
- bus_mcu C8 decoupled +3V3, a rail that sheet never uses -> 3V3_BUS.
- Storage IRQ5 was push-pull (permanently driven when idle) -> 2N7002
  + gated '125 tri-state, same convention as the LPT IRQ7 stage.
- MAX3241 pump caps resized to the 5V datasheet values (47nF/330nF).
- LPT DB25 status inputs get 4.7k pull-ups (floated with no printer).
- Audio line-out gets a 100R series isolator before the jack.

Best practices:
- Decoupling to ~1x100nF per IC on every sheet + bulk per board
  (cpu_core 7->16 incl. the naked 3.3V oscillator, storage 4->11,
  parallel 6->13, rtc/com/video/bus_mcu/card_isatest similar).
- All floating spare CMOS inputs tied ('00/'74/'157/'02/'04/'125
  sections across cpu_core, bus_mcu, rtc, storage, card_isatest).

Sourcing: new parts mapped in parts.py with JLC-verified LCSC numbers;
Power_Protection lib registered in the tools; TPS563200 stock alert
(4 pcs left at JLC) flagged in parts.py + jlcpcb-sourcing.md. All
decisi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
Parts:
- added C10, C11, C12, C13, C2, C3, C4, C5, C6, C7, C8, C9: 100nF, symbol Device:C
- added C14: 10uF, symbol Device:C
- R1: renamed from C1; value 100nF -> 4.7k; symbol Device:C -> Device:R; LCSC Part Num C14663 -> C23162
- R2: renamed from C2; value 100nF -> 4.7k; symbol Device:C -> Device:R; LCSC Part Num C14663 -> C23162
- R3: renamed from C3; value 100nF -> 4.7k; symbol Device:C -> Device:R; LCSC Part Num C14663 -> C23162
- R4: renamed from C4; value 100nF -> 4.7k; symbol Device:C -> Device:R; LCSC Part Num C14663 -> C23162
- R5: renamed from C5; value 100nF -> 4.7k; symbol Device:C -> Device:R; LCSC Part Num C14663 -> C23162
- renumbered C6 to C1
Connections:
- net +5V: now also C10.1, C11.1, C12.1, C13.1, C14.1, C2.1, C3.1, C4.1, C5.1, C6.1, C7.1, C8.1, C9.1
- net GND: now also C10.2, C11.2, C12.2, C13.2, C14.2, C2.2, C3.2, C4.2, C5.2, C6.2, C7.2, C8.2, C9.2; no longer R1.2, R2.2, R3.2, R4.2, R5.2
- net P_ACK: now also R1.2
- net P_BUSY: now also R2.2
- net P_ERR: now also R5.2
- net P_PE: now also R3.2
- net P_SEL: now also R4.2
Other:
- moved on the sheet: C1
