File: hardware/cards/card_video.kicad_sch (KiCad schematic)
At the start: 45 parts, among them J1 HDMI_A, J2 VGA HD15, M1 Core2350B (8MB PSRAM), U2 74LVC245A, U3 74LVC245A, U4 74LVC245A, U5 74LVC245A

Commit message: addr_decode: hardwire LPT/IDE bases; centralize NIC + video disables (JP1-JP6)
LPT fixed at 0x378, IDE at 0x300 -- both base straps and their pull-ups
deleted ('138 ~Y1 now NC, the '00's ~A5 gate spare, IDE OR-leg takes raw
A5). The NIC and video disable jumpers move to addr_decode as JP5/JP6
with the same fit-to-disable sense as the rest: their gating hardware
stays local (the NIC's isolation '125 inside the 5V island, video's
firmware boot strap on GPIO42), only the jumper levels cross as
mxbus.PRIV_DIS -- video's documented firmware polarity inverts (high =
disabled; no firmware exists yet). Disable row is now a uniform JP1-JP6
(COM1/COM2/LPT/IDE/NIC/VID), bare board runs everything; network JP1/R6
and video JP1/R30 deleted, VID_BASE becomes video JP1. card_video's
wrapper re-adds a local DIS_VID strap (the documented PRIV lift
pattern). Docs/tables/decision logs aligned.

Co-Authored-By: Claude Fable 5 <noreply@anthropic.com>
Parts:
- removed J2: VGA HD15, Connector_Dsub:DSUB-15-HD_Socket_Horizontal_P2.29x2.54mm_EdgePinOffset8.35mm_Housed_MountingHolesOffset10.89mm, symbol Connector_Generic:Conn_01x15
- removed R29: 100, Resistor_SMD:R_0603_1608Metric, symbol Device:R
- removed R31: 10k, Resistor_SMD:R_0603_1608Metric, symbol Device:R
- removed U2: 74LVC245A, Package_SO:TSSOP-20_4.4x6.5mm_P0.65mm, symbol mini-xt:74LVC245A
- added JP2: DIS_VID, Connector_PinHeader_2.54mm:PinHeader_1x02_P2.54mm_Vertical, symbol Connector_Generic:Conn_01x02
- added R20: 2k, Resistor_SMD:R_0603_1608Metric, symbol Device:R
- added R21: 1k, Resistor_SMD:R_0603_1608Metric, symbol Device:R
- added R30: 10k, Resistor_SMD:R_0603_1608Metric, symbol Device:R
- J2: renamed from R28; value 100 -> VGA HD15; footprint Resistor_SMD:R_0603_1608Metric -> Connector_Dsub:DSUB-15-HD_Socket_Horizontal_P2.29x2.54mm_EdgePinOffset8.35mm_Housed_MountingHolesOffset10.89mm; symbol Device:R -> Connector_Generic:Conn_01x15; LCSC Part Num C22775 -> (none)
- JP1: value VID_EN -> VID_BASE
- R22: renamed from R20; value 2k -> 510; LCSC Part Num C22975 -> C23193
- R23: renamed from R21; value 1k -> 2k; LCSC Part Num C21190 -> C22975
- R24: renamed from R22; value 510 -> 1k; LCSC Part Num C23193 -> C21190
- R25: renamed from R23; value 2k -> 510; LCSC Part Num C22975 -> C23193
- R26: renamed from R24; value 1k -> 820; LCSC Part Num C21190 -> C23253
- R27: renamed from R25; value 510 -> 470; LCSC Part Num C23193 -> C23179
- R28: renamed from R26; value 820 -> 100; LCSC Part Num C23253 -> C22775
- R29: renamed from R27; value 470 -> 100; LCSC Part Num C23179 -> C22775
- R31: renamed from JP2; value VID_BASE -> 10k; footprint Connector_PinHeader_2.54mm:PinHeader_1x02_P2.54mm_Vertical -> Resistor_SMD:R_0603_1608Metric; symbol Connector_Generic:Conn_01x02 -> Device:R; LCSC Part Num C2337 -> C25804
- U2: renamed from R30; value 10k -> 74LVC245A; footprint Resistor_SMD:R_0603_1608Metric -> Package_SO:TSSOP-20_4.4x6.5mm_P0.65mm; symbol Device:R -> mini-xt:74LVC245A; LCSC Part Num C25804 -> C6082
Connections:
- net 3V3_VID: now also R31.1, U2.20 (VCC), JP2.2 (Pin_2); no longer U2.1
- net D0: now also U2.18 (B0)
- net D1: now also U2.17 (B1)
- net D2: now also U2.16 (B2)
- net D3: now also U2.15 (B3)
- net D4: now also U2.14 (B4)
- net D5: now also U2.13 (B5)
- net D6: now also U2.12 (B6)
- net D7: now also U2.11 (B7)
- net DDIR: now also U2.1 (A->B)
- net DOE: now also U2.19 (CE)
- net GND: now also J2.10 (Pin_10), J2.5 (Pin_5), J2.6 (Pin_6), J2.7 (Pin_7), J2.8 (Pin_8), U2.10 (GND), R30.2; no longer R31.2 (Pin_2)
- net HSYNC: now also R28.1; no longer J2.1
- net HSYNC_J: now also J2.13 (Pin_13), R28.2; no longer J2.2
- net SB0: now also U2.2 (A0)
- net SB1: now also U2.3 (A1)
- net SB2: now also U2.4 (A2)
- net SB3: now also U2.5 (A3)
- net SB4: now also U2.6 (A4)
- net SB5: now also U2.7 (A5)
- net SB6: now also U2.8 (A6)
- net SB7: now also U2.9 (A7)
- net VB0: now also R26.1; no longer R28.1
- net VB1: now also R27.1; no longer R29.1
- net VG0: now also R23.1; no longer R25.1
- net VG1: now also R24.1; no longer R26.1
- net VG2: now also R25.1; no longer R27.1
- net VGA_B: now also J2.3 (Pin_3), R26.2, R27.2; no longer R28.2, R29.2
- net VGA_G: now also J2.2 (Pin_2), R23.2, R24.2; no longer R26.2, R27.2
- net VGA_R: now also J2.1 (Pin_1), R20.2, R21.2; no longer R23.2, R24.2
- net VID_BASE: now also JP1.1 (Pin_1), R31.2; no longer R31.1 (Pin_1)
- net VR0: now also R20.1; no longer R22.1
- net VR1: now also R21.1; no longer R23.1
- net VR2: now also R22.1; no longer R24.1
- net VSYNC: now also R29.1
- net VSYNC_J: now also J2.14 (Pin_14), R29.2
- removed net VID_EN: JP1.1 (Pin_1), M1.43 (GPIO42), U2.2
- new net DIS_VID: JP2.1 (Pin_1), M1.43 (GPIO42), R30.1
Other:
- note added: "SOFT CARD: ISA bus + power ONLY. Self-decodes 0xA0000-0xBFFFF and 3B4/3B5/3B8/3BA/3BF + 3D4/3D5/3D8/3D9/3DA from snooped A17-A19/A0-A9. No Y5, no link, no host RAM (design S8). Disable: addr_decode JP6 (DIS_VID high, firmware keeps all OEs off; enabled by default). JP1 = CGA (closed) / MDA (open) window set."
- note removed: "SOFT CARD: ISA bus + power ONLY. Self-decodes 0xA0000-0xBFFFF and 3B4/3B5/3B8/3BA/3BF + 3D4/3D5/3D8/3D9/3DA from snooped A17-A19/A0-A9. No Y5, no link, no host RAM (design S8). Straps: JP1 open = card disabled (firmware keeps all OEs off); JP2 = CGA (closed) / MDA (open) window set."
- moved on the sheet: JP1, R22, R23, R24, R25, R26, R27, R28, R29
Changed lines of the file:
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@@
 		)
 	)
-	(label "VID_EN"
+	(label "DIS_VID"
 		(at 181.61 156.21 0)
 		(effects
@@
 	(wire
 		(pts
-			(xy 116.84 40.64)
-			(xy 119.38 40.64)
-		)
-		(stroke
-			(width 0)
-			(type default)
-		)
-	)
-	(label "VID_EN"
-		(at 119.38 40.64 0)
-		(effects
-			(font
-				(size 1.27 1.27)
-			)
-		)
-	)
-	(wire
-		(pts
-			(xy 116.84 43.18)
-			(xy 119.38 43.18)
-		)
-		(stroke
-			(width 0)
-			(type default)
-		)
-	)
-	(global_label "GND"
-		(shape input)
-		(at 119.38 43.18 0)
-		(effects
-			(font
-				(size 1.27 1.27)
-			)
-		)
-	)
-	(wire
-		(pts
 			(xy 132.08 40.64)
 			(xy 134.62 40.64)
@@
 	(wire
 		(pts
-			(xy 121.92 57.15)
-			(xy 121.92 54.61)
-		)
-		(stroke
-			(width 0)
-			(type default)
-		)
-	)
-	(label "3V3_VID"
-		(at 121.92 54.61 90)
-		(effects
-			(font
-				(size 1.27 1.27)
-			)
-		)
-	)
-	(wire
-		(pts
-			(xy 121.92 64.77)
-			(xy 121.92 67.31)
-		)
-		(stroke
-			(width 0)
-			(type default)
-		)
-	)
-	(label "VID_EN"
-		(at 121.92 67.31 270)
-		(effects
-			(font
-				(size 1.27 1.27)
-			)
-		)
-	)
-	(wire
-		(pts
 			(xy 137.16 57.15)
 			(xy 137.16 54.61)
@@
 		(at 317.5 233.68)
 	)
-	(text "SOFT CARD: ISA bus + power ONLY. Self-decodes 0xA0000-0xBFFFF and 3B4/3B5/3B8/3BA/3BF + 3D4/3D5/3D8/3D9/3DA from snooped A17-A19/A0-A9. No Y5, no link, no host RAM (design S8). Straps: JP1 open = card disabled (firmware keeps all OEs off); JP2 = CGA (closed) / MDA (open) window set."
+	(text "SOFT CARD: ISA bus + power ONLY. Self-decodes 0xA0000-0xBFFFF and 3B4/3B5/3B8/3BA/3BF + 3D4/3D5/3D8/3D9/3DA from snooped A17-A19/A0-A9. No Y5, no link, no host RAM (design S8). Disable: addr_decode JP6 (DIS_VID high, firmware keeps all OEs off; enabled by default). JP1 = CGA (closed) / MDA (open) window set."
 		(at 38.1 20.32 0)
 		(effects
@@
 		)
 	)
+	(wire
+		(pts
+			(xy 116.84 40.64)
+			(xy 119.38 40.64)
+		)
+		(stroke
+			(width 0)
+			(type default)
+		)
+	)
+	(label "DIS_VID"
+		(at 119.38 40.64 0)
+		(effects
+			(font
+				(size 1.27 1.27)
+			)
+		)
+	)
+	(wire
+		(pts
+			(xy 116.84 43.18)
+			(xy 119.38 43.18)
+		)
+		(stroke
+			(width 0)
+			(type default)
+		)
+	)
+	(label "3V3_VID"
+		(at 119.38 43.18 0)
+		(effects
+			(font
+				(size 1.27 1.27)
+			)
+		)
+	)
+	(wire
+		(pts
+			(xy 121.92 57.15)
+			(xy 121.92 54.61)
+		)
+		(stroke
+			(width 0)
+			(type default)
+		)
+	)
+	(label "DIS_VID"
+		(at 121.92 54.61 90)
+		(effects
+			(font
+				(size 1.27 1.27)
+			)
+		)
+	)
+	(wire
+		(pts
+			(xy 121.92 64.77)
+			(xy 121.92 67.31)
+		)
+		(stroke
+			(width 0)
+			(type default)
+		)
+	)
+	(global_label "GND"
+		(shape input)
+		(at 121.92 67.31 270)
+		(effects
+			(font
+				(size 1.27 1.27)
+			)
+		)
+	)
 	(text "Standalone Video PCB: ISA bus chains J_IN -> J_OUT; card logic taps the bus by name. Daisy-chain cards header-to-header (isa_conn, S4.3)."
 		(at 38.1 12.7 0)
@@
 	(symbol
 		(lib_id "Connector_Generic:Conn_01x02")
-		(at 121.92 40.64 0)
-		(unit 1)
-		(exclude_from_sim no)
-		(in_bom yes)
-		(on_board yes)
-		(dnp no)
-		(fields_autoplaced yes)
-		(property "Reference" "JP1"
-			(at 121.92 35.56 0)
-			(effects
-				(font
-					(size 1.27 1.27)
-				)
-			)
-		)
-		(property "Value" "VID_EN"
-			(at 121.92 45.72 0)
-			(effects
-				(font
-					(size 1.27 1.27)
-				)
-			)
-		)
-		(property "Footprint" "Connector_PinHeader_2.54mm:PinHeader_1x02_P2.54mm_Vertical"
-			(at 121.92 40.64 0)
-			(effects
-				(font
-					(size 1.27 1.27)
-				)
-				(hide yes)
-			)
-		)
-		(property "LCSC Part Num" "C2337"
-			(at 121.92 40.64 0)
-			(effects
-				(font
-					(size 1.27 1.27)
-				)
-				(hide yes)
-			)
-		)
-		(pin "1"
-		)
-		(pin "2"
-		)
-		(instances
-			(project "card_video"
-				(path "/6b5ebf7b-92ce-58a1-8c1d-03e449d8e3c9"
-					(reference "JP1")
-					(unit 1)
-				)
-			)
-		)
-	)
-	(symbol
-		(lib_id "Connector_Generic:Conn_01x02")
 		(at 137.16 40.64 0)
 		(unit 1)
@@
 		(dnp no)
 		(fields_autoplaced yes)
-		(property "Reference" "JP2"
+		(property "Reference" "JP1"
 			(at 137.16 35.56 0)
 			(effects
@@
 			(project "card_video"
 				(path "/6b5ebf7b-92ce-58a1-8c1d-03e449d8e3c9"
-					(reference "JP2")
-					(unit 1)
-				)
-			)
-		)
-	)
-	(symbol
-		(lib_id "Device:R")
-		(at 121.92 60.96 0)
-		(unit 1)
-		(exclude_from_sim no)
-		(in_bom yes)
-		(on_board yes)
-		(dnp no)
-		(fields_autoplaced yes)
-		(property "Reference" "R30"
-			(at 121.92 55.88 0)
-			(effects
-				(font
-					(size 1.27 1.27)
-				)
-			)
-		)
-		(property "Value" "10k"
-			(at 121.92 66.04 0)
-			(effects
-				(font
-					(size 1.27 1.27)
-				)
-			)
-		)
-		(property "Footprint" "Resistor_SMD:R_0603_1608Metric"
-			(at 121.92 60.96 0)
-			(effects
-				(font
-					(size 1.27 1.27)
-				)
-				(hide yes)
-			)
-		)
-		(property "LCSC Part Num" "C25804"
-			(at 121.92 60.96 0)
-			(effects
-				(font
-					(size 1.27 1.27)
-				)
-				(hide yes)
-			)
-		)
-		(pin "1"
-		)
-		(pin "2"
-		)
-		(instances
-			(project "card_video"
-				(path "/6b5ebf7b-92ce-58a1-8c1d-03e449d8e3c9"
-					(reference "R30")
+					(reference "JP1")
 					(unit 1)
 				)
@@
 					(unit 1)
 				)
+			)
+		)
+	)
+	(symbol
+		(lib_id "Connector_Generic:Conn_01x02")
+		(at 121.92 40.64 0)
+		(unit 1)
+		(exclude_from_sim no)
+		(in_bom yes)
+		(on_board yes)
+		(dnp no)
+		(fields_autoplaced yes)
+		(property "Reference" "JP2"
+			(at 121.92 35.56 0)
+			(effects
+				(font
+					(size 1.27 1.27)
+				)
+			)
+		)
+		(property "Value" "DIS_VID"
+			(at 121.92 45.72 0)
+			(effects
+				(font
+					(size 1.27 1.27)
+				)
+			)
+		)
+		(property "Footprint" "Connector_PinHeader_2.54mm:PinHeader_1x02_P2.54mm_Vertical"
+			(at 121.92 40.64 0)
+			(effects
+				(font
+					(size 1.27 1.27)
+				)
+				(hide yes)
+			)
+		)
+		(property "LCSC Part Num" "C2337"
+			(at 121.92 40.64 0)
+			(effects
+				(font
+					(size 1.27 1.27)
+				)
+				(hide yes)
+			)
+		)
+		(pin "1"
+		)
+		(pin "2"
+		)
+		(instances
+			(project "card_video"
+				(path "/6b5ebf7b-92ce-58a1-8c1d-03e449d8e3c9"
+					(reference "JP2")
+					(unit 1)
+				)
+			)
+		)
+	)
+	(symbol
+		(lib_id "Device:R")
+		(at 121.92 60.96 0)
+		(unit 1)
+		(exclude_from_sim no)
+		(in_bom yes)
+		(on_board yes)
+		(dnp no)
+		(fields_autoplaced yes)
+		(property "Reference" "R30"
+			(at 121.92 55.88 0)
+			(effects
+				(font
+					(size 1.27 1.27)
+				)
+			)
+		)
+		(property "Value" "10k"
+			(at 121.92 66.04 0)
+			(effects
+				(font
+					(size 1.27 1.27)
+				)
+			)
+		)
+		(property "Footprint" "Resistor_SMD:R_0603_1608Metric"
+			(at 121.92 60.96 0)
+			(effects
+				(font
+					(size 1.27 1.27)
+				)
+				(hide yes)
+			)
+		)
+		(property "LCSC Part Num" "C25804"
+			(at 121.92 60.96 0)
+			(effects
+				(font
+					(size 1.27 1.27)
+				)
+				(hide yes)
+			)
+		)
+		(pin "1"
+		)
+		(pin "2"
+		)
+		(instances
+			(project "card_video"
+				(path "/6b5ebf7b-92ce-58a1-8c1d-03e449d8e3c9"
+					(reference "R30")
+					(unit 1)
+				)

Commit message: Passives: basic-library audit + 4x resistor-array pull consolidation
Audit: every discrete R/C value was already JLC basic except the ferrite
beads -- swapped to basic Murata BLM18PG121SN1D (C14709, 120R@100MHz,
same family/role). The 100uF electrolytic and buck inductor stay
extended (zero fee-free parts exist in those subcategories). Pruned the
orphaned 5V-era 47nF/330nF MAX3241 cap entries.

Pull consolidation: 65 discrete 10k/4.7k rail pulls across 8 sheets
collapse into 18 basic 4-element isolated arrays (4D03WGJ0103T5E /
4D03WGJ0472T5E, element k = pins k/9-k; new mxbus.r_pack4 helper).
Isolated elements let packs mix rails; every net keeps its exact rail
and semantics (verified element-by-element in the netlist). RC/divider/
series/I2C resistors stay discrete. Board 452 -> 406 components; also
de-risks the sole basic 10k 0603 line (0 stock at audit). Audit
recorded in jlcpcb-sourcing.md.

Co-Authored-By: Claude Fable 5 <noreply@anthropic.com>
Parts:
- removed JP1: VID_BASE, Connector_PinHeader_2.54mm:PinHeader_1x02_P2.54mm_Vertical, symbol Connector_Generic:Conn_01x02
- removed R33, R34, R35, R36: 10k, Resistor_SMD:R_0603_1608Metric, symbol Device:R
- added RN2: 10kx4, Resistor_SMD:R_Array_Convex_4x0603, symbol Device:R_Pack04
- JP1: renamed from R31; value 10k -> VID_BASE; footprint Resistor_SMD:R_0603_1608Metric -> Connector_PinHeader_2.54mm:PinHeader_1x02_P2.54mm_Vertical; symbol Device:R -> Connector_Generic:Conn_01x02; LCSC Part Num C25804 -> C2337
- RN1: renamed from R32; value 10k -> 10kx4; footprint Resistor_SMD:R_0603_1608Metric -> Resistor_SMD:R_Array_Convex_4x0603; symbol Device:R -> Device:R_Pack04; LCSC Part Num C25804 -> C29718
Connections:
- net 3V3_VID: now also RN1.5 (R4.2), RN1.6 (R3.2), RN1.7 (R2.2), RN1.8 (R1.2), RN2.8 (R1.2); no longer JP1.1
- net AOE_HI: now also RN1.4 (R4.1)
- net AOE_LO: now also RN1.2 (R2.1)
- net AOE_MID: now also RN1.3 (R3.1)
- net DDIR: now also RN2.2 (R2.1); no longer RN1.2
- net DOE: now also RN1.1 (R1.1)
- net GND: now also JP1.2 (Pin_2), RN2.7 (R2.2); no longer RN1.1
- net VID_BASE: now also JP1.1 (Pin_1), RN2.1 (R1.1); no longer JP1.2
- no-connect marks 32 -> 36

Commit message: Remove the on-board RTL8019AS NIC (tag full-board-with-nic preserves it)
Network sheet, symbols, and NIC-only parts.py bindings deleted; addr_decode
JP6->JP5 (DIS_VID); IRQ2 retired as an internal net like IRQ6/IRQ8 (still
reachable as EXT_IRQ2 from the expansion port). ERC stays 0/0.

Co-Authored-By: Claude Fable 5 <noreply@anthropic.com>
Other:
- note added: "SOFT CARD: ISA bus + power ONLY. Self-decodes 0xA0000-0xBFFFF and 3B4/3B5/3B8/3BA/3BF + 3D4/3D5/3D8/3D9/3DA from snooped A17-A19/A0-A9. No Y5, no link, no host RAM (design S8). Disable: addr_decode JP5 (DIS_VID high, firmware keeps all OEs off; enabled by default). JP1 = CGA (closed) / MDA (open) window set."
- note removed: "SOFT CARD: ISA bus + power ONLY. Self-decodes 0xA0000-0xBFFFF and 3B4/3B5/3B8/3BA/3BF + 3D4/3D5/3D8/3D9/3DA from snooped A17-A19/A0-A9. No Y5, no link, no host RAM (design S8). Disable: addr_decode JP6 (DIS_VID high, firmware keeps all OEs off; enabled by default). JP1 = CGA (closed) / MDA (open) window set."
Changed lines of the file:
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@@
 		(at 317.5 233.68)
 	)
-	(text "SOFT CARD: ISA bus + power ONLY. Self-decodes 0xA0000-0xBFFFF and 3B4/3B5/3B8/3BA/3BF + 3D4/3D5/3D8/3D9/3DA from snooped A17-A19/A0-A9. No Y5, no link, no host RAM (design S8). Disable: addr_decode JP6 (DIS_VID high, firmware keeps all OEs off; enabled by default). JP1 = CGA (closed) / MDA (open) window set."
+	(text "SOFT CARD: ISA bus + power ONLY. Self-decodes 0xA0000-0xBFFFF and 3B4/3B5/3B8/3BA/3BF + 3D4/3D5/3D8/3D9/3DA from snooped A17-A19/A0-A9. No Y5, no link, no host RAM (design S8). Disable: addr_decode JP5 (DIS_VID high, firmware keeps all OEs off; enabled by default). JP1 = CGA (closed) / MDA (open) window set."
 		(at 38.1 20.32 0)
 		(effects
