File: hardware/sheets/com_port.kicad_sch (KiCad schematic)
At the start: 27 parts, among them J1 DE9_Pins, J2 Conn_01x03, J3 Conn_01x04, U1 16550, U2 MAX3241, U3 74HCT04, U4 74HCT08, U5 74HCT08, U6 74HCT125, Y1 1.8432MHz

Commit message: Design-review fixes: reset parking, IRQ8 off the header, analog cleanups
Netlist-wide review sweep. IRQ8 leaves the 60-pin ISA header (pin 15 is a
second GND return; the on-board RTC owns IRQ8 exclusively, so its push-pull
drive is now correct by construction). Bus MCU Hi-Z parking completed:
~CPURESET pulled low (V20 held in reset while the MCU is unprogrammed),
~DACK1/~REFRESH parked deasserted, DRQ1 idled low. Supervisor 12 MHz crystal
damping R actually in series now (was parallel-to-nothing), plus a second
USBLC6 so both prog-port SW2 positions are ESD-protected. Audio: 0.5x PG
summing (MCP6002 headroom), 100k LINE bleed, unit B parked as a follower --
and the SUM stub moved off pin 5's row, where wiring unit B would have
silently merged SUM into VREF. CH224K VDD fed through 1k per the WCH ref
design. VGA blue ladder rescaled 1k/510 -> 820/470 (was ~12% blue-deficient).
Spare CMOS gate inputs grounded uniformly (cpu_core/rtc/storage); UART_RXD
pulled up (SIN idles at mark with JP1 open); dead pins/parts dropped
(com_port CLK, parallel RESET_DRV, storage R3). Bus CLK fixed at 7.16 MHz
logged as a decision. New passives mapped to JLC basic parts in parts.py.

Co-Authored-By: Claude Fable 5 <noreply@anthropic.com>
Parts:
- removed C1: 100nF, symbol Device:C
- removed JP3: COM_EN, symbol Connector_Generic:Conn_01x02
- added C13: 10uF, symbol Device:C
- added JP2: IRQ strap, symbol Connector_Generic:Conn_01x03
- added R2: 10k, symbol Device:R
- C12: renamed from C13; value 10uF -> 100nF; LCSC Part Num C15850 -> C14663
- JP3: renamed from R1; value 10k -> COM_EN; symbol Device:R -> Connector_Generic:Conn_01x02; LCSC Part Num C25804 -> C2337
- R1: renamed from JP2; value IRQ strap -> 10k; symbol Connector_Generic:Conn_01x03 -> Device:R; LCSC Part Num C2337 -> C25804
- renumbered C2 to C1, C11 to C10, C12 to C11, C9 to C2, C10 to C9
Connections:
- net +5V: now also JP3.2 (Pin_2), C13.1, R2.1
- net COM_EN: now also R1.1
- net COM_IRQ: now also JP2.2 (Pin_2); no longer R1.2 (Pin_2)
- net GND: now also R1.2, C13.2; no longer JP3.2
- net IRQ3: now also JP2.3 (Pin_3); no longer R1.3 (Pin_3)
- net IRQ4: now also JP2.1 (Pin_1); no longer R1.1 (Pin_1)
- net UART_RXD: now also R2.2
Other:
- note added: "J2 (base strap) has no default: it must ALWAYS be jumpered, or A8_SEL floats and the decode is undefined."
- moved on the sheet: C1, C10, C11, C12, C2, C9
Changed lines of the file:
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@@
 		)
 	)
-	(hierarchical_label "CLK"
-		(shape input)
-		(at 25.4 81.28 0)
-		(effects
-			(font
-				(size 1.27 1.27)
-			)
-		)
-	)
 	(hierarchical_label "IRQ3"
 		(shape output)
-		(at 25.4 83.82 0)
+		(at 25.4 81.28 0)
 		(effects
 			(font
@@
 	(hierarchical_label "IRQ4"
 		(shape output)
-		(at 25.4 86.36 0)
+		(at 25.4 83.82 0)
 		(effects
 			(font
@@
 	(wire
 		(pts
+			(xy 215.9 232.41)
+			(xy 215.9 229.87)
+		)
+		(stroke
+			(width 0)
+			(type default)
+		)
+	)
+	(global_label "+5V"
+		(shape input)
+		(at 215.9 229.87 90)
+		(effects
+			(font
+				(size 1.27 1.27)
+			)
+		)
+	)
+	(wire
+		(pts
+			(xy 215.9 240.03)
+			(xy 215.9 242.57)
+		)
+		(stroke
+			(width 0)
+			(type default)
+		)
+	)
+	(label "UART_RXD"
+		(at 215.9 242.57 270)
+		(effects
+			(font
+				(size 1.27 1.27)
+			)
+		)
+	)
+	(text "J2 (base strap) has no default: it must ALWAYS be jumpered, or A8_SEL floats and the decode is undefined."
+		(at 203.2 265.43 0)
+		(effects
+			(font
+				(size 1.27 1.27)
+			)
+		)
+	)
+	(wire
+		(pts
 			(xy 251.46 254)
 			(xy 254 254)
@@
 					(unit 1)
 				)
-				(path "/26736c46-8b40-5460-874f-03596d17270c/d1fcb6fc-b82b-597a-8371-e154571c8724"
+				(path "/26736c46-8b40-5460-874f-03596d17270c/4ac9139d-ec8b-5dcd-a7b7-dc5ad73e89a7"
 					(reference "U601")
 					(unit 1)
@@
 					(unit 1)
 				)
-				(path "/26736c46-8b40-5460-874f-03596d17270c/d1fcb6fc-b82b-597a-8371-e154571c8724"
+				(path "/26736c46-8b40-5460-874f-03596d17270c/4ac9139d-ec8b-5dcd-a7b7-dc5ad73e89a7"
 					(reference "Y601")
 					(unit 1)
@@
 					(unit 1)
 				)
-				(path "/26736c46-8b40-5460-874f-03596d17270c/d1fcb6fc-b82b-597a-8371-e154571c8724"
+				(path "/26736c46-8b40-5460-874f-03596d17270c/4ac9139d-ec8b-5dcd-a7b7-dc5ad73e89a7"
 					(reference "C607")
 					(unit 1)
@@
 					(unit 1)
 				)
-				(path "/26736c46-8b40-5460-874f-03596d17270c/d1fcb6fc-b82b-597a-8371-e154571c8724"
+				(path "/26736c46-8b40-5460-874f-03596d17270c/4ac9139d-ec8b-5dcd-a7b7-dc5ad73e89a7"
 					(reference "C608")
 					(unit 1)
@@
 					(unit 1)
 				)
-				(path "/26736c46-8b40-5460-874f-03596d17270c/d1fcb6fc-b82b-597a-8371-e154571c8724"
+				(path "/26736c46-8b40-5460-874f-03596d17270c/4ac9139d-ec8b-5dcd-a7b7-dc5ad73e89a7"
 					(reference "U603")
 					(unit 1)
@@
 					(unit 1)
 				)
-				(path "/26736c46-8b40-5460-874f-03596d17270c/d1fcb6fc-b82b-597a-8371-e154571c8724"
+				(path "/26736c46-8b40-5460-874f-03596d17270c/4ac9139d-ec8b-5dcd-a7b7-dc5ad73e89a7"
 					(reference "J602")
 					(unit 1)
@@
 					(unit 1)
 				)
-				(path "/26736c46-8b40-5460-874f-03596d17270c/d1fcb6fc-b82b-597a-8371-e154571c8724"
+				(path "/26736c46-8b40-5460-874f-03596d17270c/4ac9139d-ec8b-5dcd-a7b7-dc5ad73e89a7"
 					(reference "U604")
 					(unit 1)
@@
 					(unit 1)
 				)
-				(path "/26736c46-8b40-5460-874f-03596d17270c/d1fcb6fc-b82b-597a-8371-e154571c8724"
+				(path "/26736c46-8b40-5460-874f-03596d17270c/4ac9139d-ec8b-5dcd-a7b7-dc5ad73e89a7"
 					(reference "U605")
 					(unit 1)
@@
 					(unit 1)
 				)
-				(path "/26736c46-8b40-5460-874f-03596d17270c/d1fcb6fc-b82b-597a-8371-e154571c8724"
+				(path "/26736c46-8b40-5460-874f-03596d17270c/4ac9139d-ec8b-5dcd-a7b7-dc5ad73e89a7"
 					(reference "U606")
 					(unit 1)
@@
 					(unit 1)
 				)
-				(path "/26736c46-8b40-5460-874f-03596d17270c/d1fcb6fc-b82b-597a-8371-e154571c8724"
+				(path "/26736c46-8b40-5460-874f-03596d17270c/4ac9139d-ec8b-5dcd-a7b7-dc5ad73e89a7"
 					(reference "U602")
 					(unit 1)
@@
 					(unit 1)
 				)
-				(path "/26736c46-8b40-5460-874f-03596d17270c/d1fcb6fc-b82b-597a-8371-e154571c8724"
+				(path "/26736c46-8b40-5460-874f-03596d17270c/4ac9139d-ec8b-5dcd-a7b7-dc5ad73e89a7"
 					(reference "C603")
 					(unit 1)
@@
 					(unit 1)
 				)
-				(path "/26736c46-8b40-5460-874f-03596d17270c/d1fcb6fc-b82b-597a-8371-e154571c8724"
+				(path "/26736c46-8b40-5460-874f-03596d17270c/4ac9139d-ec8b-5dcd-a7b7-dc5ad73e89a7"
 					(reference "C604")
 					(unit 1)
@@
 					(unit 1)
 				)
-				(path "/26736c46-8b40-5460-874f-03596d17270c/d1fcb6fc-b82b-597a-8371-e154571c8724"
+				(path "/26736c46-8b40-5460-874f-03596d17270c/4ac9139d-ec8b-5dcd-a7b7-dc5ad73e89a7"
 					(reference "C605")
 					(unit 1)
@@
 					(unit 1)
 				)
-				(path "/26736c46-8b40-5460-874f-03596d17270c/d1fcb6fc-b82b-597a-8371-e154571c8724"
+				(path "/26736c46-8b40-5460-874f-03596d17270c/4ac9139d-ec8b-5dcd-a7b7-dc5ad73e89a7"
 					(reference "C606")
 					(unit 1)
@@
 					(unit 1)
 				)
-				(path "/26736c46-8b40-5460-874f-03596d17270c/d1fcb6fc-b82b-597a-8371-e154571c8724"
+				(path "/26736c46-8b40-5460-874f-03596d17270c/4ac9139d-ec8b-5dcd-a7b7-dc5ad73e89a7"
 					(reference "J601")
 					(unit 1)
@@
 					(unit 1)
 				)
-				(path "/26736c46-8b40-5460-874f-03596d17270c/d1fcb6fc-b82b-597a-8371-e154571c8724"
+				(path "/26736c46-8b40-5460-874f-03596d17270c/4ac9139d-ec8b-5dcd-a7b7-dc5ad73e89a7"
 					(reference "J603")
 					(unit 1)
@@
 					(unit 1)
 				)
-				(path "/26736c46-8b40-5460-874f-03596d17270c/d1fcb6fc-b82b-597a-8371-e154571c8724"
+				(path "/26736c46-8b40-5460-874f-03596d17270c/4ac9139d-ec8b-5dcd-a7b7-dc5ad73e89a7"
 					(reference "JP601")
 					(unit 1)
@@
 	)
 	(symbol
+		(lib_id "Device:R")
+		(at 215.9 236.22 0)
+		(unit 1)
+		(exclude_from_sim no)
+		(in_bom yes)
+		(on_board yes)
+		(dnp no)
+		(fields_autoplaced yes)
+		(property "Reference" "R2"
+			(at 215.9 231.14 0)
+			(effects
+				(font
+					(size 1.27 1.27)
+				)
+			)
+		)
+		(property "Value" "10k"
+			(at 215.9 241.3 0)
+			(effects
+				(font
+					(size 1.27 1.27)
+				)
+			)
+		)
+		(property "Footprint" ""
+			(at 215.9 236.22 0)
+			(effects
+				(font
+					(size 1.27 1.27)
+				)
+				(hide yes)
+			)
+		)
+		(property "LCSC Part Num" "C25804"
+			(at 215.9 236.22 0)
+			(effects
+				(font
+					(size 1.27 1.27)
+				)
+				(hide yes)
+			)
+		)
+		(pin "1"
+		)
+		(pin "2"
+		)
+		(instances
+			(project "mini-xt"
+				(path "/26736c46-8b40-5460-874f-03596d17270c/fbab751f-6bb5-5e59-bc57-f9a54ef2e9ab"
+					(reference "R502")
+					(unit 1)
+				)
+				(path "/26736c46-8b40-5460-874f-03596d17270c/4ac9139d-ec8b-5dcd-a7b7-dc5ad73e89a7"
+					(reference "R602")
+					(unit 1)
+				)
+			)
+		)
+	)
+	(symbol
 		(lib_id "Connector_Generic:Conn_01x02")
 		(at 256.54 254 0)
@@
 					(unit 1)
 				)
-				(path "/26736c46-8b40-5460-874f-03596d17270c/d1fcb6fc-b82b-597a-8371-e154571c8724"
+				(path "/26736c46-8b40-5460-874f-03596d17270c/4ac9139d-ec8b-5dcd-a7b7-dc5ad73e89a7"
 					(reference "JP603")
 					(unit 1)
@@
 					(unit 1)
 				)
-				(path "/26736c46-8b40-5460-874f-03596d17270c/d1fcb6fc-b82b-597a-8371-e154571c8724"
+				(path "/26736c46-8b40-5460-874f-03596d17270c/4ac9139d-ec8b-5dcd-a7b7-dc5ad73e89a7"
 					(reference "R601")
 					(unit 1)
@@
 					(unit 1)
 				)
-				(path "/26736c46-8b40-5460-874f-03596d17270c/d1fcb6fc-b82b-597a-8371-e154571c8724"
+				(path "/26736c46-8b40-5460-874f-03596d17270c/4ac9139d-ec8b-5dcd-a7b7-dc5ad73e89a7"
 					(reference "JP602")
 					(unit 1)
@@
 					(unit 1)
 				)
-				(path "/26736c46-8b40-5460-874f-03596d17270c/d1fcb6fc-b82b-597a-8371-e154571c8724"
+				(path "/26736c46-8b40-5460-874f-03596d17270c/4ac9139d-ec8b-5dcd-a7b7-dc5ad73e89a7"
 					(reference "C601")
 					(unit 1)
@@
 					(unit 1)
 				)
-				(path "/26736c46-8b40-5460-874f-03596d17270c/d1fcb6fc-b82b-597a-8371-e154571c8724"
+				(path "/26736c46-8b40-5460-874f-03596d17270c/4ac9139d-ec8b-5dcd-a7b7-dc5ad73e89a7"
 					(reference "C602")
 					(unit 1)
@@
 					(unit 1)
 				)
-				(path "/26736c46-8b40-5460-874f-03596d17270c/d1fcb6fc-b82b-597a-8371-e154571c8724"
+				(path "/26736c46-8b40-5460-874f-03596d17270c/4ac9139d-ec8b-5dcd-a7b7-dc5ad73e89a7"
 					(reference "C609")
 					(unit 1)
@@
 					(unit 1)
 				)
-				(path "/26736c46-8b40-5460-874f-03596d17270c/d1fcb6fc-b82b-597a-8371-e154571c8724"
+				(path "/26736c46-8b40-5460-874f-03596d17270c/4ac9139d-ec8b-5dcd-a7b7-dc5ad73e89a7"
 					(reference "C610")
 					(unit 1)
@@
 					(unit 1)
 				)
-				(path "/26736c46-8b40-5460-874f-03596d17270c/d1fcb6fc-b82b-597a-8371-e154571c8724"
+				(path "/26736c46-8b40-5460-874f-03596d17270c/4ac9139d-ec8b-5dcd-a7b7-dc5ad73e89a7"
 					(reference "C611")
 					(unit 1)
@@
 					(unit 1)
 				)
-				(path "/26736c46-8b40-5460-874f-03596d17270c/d1fcb6fc-b82b-597a-8371-e154571c8724"
+				(path "/26736c46-8b40-5460-874f-03596d17270c/4ac9139d-ec8b-5dcd-a7b7-dc5ad73e89a7"
 					(reference "C612")
 					(unit 1)
@@
 					(unit 1)
 				)
-				(path "/26736c46-8b40-5460-874f-03596d17270c/d1fcb6fc-b82b-597a-8371-e154571c8724"
+				(path "/26736c46-8b40-5460-874f-03596d17270c/4ac9139d-ec8b-5dcd-a7b7-dc5ad73e89a7"
 					(reference "C613")
 					(unit 1)
