File: hardware/sheets/rtc.kicad_sch (KiCad schematic)
At the start: 14 parts, among them U1 DS12C887, U2 74HCT138, U3 74HC02, U4 74HCT08, U5 74HCT32, U6 74HCT04

Commit message: Design-review fixes: reset parking, IRQ8 off the header, analog cleanups
Netlist-wide review sweep. IRQ8 leaves the 60-pin ISA header (pin 15 is a
second GND return; the on-board RTC owns IRQ8 exclusively, so its push-pull
drive is now correct by construction). Bus MCU Hi-Z parking completed:
~CPURESET pulled low (V20 held in reset while the MCU is unprogrammed),
~DACK1/~REFRESH parked deasserted, DRQ1 idled low. Supervisor 12 MHz crystal
damping R actually in series now (was parallel-to-nothing), plus a second
USBLC6 so both prog-port SW2 positions are ESD-protected. Audio: 0.5x PG
summing (MCP6002 headroom), 100k LINE bleed, unit B parked as a follower --
and the SUM stub moved off pin 5's row, where wiring unit B would have
silently merged SUM into VREF. CH224K VDD fed through 1k per the WCH ref
design. VGA blue ladder rescaled 1k/510 -> 820/470 (was ~12% blue-deficient).
Spare CMOS gate inputs grounded uniformly (cpu_core/rtc/storage); UART_RXD
pulled up (SIN idles at mark with JP1 open); dead pins/parts dropped
(com_port CLK, parallel RESET_DRV, storage R3). Bus CLK fixed at 7.16 MHz
logged as a decision. New passives mapped to JLC basic parts in parts.py.

Co-Authored-By: Claude Fable 5 <noreply@anthropic.com>
Connections:
- net GND: now also U5.10 (P10), U5.12 (P12), U5.13 (P13), U5.9 (P9), U6.13 (P13)
- no-connect marks 4 -> 5
Changed lines of the file:
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@@
+	(wire
+		(pts
+			(xy 138.43 161.29)
+			(xy 135.89 161.29)
+		)
+		(stroke
+			(width 0)
+			(type default)
+		)
+	)
+	(global_label "GND"
+		(shape input)
+		(at 135.89 161.29 180)
+		(effects
+			(font
+				(size 1.27 1.27)
+			)
+		)
+	)
+	(wire
+		(pts
+			(xy 138.43 163.83)
+			(xy 135.89 163.83)
+		)
+		(stroke
+			(width 0)
+			(type default)
+		)
+	)
+	(global_label "GND"
+		(shape input)
+		(at 135.89 163.83 180)
+		(effects
+			(font
+				(size 1.27 1.27)
+			)
+		)
+	)
+	(wire
+		(pts
+			(xy 138.43 166.37)
+			(xy 135.89 166.37)
+		)
+		(stroke
+			(width 0)
+			(type default)
+		)
+	)
+	(global_label "GND"
+		(shape input)
+		(at 135.89 166.37 180)
+		(effects
+			(font
+				(size 1.27 1.27)
+			)
+		)
+	)
+	(wire
+		(pts
+			(xy 138.43 168.91)
+			(xy 135.89 168.91)
+		)
+		(stroke
+			(width 0)
+			(type default)
+		)
+	)
+	(global_label "GND"
+		(shape input)
+		(at 135.89 168.91 180)
+		(effects
+			(font
+				(size 1.27 1.27)
+			)
+		)
+	)
+	(no_connect
+		(at 166.37 156.21)
+	)
+	(no_connect
+		(at 166.37 158.75)
+	)
 	(wire
 		(pts
@@
 		)
 	)
-	(no_connect
-		(at 74.93 166.37)
+	(wire
+		(pts
+			(xy 74.93 166.37)
+			(xy 72.39 166.37)
+		)
+		(stroke
+			(width 0)
+			(type default)
+		)
+	)
+	(global_label "GND"
+		(shape input)
+		(at 72.39 166.37 180)
+		(effects
+			(font
+				(size 1.27 1.27)
+			)
+		)
 	)
 	(no_connect
@@
 		(instances
 			(project "mini-xt"
-				(path "/26736c46-8b40-5460-874f-03596d17270c/3898b474-78c8-51e2-a636-c7ffe2ed1375"
+				(path "/26736c46-8b40-5460-874f-03596d17270c/fbebb8e3-66b2-5aa7-ba3c-4936c50e8f80"
 					(reference "U801")
 					(unit 1)
@@
 		(instances
 			(project "mini-xt"
-				(path "/26736c46-8b40-5460-874f-03596d17270c/3898b474-78c8-51e2-a636-c7ffe2ed1375"
+				(path "/26736c46-8b40-5460-874f-03596d17270c/fbebb8e3-66b2-5aa7-ba3c-4936c50e8f80"
 					(reference "R801")
 					(unit 1)
@@
 		(instances
 			(project "mini-xt"
-				(path "/26736c46-8b40-5460-874f-03596d17270c/3898b474-78c8-51e2-a636-c7ffe2ed1375"
+				(path "/26736c46-8b40-5460-874f-03596d17270c/fbebb8e3-66b2-5aa7-ba3c-4936c50e8f80"
 					(reference "U802")
 					(unit 1)
@@
 		(instances
 			(project "mini-xt"
-				(path "/26736c46-8b40-5460-874f-03596d17270c/3898b474-78c8-51e2-a636-c7ffe2ed1375"
+				(path "/26736c46-8b40-5460-874f-03596d17270c/fbebb8e3-66b2-5aa7-ba3c-4936c50e8f80"
 					(reference "U803")
 					(unit 1)
@@
 		(instances
 			(project "mini-xt"
-				(path "/26736c46-8b40-5460-874f-03596d17270c/3898b474-78c8-51e2-a636-c7ffe2ed1375"
+				(path "/26736c46-8b40-5460-874f-03596d17270c/fbebb8e3-66b2-5aa7-ba3c-4936c50e8f80"
 					(reference "U804")
 					(unit 1)
@@
 		(instances
 			(project "mini-xt"
-				(path "/26736c46-8b40-5460-874f-03596d17270c/3898b474-78c8-51e2-a636-c7ffe2ed1375"
+				(path "/26736c46-8b40-5460-874f-03596d17270c/fbebb8e3-66b2-5aa7-ba3c-4936c50e8f80"
 					(reference "U805")
 					(unit 1)
@@
 		(instances
 			(project "mini-xt"
-				(path "/26736c46-8b40-5460-874f-03596d17270c/3898b474-78c8-51e2-a636-c7ffe2ed1375"
+				(path "/26736c46-8b40-5460-874f-03596d17270c/fbebb8e3-66b2-5aa7-ba3c-4936c50e8f80"
 					(reference "U806")
 					(unit 1)
@@
 		(instances
 			(project "mini-xt"
-				(path "/26736c46-8b40-5460-874f-03596d17270c/3898b474-78c8-51e2-a636-c7ffe2ed1375"
+				(path "/26736c46-8b40-5460-874f-03596d17270c/fbebb8e3-66b2-5aa7-ba3c-4936c50e8f80"
 					(reference "C801")
 					(unit 1)
@@
 		(instances
 			(project "mini-xt"
-				(path "/26736c46-8b40-5460-874f-03596d17270c/3898b474-78c8-51e2-a636-c7ffe2ed1375"
+				(path "/26736c46-8b40-5460-874f-03596d17270c/fbebb8e3-66b2-5aa7-ba3c-4936c50e8f80"
 					(reference "C802")
 					(unit 1)
@@
 		(instances
 			(project "mini-xt"
-				(path "/26736c46-8b40-5460-874f-03596d17270c/3898b474-78c8-51e2-a636-c7ffe2ed1375"
+				(path "/26736c46-8b40-5460-874f-03596d17270c/fbebb8e3-66b2-5aa7-ba3c-4936c50e8f80"
 					(reference "C803")
 					(unit 1)
@@
 		(instances
 			(project "mini-xt"
-				(path "/26736c46-8b40-5460-874f-03596d17270c/3898b474-78c8-51e2-a636-c7ffe2ed1375"
+				(path "/26736c46-8b40-5460-874f-03596d17270c/fbebb8e3-66b2-5aa7-ba3c-4936c50e8f80"
 					(reference "C804")
 					(unit 1)
@@
 		(instances
 			(project "mini-xt"
-				(path "/26736c46-8b40-5460-874f-03596d17270c/3898b474-78c8-51e2-a636-c7ffe2ed1375"
+				(path "/26736c46-8b40-5460-874f-03596d17270c/fbebb8e3-66b2-5aa7-ba3c-4936c50e8f80"
 					(reference "C805")
 					(unit 1)
@@
 		(instances
 			(project "mini-xt"
-				(path "/26736c46-8b40-5460-874f-03596d17270c/3898b474-78c8-51e2-a636-c7ffe2ed1375"
+				(path "/26736c46-8b40-5460-874f-03596d17270c/fbebb8e3-66b2-5aa7-ba3c-4936c50e8f80"
 					(reference "C806")
 					(unit 1)
@@
 		(instances
 			(project "mini-xt"
-				(path "/26736c46-8b40-5460-874f-03596d17270c/3898b474-78c8-51e2-a636-c7ffe2ed1375"
+				(path "/26736c46-8b40-5460-874f-03596d17270c/fbebb8e3-66b2-5aa7-ba3c-4936c50e8f80"
 					(reference "C807")
 					(unit 1)
