File: hardware/sheets/rtc.kicad_sch (KiCad schematic)
At the start: 14 parts, among them U1 DS12C887, U2 74HCT138, U3 74HC02, U4 74HCT08, U5 74HCT32, U6 74HCT04

Commit message: ERC cleanup: NC flags on unused pins, anchored interface labels
KiCad 10 ERC drops from 366 to 16 violations, all noise:

- NC flags on the 36 genuinely unused pins (cpu_core '138/'161 spares,
  Supervisor RP2040 unused GPIO, Core2350B GPIO44-47, rtc '138 spares).
- emit_interface anchors every hier label on a stub wire ending in a
  same-name local label -- connectivity unchanged (still by name;
  netlist spans verified), but nothing dangles.
- Interface honesty: cpu_core drops AEN/IOCHRDY from PINS (both live on
  bus_mcu; nothing here touched them), bus_mcu drops PRIV_COUNTER (the
  counter chain is on-sheet, CNT_* never crosses).
- Remaining 6 label_dangling are root IRQ9-13/15: single-sheet by
  design (soft-PIC pull-ups await future 16-bit sources); kept in PINS
  as the AT-style contract.

Co-Authored-By: Claude Fable 5 <noreply@anthropic.com>
Parts:
- removed U3: 74HC02, symbol mini-xt:74HCT02
- removed U6: 74HCT04, symbol mini-xt:74HCT04
- added C5: 100nF, symbol Device:C
- added U5: 74HCT32, symbol mini-xt:74HCT32
- U3: renamed from U5; value 74HCT32 -> 74HC02; symbol mini-xt:74HCT32 -> mini-xt:74HCT02; LCSC Part Num C5985 -> C5588
- U6: renamed from C5; value 100nF -> 74HCT04; symbol Device:C -> mini-xt:74HCT04; LCSC Part Num C14663 -> C672096
Connections:
- net +5V: now also U6.14 (VCC), C5.1, U5.14 (VCC); no longer U6.1
- net A0: now also U6.1 (P1)
- net A1: now also U3.2 (P2)
- net A2: now also U3.3 (P3)
- net A3: now also U3.5 (P5)
- net A7: now also U3.6 (P6)
- net A8: now also U3.8 (P8)
- net A9: now also U3.9 (P9)
- net GND: now also U3.11 (P11), U6.13 (P13), U6.7 (GND), C5.2, U5.10 (P10), U5.12 (P12), U5.13 (P13), U5.7 (GND), U5.9 (P9); no longer U3.10 (P10), U3.13 (P13), U3.9 (P9), U6.2
- net IRQ8: now also U6.10 (P10)
- net NA0: now also U6.2 (P2), U5.2 (P2), U5.5 (P5); no longer U3.2 (P2), U3.5 (P5)
- net NIOW: now also U6.4 (P4)
- net NRTCSEL: now also U6.6 (P6)
- net RESET_DRV: now also U6.9 (P9)
- net RTC_DS: now also U5.3 (P3); no longer U3.3 (P3)
- net RTC_IRQ_L: now also U6.11 (P11)
- net RTC_RST_L: now also U6.8 (P8)
- net RTC_RW: now also U5.6 (P6); no longer U3.6 (P6)
- net ZN1: now also U3.1 (P1)
- net ZN2: now also U3.4 (P4)
- net ZN3: now also U3.10 (P10)
- net ~{IOR}: now also U5.1 (P1); no longer U3.1 (P1)
- net ~{IOW}: now also U6.3 (P3), U5.4 (P4); no longer U3.4 (P4)
- net ~{RTC_SEL}: now also U6.5 (P5)
- no-connect marks 5 -> 12
Other:
- moved on the sheet: U3

Commit message: Parts: footprints for all components, close 6 LCSC map gaps, check_parts.py
- mxsch.py emits the Footprint property from component props (was
  hard-coded empty); parts.py entries now carry a verified KiCad
  footprint, applied at build time alongside the LCSC number.
- Map keys fixed to match placed values: USB_PROG, SS34, LED (PicoGUS),
  APS6404L, CB3T3257/45 -- every combo across all sheets + cards now
  resolves (130 combos, 455 netlist components, all with footprints).
- Package corrections from JLC DB re-check: RTL8019AS is QFP-100 14x20
  P0.65 (not TQFP); C2897411 female header is a 2x10 strip -- fine for
  Core2350B, Pico needs 2x 1x20 (noted in jlcpcb-sourcing.md).
- 10 mini-xt:* placeholder footprints mark parts whose land pattern is
  authored at layout from the EasyEDA data (CH224K, magnetics, RJ45,
  HDMI, CF socket, ISA slot, switches, Core2350B PGA).
- New tools/check_parts.py: fails on unmapped combos, missing fp
  fields, or footprints absent from the installed KiCad libs.

Co-Authored-By: Claude Fable 5 <noreply@anthropic.com>
Parts:
- C1, C2, C3, C4, C5, C6: footprint (none) -> Capacitor_SMD:C_0603_1608Metric
- C7: footprint (none) -> Capacitor_SMD:C_0805_2012Metric
- R1: footprint (none) -> Resistor_SMD:R_0603_1608Metric
- U1: footprint (none) -> Package_DIP:DIP-24_W15.24mm_Socket
- U2: footprint (none) -> Package_SO:SOIC-16_3.9x9.9mm_P1.27mm
- U3, U4, U5, U6: footprint (none) -> Package_SO:SOIC-14_3.9x8.7mm_P1.27mm
Changed lines of the file:
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@@
 			)
 		)
-		(property "Footprint" ""
+		(property "Footprint" "Package_DIP:DIP-24_W15.24mm_Socket"
 			(at 228.6 116.84 0)
 			(effects
@@
 			)
 		)
-		(property "Footprint" ""
+		(property "Footprint" "Resistor_SMD:R_0603_1608Metric"
 			(at 254 88.9 0)
 			(effects
@@
 			)
 		)
-		(property "Footprint" ""
+		(property "Footprint" "Package_SO:SOIC-16_3.9x9.9mm_P1.27mm"
 			(at 88.9 81.28 0)
 			(effects
@@
 			)
 		)
-		(property "Footprint" ""
+		(property "Footprint" "Package_SO:SOIC-14_3.9x8.7mm_P1.27mm"
 			(at 88.9 215.9 0)
 			(effects
@@
 			)
 		)
-		(property "Footprint" ""
+		(property "Footprint" "Package_SO:SOIC-14_3.9x8.7mm_P1.27mm"
 			(at 152.4 215.9 0)
 			(effects
@@
 			)
 		)
-		(property "Footprint" ""
+		(property "Footprint" "Package_SO:SOIC-14_3.9x8.7mm_P1.27mm"
 			(at 152.4 160.02 0)
 			(effects
@@
 			)
 		)
-		(property "Footprint" ""
+		(property "Footprint" "Package_SO:SOIC-14_3.9x8.7mm_P1.27mm"
 			(at 88.9 160.02 0)
 			(effects
@@
 			)
 		)
-		(property "Footprint" ""
+		(property "Footprint" "Capacitor_SMD:C_0603_1608Metric"
 			(at 228.6 175.26 0)
 			(effects
@@
 			)
 		)
-		(property "Footprint" ""
+		(property "Footprint" "Capacitor_SMD:C_0603_1608Metric"
 			(at 152.4 96.52 0)
 			(effects
@@
 			)
 		)
-		(property "Footprint" ""
+		(property "Footprint" "Capacitor_SMD:C_0603_1608Metric"
 			(at 88.9 254 0)
 			(effects
@@
 			)
 		)
-		(property "Footprint" ""
+		(property "Footprint" "Capacitor_SMD:C_0603_1608Metric"
 			(at 114.3 254 0)
 			(effects
@@
 			)
 		)
-		(property "Footprint" ""
+		(property "Footprint" "Capacitor_SMD:C_0603_1608Metric"
 			(at 139.7 254 0)
 			(effects
@@
 			)
 		)
-		(property "Footprint" ""
+		(property "Footprint" "Capacitor_SMD:C_0603_1608Metric"
 			(at 165.1 254 0)
 			(effects
@@
 			)
 		)
-		(property "Footprint" ""
+		(property "Footprint" "Capacitor_SMD:C_0805_2012Metric"
 			(at 190.5 254 0)
 			(effects

Commit message: Symbols+parts: IS62WV51216, TL16C550CPT, I2C RTC; 3.3V LVC/HC rebinds
New flat mini-xt: symbols (gensym.py), pins verified against
jlc_get_pinout + datasheet (PCF8563 caught a jlc_get_pinout numbering bug):
IS62WV51216 (512Kx16 SRAM, TSOP-44), TL16C550PT (TL16C550C UART, LQFP-48,
NO.PT numbering -- distinct from the old DIP-40 16550 symbol), PCF8563
(I2C RTC, SO-8).

parts.py: bind the three new parts (SRAM in stock at JLC; TL16C550CPT
sourced elsewhere like the V20, 0 JLC stock; PCF8563 + CR2032 holder on
Device:Battery_Cell); rebind the clock dividers to 74LVC74A/74LVC161
(check 7: HC/HCT both fail fmax margin at 3.3V/14.318MHz); add LVC-grade
binds for 5V-tolerant-input octal parts (74LVC573A/244A/574A/125A/245A)
and plain-HC binds for pure-3.3V-domain gates (74HC00/04/32/138) on the
existing HCT-body symbols; add 74LVC2G07 as a value override on the
pin-identical 74LVC2G06 body. Delete the now-dead AS6C4008 DIP-32 socket,
16550 PLCC-44 socket, and DS12C887 DIP-24 socket entries (replaced parts,
no longer sourced).

Sanity build (build.py) still passes: root + 13 sheets, exit 0. The three
deleted entries leave their still-unrewired sheets (cpu_core, com_port,
rtc) temporarily unmapped in check_parts.py until Tasks 4-9 rewire them --
expected transitional state, not a regression.

Co-Authored-By: Claude Fable 5 <noreply@anthropic.com>
Parts:
- U1: footprint Package_DIP:DIP-24_W15.24mm_Socket -> (none); LCSC Part Num C2684765 -> (none)
Changed lines of the file:
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@@
 			)
 		)
-		(property "Footprint" "Package_DIP:DIP-24_W15.24mm_Socket"
+		(property "Footprint" ""
 			(at 228.6 116.84 0)
 			(effects
-				(font
-					(size 1.27 1.27)
-				)
-				(hide yes)
-			)
-		)
-		(property "LCSC Part Num" "C2684765"
-			(at 228.6 116.84 0)
-			(effects
