File: hardware/sheets/supervisor.kicad_sch (KiCad schematic)
At the start: 33 parts, among them J2 USB_HOST, J3 POST_HEX, J4 CONSOLE, J5 SWD, J6 USB_PROG, SW1 BOOTSEL, SW2 PROG SEL, U1 RP2040, U2 W25Q128JVS, U3 USBLC6-2SC6, Y1 12MHz

Commit message: Design-review fixes: reset parking, IRQ8 off the header, analog cleanups
Netlist-wide review sweep. IRQ8 leaves the 60-pin ISA header (pin 15 is a
second GND return; the on-board RTC owns IRQ8 exclusively, so its push-pull
drive is now correct by construction). Bus MCU Hi-Z parking completed:
~CPURESET pulled low (V20 held in reset while the MCU is unprogrammed),
~DACK1/~REFRESH parked deasserted, DRQ1 idled low. Supervisor 12 MHz crystal
damping R actually in series now (was parallel-to-nothing), plus a second
USBLC6 so both prog-port SW2 positions are ESD-protected. Audio: 0.5x PG
summing (MCP6002 headroom), 100k LINE bleed, unit B parked as a follower --
and the SUM stub moved off pin 5's row, where wiring unit B would have
silently merged SUM into VREF. CH224K VDD fed through 1k per the WCH ref
design. VGA blue ladder rescaled 1k/510 -> 820/470 (was ~12% blue-deficient).
Spare CMOS gate inputs grounded uniformly (cpu_core/rtc/storage); UART_RXD
pulled up (SIN idles at mark with JP1 open); dead pins/parts dropped
(com_port CLK, parallel RESET_DRV, storage R3). Bus CLK fixed at 7.16 MHz
logged as a decision. New passives mapped to JLC basic parts in parts.py.

Co-Authored-By: Claude Fable 5 <noreply@anthropic.com>
Parts:
- added SW2: PROG SEL, symbol Switch:SW_Slide_DPDT
- U4: renamed from SW2; value PROG SEL -> USBLC6-2SC6; symbol Switch:SW_Slide_DPDT -> Power_Protection:USBLC6-2SC6; LCSC Part Num C431544 -> C2687116
Connections:
- net +3V3: now also U4.5 (VBUS)
- net GND: now also U4.2 (GND)
- net PGUS_USB_DM: now also SW2.6 (C); no longer U4.6 (C)
- net PGUS_USB_DP: now also SW2.3 (C); no longer U4.3 (C)
- net PROG_DM: now also U4.1 (I/O1), U4.6 (I/O1), SW2.5 (B); no longer U4.5 (B)
- net PROG_DP: now also U4.3 (I/O2), U4.4 (I/O2), SW2.2 (B); no longer U4.2 (B)
- net USB_DM_J: now also SW2.4 (A); no longer U4.4 (A)
- net USB_DP_J: now also SW2.1 (A); no longer U4.1 (A)
- net XOUT_R: no longer C2.1, Y1.2
- net XTAL_OUT: now also C2.1, Y1.2
Changed lines of the file:
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@@
 		)
 	)
-	(label "XOUT_R"
+	(label "XTAL_OUT"
 		(at 133.35 190.5 0)
 		(effects
@@
 		)
 	)
-	(label "XOUT_R"
+	(label "XTAL_OUT"
 		(at 137.16 196.85 90)
 		(effects
@@
 	(wire
 		(pts
+			(xy 58.42 66.04)
+			(xy 55.88 66.04)
+		)
+		(stroke
+			(width 0)
+			(type default)
+		)
+	)
+	(label "PROG_DM"
+		(at 55.88 66.04 180)
+		(effects
+			(font
+				(size 1.27 1.27)
+			)
+		)
+	)
+	(wire
+		(pts
+			(xy 68.58 66.04)
+			(xy 71.12 66.04)
+		)
+		(stroke
+			(width 0)
+			(type default)
+		)
+	)
+	(label "PROG_DM"
+		(at 71.12 66.04 0)
+		(effects
+			(font
+				(size 1.27 1.27)
+			)
+		)
+	)
+	(wire
+		(pts
+			(xy 58.42 68.58)
+			(xy 55.88 68.58)
+		)
+		(stroke
+			(width 0)
+			(type default)
+		)
+	)
+	(label "PROG_DP"
+		(at 55.88 68.58 180)
+		(effects
+			(font
+				(size 1.27 1.27)
+			)
+		)
+	)
+	(wire
+		(pts
+			(xy 68.58 68.58)
+			(xy 71.12 68.58)
+		)
+		(stroke
+			(width 0)
+			(type default)
+		)
+	)
+	(label "PROG_DP"
+		(at 71.12 68.58 0)
+		(effects
+			(font
+				(size 1.27 1.27)
+			)
+		)
+	)
+	(wire
+		(pts
+			(xy 63.5 60.96)
+			(xy 66.04 60.96)
+		)
+		(stroke
+			(width 0)
+			(type default)
+		)
+	)
+	(global_label "+3V3"
+		(shape input)
+		(at 66.04 60.96 0)
+		(effects
+			(font
+				(size 1.27 1.27)
+			)
+		)
+	)
+	(wire
+		(pts
+			(xy 63.5 73.66)
+			(xy 60.96 73.66)
+		)
+		(stroke
+			(width 0)
+			(type default)
+		)
+	)
+	(global_label "GND"
+		(shape input)
+		(at 60.96 73.66 180)
+		(effects
+			(font
+				(size 1.27 1.27)
+			)
+		)
+	)
+	(wire
+		(pts
 			(xy 132.08 43.18)
 			(xy 129.54 43.18)
@@
 					(unit 1)
 				)
+			)
+		)
+	)
+	(symbol
+		(lib_id "Power_Protection:USBLC6-2SC6")
+		(at 63.5 66.04 0)
+		(unit 1)
+		(exclude_from_sim no)
+		(in_bom yes)
+		(on_board yes)
+		(dnp no)
+		(fields_autoplaced yes)
+		(property "Reference" "U4"
+			(at 63.5 60.96 0)
+			(effects
+				(font
+					(size 1.27 1.27)
+				)
+			)
+		)
+		(property "Value" "USBLC6-2SC6"
+			(at 63.5 71.12 0)
+			(effects
+				(font
+					(size 1.27 1.27)
+				)
+			)
+		)
+		(property "Footprint" ""
+			(at 63.5 66.04 0)
+			(effects
+				(font
+					(size 1.27 1.27)
+				)
+				(hide yes)
+			)
+		)
+		(property "LCSC Part Num" "C2687116"
+			(at 63.5 66.04 0)
+			(effects
+				(font
+					(size 1.27 1.27)
+				)
+				(hide yes)
+			)
+		)
+		(pin "1"
+		)
+		(pin "3"
+		)
+		(pin "5"
+		)
+		(pin "2"
+		)
+		(pin "6"
+		)
+		(pin "4"
+		)
+		(instances
+			(project "mini-xt"
+				(path "/26736c46-8b40-5460-874f-03596d17270c/e314c42b-162a-53a5-8396-214d4f49fe96"
+					(reference "U304")
+					(unit 1)
+				)

Commit message: ERC cleanup: NC flags on unused pins, anchored interface labels
KiCad 10 ERC drops from 366 to 16 violations, all noise:

- NC flags on the 36 genuinely unused pins (cpu_core '138/'161 spares,
  Supervisor RP2040 unused GPIO, Core2350B GPIO44-47, rtc '138 spares).
- emit_interface anchors every hier label on a stub wire ending in a
  same-name local label -- connectivity unchanged (still by name;
  netlist spans verified), but nothing dangles.
- Interface honesty: cpu_core drops AEN/IOCHRDY from PINS (both live on
  bus_mcu; nothing here touched them), bus_mcu drops PRIV_COUNTER (the
  counter chain is on-sheet, CNT_* never crosses).
- Remaining 6 label_dangling are root IRQ9-13/15: single-sheet by
  design (soft-PIC pull-ups await future 16-bit sources); kept in PINS
  as the AT-style contract.

Co-Authored-By: Claude Fable 5 <noreply@anthropic.com>
Parts:
- removed C1: 30pF, symbol Device:C
- removed C14, C15, C4, C5: 100nF, symbol Device:C
- removed C6: 10uF, symbol Device:C
- removed R2: 27, symbol Device:R
- removed R5: 1k, symbol Device:R
- removed Y1: 12MHz, symbol Device:Crystal
- added C17, C18, C19, C20: 100nF, symbol Device:C
- added C2: 30pF, symbol Device:C
- added J2: USB_HOST, symbol Connector:USB_A
- added R4: 1k, symbol Device:R
- added SW1: BOOTSEL, symbol Switch:SW_Push
- added U3: USBLC6-2SC6, symbol Power_Protection:USBLC6-2SC6
- C1: renamed from R4; value 1k -> 30pF; symbol Device:R -> Device:C; LCSC Part Num C21190 -> C1658
- C4: renamed from SW1; value BOOTSEL -> 100nF; symbol Switch:SW_Push -> Device:C; LCSC Part Num C318884 -> C14663
- C6: renamed from C18; value 100nF -> 10uF; LCSC Part Num C14663 -> C15850
- R2: renamed from U3; value USBLC6-2SC6 -> 27; symbol Power_Protection:USBLC6-2SC6 -> Device:R; LCSC Part Num C2687116 -> C25190
- R5: renamed from J2; value USB_HOST -> 1k; symbol Connector:USB_A -> Device:R; LCSC Part Num C456015 -> C21190
- Y1: renamed from C2; value 30pF -> 12MHz; symbol Device:C -> Device:Crystal; LCSC Part Num C1658 -> C9002
- renumbered C19 to C14, C20 to C15, C17 to C5
Connections:
- net +3V3: now also C4.1, C17.1, C18.1, C19.1, C20.1; no longer C5.1, C6.1
- net GND: now also C1.2, C17.2, C18.2, C19.2, C2.2, C20.2, J2.4 (GND), J2.5 (Shield), SW1.2, U3.2 (GND); no longer R2.2 (GND), R5.4 (GND), R5.5 (Shield), Y1.2
- net QSPI_CS: now also R5.1
- net USB_DM_J: now also J2.2 (D-), U3.1 (I/O1), U3.6 (I/O1); no longer R2.1 (I/O1), R2.6 (I/O1), R5.2 (D-)
- net USB_DP: now also R2.1
- net USB_DP_J: now also R2.2, J2.3 (D+), U3.3 (I/O2), U3.4 (I/O2); no longer R2.3 (I/O2), R2.4 (I/O2), R5.3 (D+)
- net VBUS_KBD: now also J2.1 (VBUS), U3.5 (VBUS); no longer R2.5 (VBUS), R5.1 (VBUS)
- net VCORE: now also C5.1, C6.1
- net XOUT_R: now also R4.1; no longer C1.1
- net XTAL_IN: now also C1.1, Y1.1
- net XTAL_OUT: now also Y1.2, C2.1, R4.2; no longer C1.2, Y1.1
- net ~{USB_BOOT}: now also R5.2, SW1.1; no longer C4.1
- no-connect marks 14 -> 29
Other:
- moved on the sheet: C14, C15, C5, C6

Commit message: ERC power cleanup: single flag owner, flags on series-fed rails
Full-build ERC is now just the 6 expected IRQ9-13/15 label_dangling.

- Root's duplicate PWR_FLAGs removed from build.py: power.py #FLG1-3
  own +5V/+3V3/GND; the pair made flag-vs-flag pin_to_pin errors.
- PWR_FLAGs added on the local rails ERC can't see through a series
  part: VBUS_MCU / VBUS_VID (Schottky diode-OR), VBUS_KBD / HDMI_5V
  (polyfuse), CH224_VDD (1k per WCH ref), AVDD_PGUS / AGND_PGUS
  (ferrite beads).

Net membership verified unchanged: 821 nets, node-identical to HEAD.

Co-Authored-By: Claude Fable 5 <noreply@anthropic.com>
Changed lines of the file:
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@@
+	(wire
+		(pts
+			(xy 12.7 12.7)
+			(xy 12.7 10.16)
+		)
+		(stroke
+			(width 0)
+			(type default)
+		)
+	)
+	(label "VBUS_KBD"
+		(at 12.7 10.16 90)
+		(effects
+			(font
+				(size 1.27 1.27)
+			)
+		)
+	)
 	(wire
 		(pts
@@
 					(unit 1)
 				)
+			)
+		)
+	)
+	(symbol
+		(lib_id "power:PWR_FLAG")
+		(at 12.7 12.7 0)
+		(unit 1)
+		(exclude_from_sim no)
+		(in_bom yes)
+		(on_board yes)
+		(dnp no)
+		(fields_autoplaced yes)
+		(property "Reference" "#FLG1"
+			(at 12.7 7.62 0)
+			(effects
+				(font
+					(size 1.27 1.27)
+				)
+			)
+		)
+		(property "Value" "PWR_FLAG"
+			(at 12.7 17.78 0)
+			(effects
+				(font
+					(size 1.27 1.27)
+				)
+			)
+		)
+		(property "Footprint" ""
+			(at 12.7 12.7 0)
+			(effects
+				(font
+					(size 1.27 1.27)
+				)
+				(hide yes)
+			)
+		)
+		(pin "1"
+		)
+		(instances
+			(project "mini-xt"
+				(path "/26736c46-8b40-5460-874f-03596d17270c/c7457a0c-5b8c-5583-b336-de83d70434f7"
+					(reference "#FLG301")
+					(unit 1)
+				)
