File: hardware/sheets/network.kicad_sch (KiCad schematic)
At the start: 32 parts, among them J1 RJ45_LED, T1 13F-39MNL, U1 RTL8019AS, U2 AT93C46, U3 74HCT125, Y1 20MHz

Commit message: Network: 2kV line-side CT caps (isolation barrier, as upstream)
Parts:
- C7, C8: value 1nF -> 1nF/2kV; LCSC Part Num C1588 -> C9196
Changed lines of the file:
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@@
 			)
 		)
-		(property "Value" "1nF"
+		(property "Value" "1nF/2kV"
 			(at 342.9 68.58 0)
 			(effects
@@
 			)
 		)
-		(property "LCSC Part Num" "C1588"
+		(property "LCSC Part Num" "C9196"
 			(at 342.9 63.5 0)
 			(effects
@@
 			)
 		)
-		(property "Value" "1nF"
+		(property "Value" "1nF/2kV"
 			(at 342.9 144.78 0)
 			(effects
@@
 			)
 		)
-		(property "LCSC Part Num" "C1588"
+		(property "LCSC Part Num" "C9196"
 			(at 342.9 139.7 0)
 			(effects
