File: hardware/sheets/network.kicad_sch (KiCad schematic)
At the start: 32 parts, among them J1 RJ45_LED, T1 13F-39MNL, U1 RTL8019AS, U2 AT93C46, U3 74HCT125, Y1 20MHz

Commit message: Parts: footprints for all components, close 6 LCSC map gaps, check_parts.py
- mxsch.py emits the Footprint property from component props (was
  hard-coded empty); parts.py entries now carry a verified KiCad
  footprint, applied at build time alongside the LCSC number.
- Map keys fixed to match placed values: USB_PROG, SS34, LED (PicoGUS),
  APS6404L, CB3T3257/45 -- every combo across all sheets + cards now
  resolves (130 combos, 455 netlist components, all with footprints).
- Package corrections from JLC DB re-check: RTL8019AS is QFP-100 14x20
  P0.65 (not TQFP); C2897411 female header is a 2x10 strip -- fine for
  Core2350B, Pico needs 2x 1x20 (noted in jlcpcb-sourcing.md).
- 10 mini-xt:* placeholder footprints mark parts whose land pattern is
  authored at layout from the EasyEDA data (CH224K, magnetics, RJ45,
  HDMI, CF socket, ISA slot, switches, Core2350B PGA).
- New tools/check_parts.py: fails on unmapped combos, missing fp
  fields, or footprints absent from the installed KiCad libs.

Co-Authored-By: Claude Fable 5 <noreply@anthropic.com>
Parts:
- C1, C10, C11, C12, C13, C14, C2, C3, C4, C5, C6, C9: footprint (none) -> Capacitor_SMD:C_0603_1608Metric
- C15: footprint (none) -> Capacitor_SMD:C_0805_2012Metric
- C7, C8: footprint (none) -> Capacitor_SMD:C_1206_3216Metric
- FB1: footprint (none) -> Inductor_SMD:L_0603_1608Metric
- J1: footprint (none) -> mini-xt:RJ45_R-RJ45R08P-C000
- JP1: footprint (none) -> Connector_PinHeader_2.54mm:PinHeader_1x02_P2.54mm_Vertical
- R1, R2, R3, R4, R5, R6, R7, R8, R9: footprint (none) -> Resistor_SMD:R_0603_1608Metric
- T1: footprint (none) -> mini-xt:LAN_13F-39MNL
- U1: footprint (none) -> Package_QFP:PQFP-100_14x20mm_P0.65mm
- U2: footprint (none) -> Package_SO:SOIC-8_3.9x4.9mm_P1.27mm
- U3: footprint (none) -> Package_SO:SOIC-14_3.9x8.7mm_P1.27mm
- Y1: footprint (none) -> Crystal:Crystal_SMD_3225-4Pin_3.2x2.5mm
Changed lines of the file:
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@@
 			)
 		)
-		(property "Footprint" ""
+		(property "Footprint" "Package_QFP:PQFP-100_14x20mm_P0.65mm"
 			(at 152.4 152.4 0)
 			(effects
@@
 			)
 		)
-		(property "Footprint" ""
+		(property "Footprint" "Resistor_SMD:R_0603_1608Metric"
 			(at 228.6 25.4 0)
 			(effects
@@
 			)
 		)
-		(property "Footprint" ""
+		(property "Footprint" "Resistor_SMD:R_0603_1608Metric"
 			(at 241.3 25.4 0)
 			(effects
@@
 			)
 		)
-		(property "Footprint" ""
+		(property "Footprint" "Resistor_SMD:R_0603_1608Metric"
 			(at 254 25.4 0)
 			(effects
@@
 			)
 		)
-		(property "Footprint" ""
+		(property "Footprint" "Resistor_SMD:R_0603_1608Metric"
 			(at 152.4 266.7 0)
 			(effects
@@
 			)
 		)
-		(property "Footprint" ""
+		(property "Footprint" "Resistor_SMD:R_0603_1608Metric"
 			(at 304.8 152.4 0)
 			(effects
@@
 			)
 		)
-		(property "Footprint" ""
+		(property "Footprint" "Resistor_SMD:R_0603_1608Metric"
 			(at 342.9 190.5 0)
 			(effects
@@
 			)
 		)
-		(property "Footprint" ""
+		(property "Footprint" "Resistor_SMD:R_0603_1608Metric"
 			(at 355.6 190.5 0)
 			(effects
@@
 			)
 		)
-		(property "Footprint" ""
+		(property "Footprint" "Resistor_SMD:R_0603_1608Metric"
 			(at 368.3 254 0)
 			(effects
@@
 			)
 		)
-		(property "Footprint" ""
+		(property "Footprint" "Resistor_SMD:R_0603_1608Metric"
 			(at 381 254 0)
 			(effects
@@
 			)
 		)
-		(property "Footprint" ""
+		(property "Footprint" "Package_SO:SOIC-8_3.9x4.9mm_P1.27mm"
 			(at 254 152.4 0)
 			(effects
@@
 			)
 		)
-		(property "Footprint" ""
+		(property "Footprint" "Capacitor_SMD:C_0603_1608Metric"
 			(at 266.7 165.1 0)
 			(effects
@@
 			)
 		)
-		(property "Footprint" ""
+		(property "Footprint" "Package_SO:SOIC-14_3.9x8.7mm_P1.27mm"
 			(at 254 203.2 0)
 			(effects
@@
 			)
 		)
-		(property "Footprint" ""
+		(property "Footprint" "Capacitor_SMD:C_0603_1608Metric"
 			(at 266.7 215.9 0)
 			(effects
@@
 			)
 		)
-		(property "Footprint" ""
+		(property "Footprint" "Connector_PinHeader_2.54mm:PinHeader_1x02_P2.54mm_Vertical"
 			(at 254 254 0)
 			(effects
@@
 			)
 		)
-		(property "Footprint" ""
+		(property "Footprint" "Crystal:Crystal_SMD_3225-4Pin_3.2x2.5mm"
 			(at 152.4 254 0)
 			(effects
@@
 			)
 		)
-		(property "Footprint" ""
+		(property "Footprint" "Capacitor_SMD:C_0603_1608Metric"
 			(at 139.7 266.7 0)
 			(effects
@@
 			)
 		)
-		(property "Footprint" ""
+		(property "Footprint" "Capacitor_SMD:C_0603_1608Metric"
 			(at 165.1 266.7 0)
 			(effects
@@
 			)
 		)
-		(property "Footprint" ""
+		(property "Footprint" "mini-xt:LAN_13F-39MNL"
 			(at 330.2 101.6 0)
 			(effects
@@
 			)
 		)
-		(property "Footprint" ""
+		(property "Footprint" "Capacitor_SMD:C_0603_1608Metric"
 			(at 317.5 63.5 0)
 			(effects
@@
 			)
 		)
-		(property "Footprint" ""
+		(property "Footprint" "Capacitor_SMD:C_0603_1608Metric"
 			(at 317.5 139.7 0)
 			(effects
@@
 			)
 		)
-		(property "Footprint" ""
+		(property "Footprint" "Capacitor_SMD:C_1206_3216Metric"
 			(at 342.9 63.5 0)
 			(effects
@@
 			)
 		)
-		(property "Footprint" ""
+		(property "Footprint" "Capacitor_SMD:C_1206_3216Metric"
 			(at 342.9 139.7 0)
 			(effects
@@
 			)
 		)
-		(property "Footprint" ""
+		(property "Footprint" "mini-xt:RJ45_R-RJ45R08P-C000"
 			(at 381 101.6 0)
 			(effects
@@
 			)
 		)
-		(property "Footprint" ""
+		(property "Footprint" "Inductor_SMD:L_0603_1608Metric"
 			(at 381 152.4 0)
 			(effects
@@
 			)
 		)
-		(property "Footprint" ""
+		(property "Footprint" "Capacitor_SMD:C_0603_1608Metric"
 			(at 101.6 292.1 0)
 			(effects
@@
 			)
 		)
-		(property "Footprint" ""
+		(property "Footprint" "Capacitor_SMD:C_0603_1608Metric"
 			(at 129.54 292.1 0)
 			(effects
@@
 			)
 		)
-		(property "Footprint" ""
+		(property "Footprint" "Capacitor_SMD:C_0603_1608Metric"
 			(at 158.75 292.1 0)
 			(effects
@@
 			)
 		)
-		(property "Footprint" ""
+		(property "Footprint" "Capacitor_SMD:C_0603_1608Metric"
 			(at 187.96 292.1 0)
 			(effects
@@
 			)
 		)
-		(property "Footprint" ""
+		(property "Footprint" "Capacitor_SMD:C_0603_1608Metric"
 			(at 217.17 292.1 0)
 			(effects
@@
 			)
 		)
-		(property "Footprint" ""
+		(property "Footprint" "Capacitor_SMD:C_0603_1608Metric"
 			(at 246.38 292.1 0)
 			(effects
@@
 			)
 		)
-		(property "Footprint" ""
+		(property "Footprint" "Capacitor_SMD:C_0805_2012Metric"
 			(at 274.32 292.1 0)
 			(effects

Commit message: com/network/storage/parallel: 3.3V; TL16C550CPT soldered; LVC at external connectors
com_port: PLCC-44 16550 socket -> soldered TL16C550PT (LQFP-48) at +3V3,
rewired signal-for-signal from pins.py (RD/WR split renamed RD1/RD2/WR1/WR2,
INTR->INTRPT, GND->VSS, 8 new NC pins). Decode glue -> HC-grade, IRQ buffer
-> LVC125A, all +3V3. MAX3241 untouched (+5V, spec: already 3.3V-compatible).

network: only U3 (IRQ/AEN gate) moves, to LVC125A @ +3V3 -- RTL8019AS and
its EEPROM stay +5V (datasheet-verified 5V-only part, same treatment as
MAX3241), deviating from a literal reading of the brief's "power sweep"
instruction in favor of its own MAX3241 precedent.

storage: full brief table applied, all +3V3 except the CompactFlash
socket's own VCC power-feed pins (real CF-spec requirement, not a logic
signal).

parallel: brief's swap table only named 8 of 13 chips; traced the DB25
connector's actual net fan-out to fill the gap (U5, U9 also need
5V-tolerant inputs; U6/U7/U8/U12 are purely internal decode -> HC-grade).
U9 reuses the already-bound 74AHC14 value (no bare LVC04A entry exists).

Decisions logged in hardware/notes/questions-{com_port,network,storage,parallel}.md.

Co-Authored-By: Claude Fable 5 <noreply@anthropic.com>
Parts:
- U3: value 74HCT125 -> 74LVC125A; LCSC Part Num C5962 -> C6057
Connections:
- net +5V: no longer C2.1, R6.2, U3.10 (P10), U3.13 (P13), U3.14 (VCC)
- new net +3V3: C2.1, R6.2, U3.10 (P10), U3.13 (P13), U3.14 (VCC)
Changed lines of the file:
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@@
 		)
 	)
-	(global_label "+5V"
+	(global_label "+3V3"
 		(shape input)
 		(at 342.9 196.85 270)
@@
 		)
 	)
-	(global_label "+5V"
+	(global_label "+3V3"
 		(shape input)
 		(at 254 185.42 90)
@@
 		)
 	)
-	(global_label "+5V"
+	(global_label "+3V3"
 		(shape input)
 		(at 237.49 207.01 180)
@@
 		)
 	)
-	(global_label "+5V"
+	(global_label "+3V3"
 		(shape input)
 		(at 237.49 212.09 180)
@@
 		)
 	)
-	(global_label "+5V"
+	(global_label "+3V3"
 		(shape input)
 		(at 266.7 209.55 90)
@@
 			)
 		)
-		(property "Value" "74HCT125"
+		(property "Value" "74LVC125A"
 			(at 254 208.28 0)
 			(effects
@@
 			)
 		)
-		(property "LCSC Part Num" "C5962"
+		(property "LCSC Part Num" "C6057"
 			(at 254 203.2 0)
 			(effects

Commit message: network: isolate RTL8019AS 5V data bus behind gated LVC245 (review fix)
The RTL8019AS (U1) is a 5V-only part; its SD0-7 pins were wired directly to
the shared 3.3V bus D0-7, driving 5V TTL onto nets that reach the non-5V-
tolerant RP2040/PicoGUS during NIC I/O reads. Insert U4 (74LVC245A @ +3V3)
between U1's SD pins (now SD0_NIC..SD7_NIC) and D0-7: DIR = ~{IOR}, ~OE =
~{NIC_SEL}. The RTL8019AS decodes its 0x340 window internally and exposes no
select pin, so add U5 (74HC138) to reproduce that decode for the buffer
enable: ~Y5 low <=> A9.A8.~A7.A6.~A5.~AEN_CHIP, so U4 is Hi-Z on both sides
unless the NIC is the addressed target (no contention on other cards' reads;
full bus release when JP1 opens). Same idiom as storage.py U8.

Also model the gensym RTL8019AS symbol's IOCHRDY as open_collector and INT0
as tri_state (byte-stable regen; drops one ERC driver conflict).

Co-Authored-By: Claude Fable 5 <noreply@anthropic.com>
Parts:
- added C16, C17: 100nF, Capacitor_SMD:C_0603_1608Metric, symbol Device:C
- added R1: 10k, Resistor_SMD:R_0603_1608Metric, symbol Device:R
- added U5: 74HC138, Package_SO:SOIC-16_3.9x9.9mm_P1.27mm, symbol mini-xt:74HCT138
- U4: renamed from R1; value 10k -> 74LVC245A; footprint Resistor_SMD:R_0603_1608Metric -> Package_SO:TSSOP-20_4.4x6.5mm_P0.65mm; symbol Device:R -> mini-xt:74HCT245; LCSC Part Num C25804 -> C6082
Connections:
- net +3V3: now also U4.20 (VCC), C16.1, C17.1, U5.16 (VCC)
- net +5V: now also R1.2; no longer U4.2
- net A5: now also U5.5 (~{E1})
- net A6: now also U5.1 (A0)
- net A7: now also U5.2 (A1)
- net A8: now also U5.3 (A2)
- net A9: now also U5.6 (E2)
- net AEN_CHIP: now also U5.4 (~{E0})
- net D0: now also U4.2 (A0); no longer U1.36 (SD0)
- net D1: now also U4.3 (A1); no longer U1.37 (SD1)
- net D2: now also U4.4 (A2); no longer U1.38 (SD2)
- net D3: now also U4.5 (A3); no longer U1.39 (SD3)
- net D4: now also U4.6 (A4); no longer U1.40 (SD4)
- net D5: now also U4.7 (A5); no longer U1.41 (SD5)
- net D6: now also U4.8 (A6); no longer U1.42 (SD6)
- net D7: now also U4.9 (A7); no longer U1.43 (SD7)
- net GND: now also U4.10 (GND), C16.2, C17.2, U5.8 (GND)
- net JP_HI: now also R1.1; no longer U4.1
- net ~{IOR}: now also U4.1 (A->B)
- new net SD0_NIC: U1.36 (SD0), U4.18 (B0)
- new net SD1_NIC: U1.37 (SD1), U4.17 (B1)
- new net SD2_NIC: U1.38 (SD2), U4.16 (B2)
- new net SD3_NIC: U1.39 (SD3), U4.15 (B3)
- new net SD4_NIC: U1.40 (SD4), U4.14 (B4)
- new net SD5_NIC: U1.41 (SD5), U4.13 (B5)
- new net SD6_NIC: U1.42 (SD6), U4.12 (B6)
- new net SD7_NIC: U1.43 (SD7), U4.11 (B7)
- new net ~{NIC_SEL}: U4.19 (CE), U5.10 (~{Y5})
- no-connect marks 43 -> 50

Commit message: 3.3V redesign: final-review fix wave (6 findings)
Reviewer-verified fixes, all at the generator level + regenerated outputs:

1. (Critical) bus_mcu U17 '04 @+3V3 had the V20's 5V HLDA on its input ->
   value-override to 74LVC04A (5V-tolerant input; parts.py binds C282341).
2. network R7 (AEN_CHIP park) +5V -> +3V3: it also feeds U5's '138 @+3V3;
   RTL8019AS AEN is 5V-TTL so 3.3V still reads high.
3. sidecar buf244(): tie unused '244 A inputs to GND, no_connect the Y
   outputs (U1105: 6 spare, U1108: 7) -- no floating always-enabled inputs.
4. MAX3241s (both com_port instances) +5V -> +3V3; charge-pump caps to the
   datasheet 3.0-3.6V column (all 0.1uF). Removes the 5V-R*OUT-into-3.3V-UART
   receiver path; com_port now has no +5V rail.
5. V20 READY/HOLD re-buffered through cpu_core U13's 3 spare '04 gates (zero
   package cost). READY = 2 gates (non-inverting), single-driver (no fold).
   HOLD = 1 inverting gate -> FIRMWARE MUST DRIVE HOLD ACTIVE-LOW at GPIO25
   (mxbus HOLD name intact). U13 nudged to clear a stub collision with U12.
6. Docs census + staleness: rewrote the 5V census to post-fix reality across
   CLAUDE.md, spec, design doc, README, irq-io-map (IRQ8 soft-PIC/undriven),
   parts.py header notes.

Build exit 0; check_parts 0 problems; all five sheets validate with zero
structural violations. Netlist evidence in questions-*.md.

Co-Authored-By: Claude Fable 5 <noreply@anthropic.com>
Connections:
- net +3V3: now also R7.2
- net +5V: no longer R7.2
Changed lines of the file:
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@@
 		)
 	)
-	(global_label "+5V"
+	(global_label "+3V3"
 		(shape input)
 		(at 355.6 196.85 270)
