File: hardware/sheets/cpu_core.kicad_sch (KiCad schematic)
At the start: 37 parts, among them U1 V20, U10 74HCT32, U11 74LVC125A, U12 74HC157, U13 74HCT04, U14 TCM809, U15 74LVC125A, U2 74LVC573A, U3 74LVC573A, U4 74LVC573A, U5 74LVC245A, U6 74HC138, U7 74HC00, U8 74LVC74A, U9 74LVC161

Commit message: Decoupling audit: drop video's 2 orphan caps, add 5 missing ones
Audit of every bypass cap against the ICs it decouples found one stale
remnant: video kept 6 3V3_VID caps for what are now 4 shifters (C6/C7
belonged to the deleted U6/U7). Removed them. All other sheets tally
one-per-IC.

Under-provisioned spots filled in the same pass: cpu_core C28 gives the
third surviving 5V part its own 100nF (V20/U10/U13 now 1 each), and
sidecar C8-C11 bring the port buffers to one cap per IC (U1-U4, U6-U9).

ERC 0/0; netlist verified (C128 on +5V, C1008-C1011 on +3V3).

Co-Authored-By: Claude Fable 5 <noreply@anthropic.com>
Parts:
- added C27: 10uF, Capacitor_SMD:C_0805_2012Metric, symbol Device:C
- C26: renamed from C27; value 10uF -> 100nF; footprint Capacitor_SMD:C_0805_2012Metric -> Capacitor_SMD:C_0603_1608Metric; LCSC Part Num C15850 -> C14663
- renumbered C26 to C28
Connections:
- net +3V3: now also C26.1; no longer C28.1
- net +5V: now also C28.1, C27.1; no longer C26.1
- net GND: now also C27.2
Other:
- moved on the sheet: C26, C28
Changed lines of the file:
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@@
+	(wire
+		(pts
+			(xy 359.41 266.7)
+			(xy 359.41 264.16)
+		)
+		(stroke
+			(width 0)
+			(type default)
+		)
+	)
+	(global_label "+5V"
+		(shape input)
+		(at 359.41 264.16 90)
+		(effects
+			(font
+				(size 1.27 1.27)
+			)
+		)
+	)
+	(wire
+		(pts
+			(xy 359.41 274.32)
+			(xy 359.41 276.86)
+		)
+		(stroke
+			(width 0)
+			(type default)
+		)
+	)
+	(global_label "GND"
+		(shape input)
+		(at 359.41 276.86 270)
+		(effects
+			(font
+				(size 1.27 1.27)
+			)
+		)
+	)
 	(wire
 		(pts
@@
 					(unit 1)
 				)
+			)
+		)
+	)
+	(symbol
+		(lib_id "Device:C")
+		(at 359.41 270.51 0)
+		(unit 1)
+		(exclude_from_sim no)
+		(in_bom yes)
+		(on_board yes)
+		(dnp no)
+		(fields_autoplaced yes)
+		(property "Reference" "C28"
+			(at 359.41 265.43 0)
+			(effects
+				(font
+					(size 1.27 1.27)
+				)
+			)
+		)
+		(property "Value" "100nF"
+			(at 359.41 275.59 0)
+			(effects
+				(font
+					(size 1.27 1.27)
+				)
+			)
+		)
+		(property "Footprint" "Capacitor_SMD:C_0603_1608Metric"
+			(at 359.41 270.51 0)
+			(effects
+				(font
+					(size 1.27 1.27)
+				)
+				(hide yes)
+			)
+		)
+		(property "LCSC Part Num" "C14663"
+			(at 359.41 270.51 0)
+			(effects
+				(font
+					(size 1.27 1.27)
+				)
+				(hide yes)
+			)
+		)
+		(pin "1"
+		)
+		(pin "2"
+		)
+		(instances
+			(project "mini-xt"
+				(path "/26736c46-8b40-5460-874f-03596d17270c/36a61212-e622-5b01-8e81-aba0acbc9887"
+					(reference "C128")
+					(unit 1)
+				)
