File: hardware/sheets/picogus.kicad_sch (KiCad schematic)
At the start: 58 parts, among them J1 DMA_JP, J5 SWD, SW1 BOOTSEL, U1 RP2040, U10 74LVC2G06, U11 APS6404L, U12 PCM5102A, U2 W25Q128JVS, U3 AMS1117-3.3, U4 CB3T3257, U5 CB3T3257, U7 74AHC14, U8 74HC00, U9 74HC00, Y1 12MHz

Commit message: Expansion port: 50-pin header, port DMA channel, dev cards deleted
Two waves of the 2026-07-14/15 expansion-port rework (the first was
uncommitted): the IRQ-scan collapse to one '165 + '32 OR rank with
ISA-card DMA removed outright, then the port redesign that brings one
DMA channel back:

- isa_conn: 60-pin (2x30, PicoGUS-standard layout) -> 50-pin (2x25,
  project-private pinout; 50-way IDC is far easier to source). OSC and
  ~REFRESH dropped to fit (no on-board consumer / no DRAM refresh; the
  planned ISA backplane board re-creates both for period cards).
- Port DMA: EXT_DRQ rides the sidecar inbound '244 + U12 '165 spare D6
  lane (zero GPIO); ~EXT_DACK = GPIO47 (freed by ~REFRESH) out through
  the strobe '244. Separate nets from the internal PicoGUS pair, so a
  port card never sees the on-board acknowledge.
- DRQ1/~DACK1 renamed DRQ/~DACK (ch2/3 long retired); DRQ2/3 +
  ~DACK2/3 removed from the mxbus contract.
- card_video + card_isatest deleted (sheets, hardware/cards/,
  build_cards()); superseded by the backplane plan. History has them.
- Connector parts: IDE header -> shrouded 2x20 IDC box (C9138, keypin
  20 NC'd); expansion port -> 90-degree 2x25 female socket (C21262364);
  addr_decode's five disable jumpers folded into ONE fixed 2x5 block
  JP1 (C492422), positions JP1.1-JP1.5 = COM1/COM2/LPT/IDE/VID.

ERC 0/0, check_parts 0 problems; docs/notes updated throughout.

Co-Authored-By: Claude Fable 5 <noreply@anthropic.com>
Parts:
- removed J1: DMA_JP, Connector_PinHeader_2.54mm:PinHeader_2x04_P2.54mm_Vertical, symbol Connector_Generic:Conn_02x04_Odd_Even
- removed R9: 15k, Resistor_SMD:R_0603_1608Metric, symbol Device:R
Connections:
- net DACK renamed ~{DACK}
Other:
- note added: "DMA hardwired to ch1 timing (DRQ/DACK; jumper deleted -- Bus MCU services ch1 ONLY). IRQ hardwired to IRQ5 (the free line, sole driver); pgusinit sets the firmware to match."
- note removed: "DMA jumpers: one DRQ/DACK pair -- our Bus MCU services DMA ch1 ONLY, so jumper DRQ1/DACK1. IRQ hardwired to IRQ5 (the free line, sole driver); pgusinit sets the firmware to match."

Commit message: Sourcing: 10k pulls to 0805 basic C17414, DB25 to socket footprint
parts.py swaps propagate through the regenerated sheets/netlist; LCSC
price cache and jlcpcb-sourcing notes updated to match.

Co-Authored-By: Claude Fable 5 <noreply@anthropic.com>
Claude-Session: https://claude.ai/code/session_01Y7zRS7ikVENkjZFFBcegCP
Parts:
- R6, R7: footprint Resistor_SMD:R_0603_1608Metric -> Resistor_SMD:R_0805_2012Metric; LCSC Part Num C25804 -> C17414
Changed lines of the file:
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@@
 			)
 		)
-		(property "Footprint" "Resistor_SMD:R_0603_1608Metric"
+		(property "Footprint" "Resistor_SMD:R_0805_2012Metric"
 			(at 228.6 25.4 0)
 			(effects
@@
 			)
 		)
-		(property "LCSC Part Num" "C25804"
+		(property "LCSC Part Num" "C17414"
 			(at 228.6 25.4 0)
 			(effects
@@
 			)
 		)
-		(property "Footprint" "Resistor_SMD:R_0603_1608Metric"
+		(property "Footprint" "Resistor_SMD:R_0805_2012Metric"
 			(at 241.3 25.4 0)
 			(effects
@@
 			)
 		)
-		(property "LCSC Part Num" "C25804"
+		(property "LCSC Part Num" "C17414"
 			(at 241.3 25.4 0)
 			(effects
