File: hardware/sheets/storage.kicad_sch (KiCad schematic)
At the start: 34 parts, among them J1 Conn_02x20_Odd_Even, J2 Conn_02x25_Odd_Even, Q1 2N7002, U1 74HCT04, U10 74HCT573, U11 74HCT138, U2 74HCT08, U3 74HCT08, U4 74HCT32, U5 74HCT125, U6 74HCT138, U7 74HCT138, U8 74HCT245, U9 74HCT573

Commit message: Design-review fixes: reset parking, IRQ8 off the header, analog cleanups
Netlist-wide review sweep. IRQ8 leaves the 60-pin ISA header (pin 15 is a
second GND return; the on-board RTC owns IRQ8 exclusively, so its push-pull
drive is now correct by construction). Bus MCU Hi-Z parking completed:
~CPURESET pulled low (V20 held in reset while the MCU is unprogrammed),
~DACK1/~REFRESH parked deasserted, DRQ1 idled low. Supervisor 12 MHz crystal
damping R actually in series now (was parallel-to-nothing), plus a second
USBLC6 so both prog-port SW2 positions are ESD-protected. Audio: 0.5x PG
summing (MCP6002 headroom), 100k LINE bleed, unit B parked as a follower --
and the SUM stub moved off pin 5's row, where wiring unit B would have
silently merged SUM into VREF. CH224K VDD fed through 1k per the WCH ref
design. VGA blue ladder rescaled 1k/510 -> 820/470 (was ~12% blue-deficient).
Spare CMOS gate inputs grounded uniformly (cpu_core/rtc/storage); UART_RXD
pulled up (SIN idles at mark with JP1 open); dead pins/parts dropped
(com_port CLK, parallel RESET_DRV, storage R3). Bus CLK fixed at 7.16 MHz
logged as a decision. New passives mapped to JLC basic parts in parts.py.

Co-Authored-By: Claude Fable 5 <noreply@anthropic.com>
Parts:
- removed R3: 10k, symbol Device:R
Connections:
- net GND: now also U3.10 (P10), U3.12 (P12), U3.13 (P13), U3.9 (P9)
- no-connect marks 38 -> 36
Other:
- note added: "Populate ONE of J1 (IDE) / J2 (CF): both CSELs are grounded, so both devices ID as master on the shared cable."

Commit message: Hardwire storage IRQ14 and PicoGUS IRQ5; drop their IRQ jumpers
- Storage JP3 deleted: INTRQ -> '125 -> IRQ14 directly (the soft PIC
  is AT-style anyway). Poll vs interrupt is an XTIDE UB per-controller
  config choice, safe with the line wired either way -- the tri-state
  driver is silent unless the drive asserts INTRQ. ~{IRQ5_OE} renamed
  ~{IRQ_OE} to match.
- PicoGUS IRQ jumper row deleted: the shifter output drives IRQ5
  directly -- the free line and now its sole driver; every personality
  works on IRQ5 and pgusinit sets the firmware to match, so the 5-row
  jumper bought nothing. J1 shrinks 2x9 -> 2x4 (DMA pairs only, ch1 is
  the only MCU-serviced channel); parts.py header entry follows.
- IRQ5 contention is now zero: the sidecar header is the only other
  possible driver.

Full-build ERC: 0 violations; cards build clean.

Co-Authored-By: Claude Fable 5 <noreply@anthropic.com>
Parts:
- removed C11: 100nF, symbol Device:C
- removed C12: 10uF, symbol Device:C
- removed JP3: IRQ 14/5, symbol Connector_Generic:Conn_01x03
- added C1: 100nF, symbol Device:C
- added R5: 10k, symbol Device:R
- C12: renamed from C10; value 100nF -> 10uF; LCSC Part Num C14663 -> C15850
- C2: renamed from R5; value 10k -> 100nF; symbol Device:R -> Device:C; LCSC Part Num C25804 -> C14663
- renumbered C8 to C10, C9 to C11, C1 to C3, C2 to C4, C3 to C5, C4 to C6, C5 to C7, C6 to C8, C7 to C9
Connections:
- net STOR_IRQ is gone; now on net IRQ14: U5.3 (P3)
- net +5V: now also C1.1, R5.1
- net GND: now also C2.2, C1.2
- net ~{STOR_EN}: now also R5.2; no longer C2.2
- net ~{IRQ5_OE} renamed ~{IRQ_OE}
Other:
- note added: "JP1 base 0x300/0x320 (XTIDE UB); JP2 open = card disabled; IRQ14 hardwired (poll vs IRQ = XTIDE UB config)."
- note removed: "JP1 base 0x300/0x320 (XTIDE UB); JP2 open = card disabled; JP3 1-2=IRQ14(default)/2-3=IRQ5/open=polled."
- moved on the sheet: C10, C11, C12, C3, C4, C5, C6, C7, C8, C9
Changed lines of the file:
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@@
 		)
 	)
-	(label "IRQ5"
-		(at 22.86 81.28 180)
-		(effects
-			(font
-				(size 1.27 1.27)
-			)
-			(justify right)
-		)
-	)
-	(hierarchical_label "IRQ5"
-		(shape output)
-		(at 25.4 81.28 0)
-		(effects
-			(font
-				(size 1.27 1.27)
-			)
-		)
-	)
-	(wire
-		(pts
-			(xy 22.86 83.82)
-			(xy 25.4 83.82)
-		)
-		(stroke
-			(width 0)
-			(type default)
-		)
-	)
 	(label "IRQ14"
-		(at 22.86 83.82 180)
+		(at 22.86 81.28 180)
 		(effects
 			(font
@@
 	(hierarchical_label "IRQ14"
 		(shape output)
-		(at 25.4 83.82 0)
+		(at 25.4 81.28 0)
 		(effects
 			(font
@@
 		)
 	)
-	(label "~{IRQ5_OE}"
+	(label "~{IRQ_OE}"
 		(at 21.59 250.19 180)
 		(effects
@@
 		)
 	)
-	(label "STOR_IRQ"
+	(label "IRQ14"
 		(at 54.61 247.65 0)
 		(effects
@@
 		)
 	)
-	(label "~{IRQ5_OE}"
+	(label "~{IRQ_OE}"
 		(at 78.74 248.92 90)
 		(effects
@@
 		)
 	)
-	(label "~{IRQ5_OE}"
+	(label "~{IRQ_OE}"
 		(at 91.44 250.19 270)
 		(effects
@@
 	(wire
 		(pts
-			(xy 299.72 22.86)
-			(xy 302.26 22.86)
-		)
-		(stroke
-			(width 0)
-			(type default)
-		)
-	)
-	(label "IRQ14"
-		(at 302.26 22.86 0)
-		(effects
-			(font
-				(size 1.27 1.27)
-			)
-		)
-	)
-	(wire
-		(pts
-			(xy 299.72 25.4)
-			(xy 302.26 25.4)
-		)
-		(stroke
-			(width 0)
-			(type default)
-		)
-	)
-	(label "STOR_IRQ"
-		(at 302.26 25.4 0)
-		(effects
-			(font
-				(size 1.27 1.27)
-			)
-		)
-	)
-	(wire
-		(pts
-			(xy 299.72 27.94)
-			(xy 302.26 27.94)
-		)
-		(stroke
-			(width 0)
-			(type default)
-		)
-	)
-	(label "IRQ5"
-		(at 302.26 27.94 0)
-		(effects
-			(font
-				(size 1.27 1.27)
-			)
-		)
-	)
-	(wire
-		(pts
 			(xy 320.04 21.59)
 			(xy 320.04 19.05)
@@
 		)
 	)
-	(text "JP1 base 0x300/0x320 (XTIDE UB); JP2 open = card disabled; JP3 1-2=IRQ14(default)/2-3=IRQ5/open=polled."
+	(text "JP1 base 0x300/0x320 (XTIDE UB); JP2 open = card disabled; IRQ14 hardwired (poll vs IRQ = XTIDE UB config)."
 		(at 266.7 17.78 0)
 		(effects
@@
 					(unit 1)
 				)
-			)
-		)
-	)
-	(symbol
-		(lib_id "Connector_Generic:Conn_01x03")
-		(at 304.8 25.4 0)
-		(unit 1)
-		(exclude_from_sim no)
-		(in_bom yes)
-		(on_board yes)
-		(dnp no)
-		(fields_autoplaced yes)
-		(property "Reference" "JP3"
-			(at 304.8 20.32 0)
-			(effects
-				(font
-					(size 1.27 1.27)
-				)
-			)
-		)
-		(property "Value" "IRQ 14/5"
-			(at 304.8 30.48 0)
-			(effects
-				(font
-					(size 1.27 1.27)
-				)
-			)
-		)
-		(property "Footprint" ""
-			(at 304.8 25.4 0)
-			(effects
-				(font
-					(size 1.27 1.27)
-				)
-				(hide yes)
-			)
-		)
-		(property "LCSC Part Num" "C2337"
-			(at 304.8 25.4 0)
-			(effects
-				(font
-					(size 1.27 1.27)
-				)
-				(hide yes)
-			)
-		)
-		(pin "1"
-		)
-		(pin "2"
-		)
-		(pin "3"
-		)
-		(instances
-			(project "mini-xt"
-				(path "/26736c46-8b40-5460-874f-03596d17270c/07112233-9dc6-58fa-9d50-2b89ae78e000"
-					(reference "JP1003")
-					(unit 1)
-				)

Commit message: Parts: footprints for all components, close 6 LCSC map gaps, check_parts.py
- mxsch.py emits the Footprint property from component props (was
  hard-coded empty); parts.py entries now carry a verified KiCad
  footprint, applied at build time alongside the LCSC number.
- Map keys fixed to match placed values: USB_PROG, SS34, LED (PicoGUS),
  APS6404L, CB3T3257/45 -- every combo across all sheets + cards now
  resolves (130 combos, 455 netlist components, all with footprints).
- Package corrections from JLC DB re-check: RTL8019AS is QFP-100 14x20
  P0.65 (not TQFP); C2897411 female header is a 2x10 strip -- fine for
  Core2350B, Pico needs 2x 1x20 (noted in jlcpcb-sourcing.md).
- 10 mini-xt:* placeholder footprints mark parts whose land pattern is
  authored at layout from the EasyEDA data (CH224K, magnetics, RJ45,
  HDMI, CF socket, ISA slot, switches, Core2350B PGA).
- New tools/check_parts.py: fails on unmapped combos, missing fp
  fields, or footprints absent from the installed KiCad libs.

Co-Authored-By: Claude Fable 5 <noreply@anthropic.com>
Parts:
- C1, C10, C11, C2, C3, C4, C5, C6, C7, C8, C9: footprint (none) -> Capacitor_SMD:C_0603_1608Metric
- C12: footprint (none) -> Capacitor_SMD:C_0805_2012Metric
- J1: footprint (none) -> Connector_PinHeader_2.54mm:PinHeader_2x20_P2.54mm_Vertical
- J2: footprint (none) -> mini-xt:CF_HYCW01-CF50-395B
- JP1: footprint (none) -> Connector_PinHeader_2.54mm:PinHeader_1x03_P2.54mm_Vertical
- JP2: footprint (none) -> Connector_PinHeader_2.54mm:PinHeader_1x02_P2.54mm_Vertical
- Q1: footprint (none) -> Package_TO_SOT_SMD:SOT-23
- R1, R2, R4, R5: footprint (none) -> Resistor_SMD:R_0603_1608Metric
- U1, U2, U3, U4, U5: footprint (none) -> Package_SO:SOIC-14_3.9x8.7mm_P1.27mm
- U10, U8, U9: footprint (none) -> Package_SO:SOIC-20W_7.5x12.8mm_P1.27mm
- U11, U6, U7: footprint (none) -> Package_SO:SOIC-16_3.9x9.9mm_P1.27mm
Changed lines of the file:
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@@
 			)
 		)
-		(property "Footprint" ""
+		(property "Footprint" "Package_SO:SOIC-14_3.9x8.7mm_P1.27mm"
 			(at 38.1 76.2 0)
 			(effects
@@
 			)
 		)
-		(property "Footprint" ""
+		(property "Footprint" "Package_SO:SOIC-14_3.9x8.7mm_P1.27mm"
 			(at 38.1 142.24 0)
 			(effects
@@
 			)
 		)
-		(property "Footprint" ""
+		(property "Footprint" "Package_SO:SOIC-14_3.9x8.7mm_P1.27mm"
 			(at 38.1 205.74 0)
 			(effects
@@
 			)
 		)
-		(property "Footprint" ""
+		(property "Footprint" "Package_SO:SOIC-14_3.9x8.7mm_P1.27mm"
 			(at 114.3 210.82 0)
 			(effects
@@
 			)
 		)
-		(property "Footprint" ""
+		(property "Footprint" "Package_SO:SOIC-14_3.9x8.7mm_P1.27mm"
 			(at 38.1 256.54 0)
 			(effects
@@
 			)
 		)
-		(property "Footprint" ""
+		(property "Footprint" "Package_TO_SOT_SMD:SOT-23"
 			(at 76.2 256.54 0)
 			(effects
@@
 			)
 		)
-		(property "Footprint" ""
+		(property "Footprint" "Package_SO:SOIC-16_3.9x9.9mm_P1.27mm"
 			(at 114.3 63.5 0)
 			(effects
@@
 			)
 		)
-		(property "Footprint" ""
+		(property "Footprint" "Package_SO:SOIC-16_3.9x9.9mm_P1.27mm"
 			(at 114.3 142.24 0)
 			(effects
@@
 			)
 		)
-		(property "Footprint" ""
+		(property "Footprint" "Package_SO:SOIC-16_3.9x9.9mm_P1.27mm"
 			(at 152.4 63.5 0)
 			(effects
@@
 			)
 		)
-		(property "Footprint" ""
+		(property "Footprint" "Package_SO:SOIC-20W_7.5x12.8mm_P1.27mm"
 			(at 190.5 63.5 0)
 			(effects
@@
 			)
 		)
-		(property "Footprint" ""
+		(property "Footprint" "Package_SO:SOIC-20W_7.5x12.8mm_P1.27mm"
 			(at 190.5 142.24 0)
 			(effects
@@
 			)
 		)
-		(property "Footprint" ""
+		(property "Footprint" "Package_SO:SOIC-20W_7.5x12.8mm_P1.27mm"
 			(at 190.5 215.9 0)
 			(effects
@@
 			)
 		)
-		(property "Footprint" ""
+		(property "Footprint" "Connector_PinHeader_2.54mm:PinHeader_2x20_P2.54mm_Vertical"
 			(at 292.1 127 0)
 			(effects
@@
 			)
 		)
-		(property "Footprint" ""
+		(property "Footprint" "mini-xt:CF_HYCW01-CF50-395B"
 			(at 368.3 127 0)
 			(effects
@@
 			)
 		)
-		(property "Footprint" ""
+		(property "Footprint" "Resistor_SMD:R_0603_1608Metric"
 			(at 228.6 25.4 0)
 			(effects
@@
 			)
 		)
-		(property "Footprint" ""
+		(property "Footprint" "Resistor_SMD:R_0603_1608Metric"
 			(at 243.84 25.4 0)
 			(effects
@@
 			)
 		)
-		(property "Footprint" ""
+		(property "Footprint" "Resistor_SMD:R_0603_1608Metric"
 			(at 91.44 243.84 0)
 			(effects
@@
 			)
 		)
-		(property "Footprint" ""
+		(property "Footprint" "Connector_PinHeader_2.54mm:PinHeader_1x03_P2.54mm_Vertical"
 			(at 274.32 25.4 0)
 			(effects
@@
 			)
 		)
-		(property "Footprint" ""
+		(property "Footprint" "Connector_PinHeader_2.54mm:PinHeader_1x02_P2.54mm_Vertical"
 			(at 289.56 25.4 0)
 			(effects
@@
 			)
 		)
-		(property "Footprint" ""
+		(property "Footprint" "Resistor_SMD:R_0603_1608Metric"
 			(at 320.04 25.4 0)
 			(effects
@@
 			)
 		)
-		(property "Footprint" ""
+		(property "Footprint" "Capacitor_SMD:C_0603_1608Metric"
 			(at 30.48 276.86 0)
 			(effects
@@
 			)
 		)
-		(property "Footprint" ""
+		(property "Footprint" "Capacitor_SMD:C_0603_1608Metric"
 			(at 49.53 276.86 0)
 			(effects
@@
 			)
 		)
-		(property "Footprint" ""
+		(property "Footprint" "Capacitor_SMD:C_0603_1608Metric"
 			(at 69.85 276.86 0)
 			(effects
@@
 			)
 		)
-		(property "Footprint" ""
+		(property "Footprint" "Capacitor_SMD:C_0603_1608Metric"
 			(at 90.17 276.86 0)
 			(effects
@@
 			)
 		)
-		(property "Footprint" ""
+		(property "Footprint" "Capacitor_SMD:C_0603_1608Metric"
 			(at 110.49 276.86 0)
 			(effects
@@
 			)
 		)
-		(property "Footprint" ""
+		(property "Footprint" "Capacitor_SMD:C_0603_1608Metric"
 			(at 129.54 276.86 0)
 			(effects
@@
 			)
 		)
-		(property "Footprint" ""
+		(property "Footprint" "Capacitor_SMD:C_0603_1608Metric"
 			(at 149.86 276.86 0)
 			(effects
@@
 			)
 		)
-		(property "Footprint" ""
+		(property "Footprint" "Capacitor_SMD:C_0603_1608Metric"
 			(at 170.18 276.86 0)
 			(effects
@@
 			)
 		)
-		(property "Footprint" ""
+		(property "Footprint" "Capacitor_SMD:C_0603_1608Metric"
 			(at 190.5 276.86 0)
 			(effects
@@
 			)
 		)
-		(property "Footprint" ""
+		(property "Footprint" "Capacitor_SMD:C_0603_1608Metric"
 			(at 209.55 276.86 0)
 			(effects
@@
 			)
 		)
-		(property "Footprint" ""
+		(property "Footprint" "Capacitor_SMD:C_0603_1608Metric"
 			(at 229.87 276.86 0)
 			(effects
@@
 			)
 		)
-		(property "Footprint" ""
+		(property "Footprint" "Capacitor_SMD:C_0805_2012Metric"
 			(at 256.54 276.86 0)
 			(effects
