File: hardware/sheets/storage.kicad_sch (KiCad schematic)
At the start: 25 parts, among them J1 Conn_02x20_Odd_Even, J2 Conn_02x25_Odd_Even, Q1 2N7002, U1 74HC04, U10 74LVC573A, U11 74HC138, U3 74HC08, U4 74HC32, U6 74HC138, U7 74HC138, U8 74LVC245A, U9 74LVC573A

Commit message: Passives: basic-library audit + 4x resistor-array pull consolidation
Audit: every discrete R/C value was already JLC basic except the ferrite
beads -- swapped to basic Murata BLM18PG121SN1D (C14709, 120R@100MHz,
same family/role). The 100uF electrolytic and buck inductor stay
extended (zero fee-free parts exist in those subcategories). Pruned the
orphaned 5V-era 47nF/330nF MAX3241 cap entries.

Pull consolidation: 65 discrete 10k/4.7k rail pulls across 8 sheets
collapse into 18 basic 4-element isolated arrays (4D03WGJ0103T5E /
4D03WGJ0472T5E, element k = pins k/9-k; new mxbus.r_pack4 helper).
Isolated elements let packs mix rails; every net keeps its exact rail
and semantics (verified element-by-element in the netlist). RC/divider/
series/I2C resistors stay discrete. Board 452 -> 406 components; also
de-risks the sole basic 10k 0603 line (0 stock at audit). Audit
recorded in jlcpcb-sourcing.md.

Co-Authored-By: Claude Fable 5 <noreply@anthropic.com>
Parts:
- removed R2, R4: 10k, Resistor_SMD:R_0603_1608Metric, symbol Device:R
- RN1: renamed from R1; value 10k -> 10kx4; footprint Resistor_SMD:R_0603_1608Metric -> Resistor_SMD:R_Array_Convex_4x0603; symbol Device:R -> Device:R_Pack04; LCSC Part Num C25804 -> C29718
Connections:
- net +3V3: now also RN1.7 (R2.2), RN1.8 (R1.2); no longer RN1.1
- net GND: now also RN1.6 (R3.2)
- net IDE_IRQ: now also RN1.3 (R3.1)
- net ~{IORDY}: now also RN1.1 (R1.1); no longer RN1.2
- net ~{IRQ_IDE}: now also RN1.2 (R2.1)
- no-connect marks 36 -> 38
Changed lines of the file:
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@@
 	(wire
 		(pts
-			(xy 228.6 21.59)
-			(xy 228.6 19.05)
+			(xy 223.52 30.48)
+			(xy 223.52 33.02)
+		)
+		(stroke
+			(width 0)
+			(type default)
+		)
+	)
+	(label "~{IORDY}"
+		(at 223.52 33.02 270)
+		(effects
+			(font
+				(size 1.27 1.27)
+			)
+		)
+	)
+	(wire
+		(pts
+			(xy 223.52 20.32)
+			(xy 223.52 17.78)
 		)
 		(stroke
@@
 	(global_label "+3V3"
 		(shape input)
-		(at 228.6 19.05 90)
-		(effects
-			(font
-				(size 1.27 1.27)
-			)
-		)
-	)
-	(wire
-		(pts
-			(xy 228.6 29.21)
-			(xy 228.6 31.75)
-		)
-		(stroke
-			(width 0)
-			(type default)
-		)
-	)
-	(label "~{IORDY}"
-		(at 228.6 31.75 270)
-		(effects
-			(font
-				(size 1.27 1.27)
-			)
-		)
-	)
-	(wire
-		(pts
-			(xy 243.84 21.59)
-			(xy 243.84 19.05)
+		(at 223.52 17.78 90)
+		(effects
+			(font
+				(size 1.27 1.27)
+			)
+		)
+	)
+	(wire
+		(pts
+			(xy 226.06 30.48)
+			(xy 226.06 33.02)
+		)
+		(stroke
+			(width 0)
+			(type default)
+		)
+	)
+	(label "~{IRQ_IDE}"
+		(at 226.06 33.02 270)
+		(effects
+			(font
+				(size 1.27 1.27)
+			)
+		)
+	)
+	(wire
+		(pts
+			(xy 226.06 20.32)
+			(xy 226.06 17.78)
+		)
+		(stroke
+			(width 0)
+			(type default)
+		)
+	)
+	(global_label "+3V3"
+		(shape input)
+		(at 226.06 17.78 90)
+		(effects
+			(font
+				(size 1.27 1.27)
+			)
+		)
+	)
+	(wire
+		(pts
+			(xy 228.6 30.48)
+			(xy 228.6 33.02)
 		)
 		(stroke
@@
 	)
 	(label "IDE_IRQ"
-		(at 243.84 19.05 90)
-		(effects
-			(font
-				(size 1.27 1.27)
-			)
-		)
-	)
-	(wire
-		(pts
-			(xy 243.84 29.21)
-			(xy 243.84 31.75)
+		(at 228.6 33.02 270)
+		(effects
+			(font
+				(size 1.27 1.27)
+			)
+		)
+	)
+	(wire
+		(pts
+			(xy 228.6 20.32)
+			(xy 228.6 17.78)
 		)
 		(stroke
@@
 	(global_label "GND"
 		(shape input)
-		(at 243.84 31.75 270)
-		(effects
-			(font
-				(size 1.27 1.27)
-			)
-		)
-	)
-	(wire
-		(pts
-			(xy 91.44 240.03)
-			(xy 91.44 237.49)
-		)
-		(stroke
-			(width 0)
-			(type default)
-		)
-	)
-	(global_label "+3V3"
-		(shape input)
-		(at 91.44 237.49 90)
-		(effects
-			(font
-				(size 1.27 1.27)
-			)
-		)
-	)
-	(wire
-		(pts
-			(xy 91.44 247.65)
-			(xy 91.44 250.19)
-		)
-		(stroke
-			(width 0)
-			(type default)
-		)
-	)
-	(label "~{IRQ_IDE}"
-		(at 91.44 250.19 270)
-		(effects
-			(font
-				(size 1.27 1.27)
-			)
-		)
+		(at 228.6 17.78 90)
+		(effects
+			(font
+				(size 1.27 1.27)
+			)
+		)
+	)
+	(no_connect
+		(at 231.14 30.48)
+	)
+	(no_connect
+		(at 231.14 20.32)
 	)
 	(wire
@@
 	)
 	(symbol
-		(lib_id "Device:R")
+		(lib_id "Device:R_Pack04")
 		(at 228.6 25.4 0)
 		(unit 1)
@@
 		(dnp no)
 		(fields_autoplaced yes)
-		(property "Reference" "R1"
+		(property "Reference" "RN1"
 			(at 228.6 20.32 0)
 			(effects
@@
 			)
 		)
-		(property "Value" "10k"
+		(property "Value" "10kx4"
 			(at 228.6 30.48 0)
 			(effects
@@
 			)
 		)
-		(property "Footprint" "Resistor_SMD:R_0603_1608Metric"
+		(property "Footprint" "Resistor_SMD:R_Array_Convex_4x0603"
 			(at 228.6 25.4 0)
 			(effects
@@
 			)
 		)
-		(property "LCSC Part Num" "C25804"
+		(property "LCSC Part Num" "C29718"
 			(at 228.6 25.4 0)
 			(effects
@@
 			)
 		)
+		(pin "8"
+		)
 		(pin "1"
 		)
+		(pin "7"
+		)
 		(pin "2"
+		)
+		(pin "6"
+		)
+		(pin "3"
+		)
+		(pin "5"
+		)
+		(pin "4"
 		)
 		(instances
 			(project "mini-xt"
 				(path "/26736c46-8b40-5460-874f-03596d17270c/3d789b7e-8571-58c2-8404-2016fa912ed0"
-					(reference "R801")
+					(reference "RN801")
 					(unit 1)
 				)
-			)
-		)
-	)
-	(symbol
-		(lib_id "Device:R")
-		(at 243.84 25.4 0)
-		(unit 1)
-		(exclude_from_sim no)
-		(in_bom yes)
-		(on_board yes)
-		(dnp no)
-		(fields_autoplaced yes)
-		(property "Reference" "R2"
-			(at 243.84 20.32 0)
-			(effects
-				(font
-					(size 1.27 1.27)
-				)
-			)
-		)
-		(property "Value" "10k"
-			(at 243.84 30.48 0)
-			(effects
-				(font
-					(size 1.27 1.27)
-				)
-			)
-		)
-		(property "Footprint" "Resistor_SMD:R_0603_1608Metric"
-			(at 243.84 25.4 0)
-			(effects
-				(font
-					(size 1.27 1.27)
-				)
-				(hide yes)
-			)
-		)
-		(property "LCSC Part Num" "C25804"
-			(at 243.84 25.4 0)
-			(effects
-				(font
-					(size 1.27 1.27)
-				)
-				(hide yes)
-			)
-		)
-		(pin "1"
-		)
-		(pin "2"
-		)
-		(instances
-			(project "mini-xt"
-				(path "/26736c46-8b40-5460-874f-03596d17270c/3d789b7e-8571-58c2-8404-2016fa912ed0"
-					(reference "R802")
-					(unit 1)
-				)
-			)
-		)
-	)
-	(symbol
-		(lib_id "Device:R")
-		(at 91.44 243.84 0)
-		(unit 1)
-		(exclude_from_sim no)
-		(in_bom yes)
-		(on_board yes)
-		(dnp no)
-		(fields_autoplaced yes)
-		(property "Reference" "R4"
-			(at 91.44 238.76 0)
-			(effects
-				(font
-					(size 1.27 1.27)
-				)
-			)
-		)
-		(property "Value" "10k"
-			(at 91.44 248.92 0)
-			(effects
-				(font
-					(size 1.27 1.27)
-				)
-			)
-		)
-		(property "Footprint" "Resistor_SMD:R_0603_1608Metric"
-			(at 91.44 243.84 0)
-			(effects
-				(font
-					(size 1.27 1.27)
-				)
-				(hide yes)
-			)
-		)
-		(property "LCSC Part Num" "C25804"
-			(at 91.44 243.84 0)
-			(effects
-				(font
-					(size 1.27 1.27)
-				)
-				(hide yes)
-			)
-		)
-		(pin "1"
-		)
-		(pin "2"
-		)
-		(instances
-			(project "mini-xt"
-				(path "/26736c46-8b40-5460-874f-03596d17270c/3d789b7e-8571-58c2-8404-2016fa912ed0"
-					(reference "R804")
-					(unit 1)
-				)
