File: hardware/sheets/sidecar.kicad_sch (KiCad schematic)
At the start: 31 parts, among them J1 ISA 8-bit (60p), U1 74LVC245A, U2 74LVC245A, U3 74LVC245A, U4 74LVC244A, U5 74LVC244A, U6 74LVC245A, U7 74LVC244A, U8 74LVC244A, U9 74LVC2G07

Commit message: 3.3V redesign: final-review fix wave (6 findings)
Reviewer-verified fixes, all at the generator level + regenerated outputs:

1. (Critical) bus_mcu U17 '04 @+3V3 had the V20's 5V HLDA on its input ->
   value-override to 74LVC04A (5V-tolerant input; parts.py binds C282341).
2. network R7 (AEN_CHIP park) +5V -> +3V3: it also feeds U5's '138 @+3V3;
   RTL8019AS AEN is 5V-TTL so 3.3V still reads high.
3. sidecar buf244(): tie unused '244 A inputs to GND, no_connect the Y
   outputs (U1105: 6 spare, U1108: 7) -- no floating always-enabled inputs.
4. MAX3241s (both com_port instances) +5V -> +3V3; charge-pump caps to the
   datasheet 3.0-3.6V column (all 0.1uF). Removes the 5V-R*OUT-into-3.3V-UART
   receiver path; com_port now has no +5V rail.
5. V20 READY/HOLD re-buffered through cpu_core U13's 3 spare '04 gates (zero
   package cost). READY = 2 gates (non-inverting), single-driver (no fold).
   HOLD = 1 inverting gate -> FIRMWARE MUST DRIVE HOLD ACTIVE-LOW at GPIO25
   (mxbus HOLD name intact). U13 nudged to clear a stub collision with U12.
6. Docs census + staleness: rewrote the 5V census to post-fix reality across
   CLAUDE.md, spec, design doc, README, irq-io-map (IRQ8 soft-PIC/undriven),
   parts.py header notes.

Build exit 0; check_parts 0 problems; all five sheets validate with zero
structural violations. Netlist evidence in questions-*.md.

Co-Authored-By: Claude Fable 5 <noreply@anthropic.com>
Parts:
- removed U8: 74LVC244A, Package_SO:TSSOP-20_4.4x6.5mm_P0.65mm, symbol mini-xt:74HCT244
- added R3: 100k, Resistor_SMD:R_0603_1608Metric, symbol Device:R
- U8: renamed from R3; value 100k -> 74LVC244A; footprint Resistor_SMD:R_0603_1608Metric -> Package_SO:TSSOP-20_4.4x6.5mm_P0.65mm; symbol Device:R -> mini-xt:74HCT244; LCSC Part Num C25803 -> C6079
Connections:
- net +3V3: now also U8.20 (VCC)
- net EXT_IRQ3: now also U8.18 (1Y0)
- net GND: now also U5.11 (2A3), U5.13 (2A2), U5.15 (2A1), U5.17 (2A0), U5.6 (1A2), U5.8 (1A3), U8.1 (1OE), U8.10 (GND), U8.11 (2A3), U8.13 (2A2), U8.15 (2A1), U8.17 (2A0), U8.19 (2OE), U8.4 (1A1), U8.6 (1A2), U8.8 (1A3), R3.2; no longer U8.2
- net X_DRQ2: now also R3.1; no longer U8.1
- net X_IRQ3: now also U8.2 (1A0)
- no-connect marks 1 -> 14
