File: hardware/sheets/parallel.kicad_sch (KiCad schematic)
At the start: 37 parts, among them J1 DB25_Pins, U1 74HCT574, U10 74HCT32, U11 74HCT32, U12 74HCT00, U13 74HCT125, U2 74HCT574, U3 74HCT244, U4 74HCT245, U5 74HCT244, U6 74HCT138, U7 74HCT08, U8 74HCT08, U9 74HCT04

Commit message: IRQ rework: single-'165 collector, hardwired COM/LPT IRQs
- IRQ collector shrunk to one 74HCT165: D0-D6 = IRQ2-8, D7 = IRQ14
  (replacing the source-less IRQ9). U19 + pull-downs R19-R24 + C18
  deleted; IRQ9-13/15 dropped everywhere (nothing on the board or the
  8-bit header can drive them). Firmware shifts 8 bits, Q7-first.
- COM/LPT IRQ straps deleted, hardwired to the PC conventions:
  COM1=IRQ4, COM2=IRQ3 (COM_IRQ per-instance netmap remap -- first use
  of the INSTANCES netmap), LPT=IRQ7 (U13 '125 drives the net
  directly). The enable jumpers (COM JP3, LPT JP2) free an IRQ by
  disabling the port; the tri-state drivers go silent with it.
- Storage JP3 (IRQ14/IRQ5) kept: both positions are real conventions
  (AT vs XT), not conflict avoidance. Its IRQ5 warning now points at
  the PicoGUS jumper block, the only remaining IRQ5 contention.
- Design doc: fix stale claim that IRQ8 rides a reclaimed header pin
  (that pin is a ground return; IRQ8 is motherboard-internal).

Full-build ERC: 0 violations.

Co-Authored-By: Claude Fable 5 <noreply@anthropic.com>
Parts:
- removed C13: 100nF, symbol Device:C
- removed C14: 10uF, symbol Device:C
- removed JP3: IRQ strap, symbol Connector_Generic:Conn_01x03
- added C1, C2: 100nF, symbol Device:C
- C14: renamed from C12; value 100nF -> 10uF; LCSC Part Num C14663 -> C15850
- renumbered C8 to C10, C9 to C11, C10 to C12, C11 to C13, C1 to C3, C2 to C4, C3 to C5, C4 to C6, C5 to C7, C6 to C8, C7 to C9
Connections:
- net LPT_IRQ is gone; now on net IRQ7: U13.3 (P3)
- net +5V: now also C1.1, C2.1
- net GND: now also C1.2, C2.2
Other:
- note added: "JP1: base 0x378/0x278; JP2: open=port disabled (frees IRQ7); IRQ7 hardwired"
- note removed: "JP1: base 0x378/0x278; JP2: open=port disabled; JP3: IRQ7/IRQ5/open=polled"
- moved on the sheet: C10, C11, C12, C13, C14, C3, C4, C5, C6, C7, C8, C9

Commit message: Parts: footprints for all components, close 6 LCSC map gaps, check_parts.py
- mxsch.py emits the Footprint property from component props (was
  hard-coded empty); parts.py entries now carry a verified KiCad
  footprint, applied at build time alongside the LCSC number.
- Map keys fixed to match placed values: USB_PROG, SS34, LED (PicoGUS),
  APS6404L, CB3T3257/45 -- every combo across all sheets + cards now
  resolves (130 combos, 455 netlist components, all with footprints).
- Package corrections from JLC DB re-check: RTL8019AS is QFP-100 14x20
  P0.65 (not TQFP); C2897411 female header is a 2x10 strip -- fine for
  Core2350B, Pico needs 2x 1x20 (noted in jlcpcb-sourcing.md).
- 10 mini-xt:* placeholder footprints mark parts whose land pattern is
  authored at layout from the EasyEDA data (CH224K, magnetics, RJ45,
  HDMI, CF socket, ISA slot, switches, Core2350B PGA).
- New tools/check_parts.py: fails on unmapped combos, missing fp
  fields, or footprints absent from the installed KiCad libs.

Co-Authored-By: Claude Fable 5 <noreply@anthropic.com>
Parts:
- C1, C10, C11, C12, C13, C2, C3, C4, C5, C6, C7, C8, C9: footprint (none) -> Capacitor_SMD:C_0603_1608Metric
- C14: footprint (none) -> Capacitor_SMD:C_0805_2012Metric
- J1: footprint (none) -> Connector_Dsub:DSUB-25_Pins_Horizontal_P2.77x2.84mm_EdgePinOffset9.90mm_Housed_MountingHolesOffset11.32mm
- JP1: footprint (none) -> Connector_PinHeader_2.54mm:PinHeader_1x03_P2.54mm_Vertical
- JP2: footprint (none) -> Connector_PinHeader_2.54mm:PinHeader_1x02_P2.54mm_Vertical
- R1, R2, R3, R4, R5, R6: footprint (none) -> Resistor_SMD:R_0603_1608Metric
- U1, U2, U3, U4, U5: footprint (none) -> Package_SO:SOIC-20W_7.5x12.8mm_P1.27mm
- U10, U11, U12, U13, U7, U8, U9: footprint (none) -> Package_SO:SOIC-14_3.9x8.7mm_P1.27mm
- U6: footprint (none) -> Package_SO:SOIC-16_3.9x9.9mm_P1.27mm
Changed lines of the file:
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@@
 			)
 		)
-		(property "Footprint" ""
+		(property "Footprint" "Package_SO:SOIC-14_3.9x8.7mm_P1.27mm"
 			(at 76.2 76.2 0)
 			(effects
@@
 			)
 		)
-		(property "Footprint" ""
+		(property "Footprint" "Package_SO:SOIC-14_3.9x8.7mm_P1.27mm"
 			(at 76.2 127 0)
 			(effects
@@
 			)
 		)
-		(property "Footprint" ""
+		(property "Footprint" "Package_SO:SOIC-14_3.9x8.7mm_P1.27mm"
 			(at 76.2 177.8 0)
 			(effects
@@
 			)
 		)
-		(property "Footprint" ""
+		(property "Footprint" "Package_SO:SOIC-14_3.9x8.7mm_P1.27mm"
 			(at 266.7 76.2 0)
 			(effects
@@
 			)
 		)
-		(property "Footprint" ""
+		(property "Footprint" "Package_SO:SOIC-14_3.9x8.7mm_P1.27mm"
 			(at 266.7 127 0)
 			(effects
@@
 			)
 		)
-		(property "Footprint" ""
+		(property "Footprint" "Package_SO:SOIC-16_3.9x9.9mm_P1.27mm"
 			(at 139.7 177.8 0)
 			(effects
@@
 			)
 		)
-		(property "Footprint" ""
+		(property "Footprint" "Package_SO:SOIC-14_3.9x8.7mm_P1.27mm"
 			(at 203.2 177.8 0)
 			(effects
@@
 			)
 		)
-		(property "Footprint" ""
+		(property "Footprint" "Package_SO:SOIC-14_3.9x8.7mm_P1.27mm"
 			(at 266.7 177.8 0)
 			(effects
@@
 			)
 		)
-		(property "Footprint" ""
+		(property "Footprint" "Package_SO:SOIC-20W_7.5x12.8mm_P1.27mm"
 			(at 139.7 76.2 0)
 			(effects
@@
 			)
 		)
-		(property "Footprint" ""
+		(property "Footprint" "Package_SO:SOIC-20W_7.5x12.8mm_P1.27mm"
 			(at 203.2 76.2 0)
 			(effects
@@
 			)
 		)
-		(property "Footprint" ""
+		(property "Footprint" "Package_SO:SOIC-20W_7.5x12.8mm_P1.27mm"
 			(at 139.7 127 0)
 			(effects
@@
 			)
 		)
-		(property "Footprint" ""
+		(property "Footprint" "Package_SO:SOIC-20W_7.5x12.8mm_P1.27mm"
 			(at 203.2 127 0)
 			(effects
@@
 			)
 		)
-		(property "Footprint" ""
+		(property "Footprint" "Package_SO:SOIC-20W_7.5x12.8mm_P1.27mm"
 			(at 203.2 228.6 0)
 			(effects
@@
 			)
 		)
-		(property "Footprint" ""
+		(property "Footprint" "Connector_Dsub:DSUB-25_Pins_Horizontal_P2.77x2.84mm_EdgePinOffset9.90mm_Housed_MountingHolesOffset11.32mm"
 			(at 355.6 127 0)
 			(effects
@@
 			)
 		)
-		(property "Footprint" ""
+		(property "Footprint" "Resistor_SMD:R_0603_1608Metric"
 			(at 314.96 45.72 0)
 			(effects
@@
 			)
 		)
-		(property "Footprint" ""
+		(property "Footprint" "Resistor_SMD:R_0603_1608Metric"
 			(at 330.2 45.72 0)
 			(effects
@@
 			)
 		)
-		(property "Footprint" ""
+		(property "Footprint" "Resistor_SMD:R_0603_1608Metric"
 			(at 345.44 45.72 0)
 			(effects
@@
 			)
 		)
-		(property "Footprint" ""
+		(property "Footprint" "Resistor_SMD:R_0603_1608Metric"
 			(at 360.68 45.72 0)
 			(effects
@@
 			)
 		)
-		(property "Footprint" ""
+		(property "Footprint" "Resistor_SMD:R_0603_1608Metric"
 			(at 375.92 45.72 0)
 			(effects
@@
 			)
 		)
-		(property "Footprint" ""
+		(property "Footprint" "Connector_PinHeader_2.54mm:PinHeader_1x03_P2.54mm_Vertical"
 			(at 299.72 195.58 0)
 			(effects
@@
 			)
 		)
-		(property "Footprint" ""
+		(property "Footprint" "Connector_PinHeader_2.54mm:PinHeader_1x02_P2.54mm_Vertical"
 			(at 314.96 195.58 0)
 			(effects
@@
 			)
 		)
-		(property "Footprint" ""
+		(property "Footprint" "Resistor_SMD:R_0603_1608Metric"
 			(at 345.44 195.58 0)
 			(effects
@@
 			)
 		)
-		(property "Footprint" ""
+		(property "Footprint" "Capacitor_SMD:C_0603_1608Metric"
 			(at 30.48 264.16 0)
 			(effects
@@
 			)
 		)
-		(property "Footprint" ""
+		(property "Footprint" "Capacitor_SMD:C_0603_1608Metric"
 			(at 60.96 264.16 0)
 			(effects
@@
 			)
 		)
-		(property "Footprint" ""
+		(property "Footprint" "Capacitor_SMD:C_0603_1608Metric"
 			(at 91.44 264.16 0)
 			(effects
@@
 			)
 		)
-		(property "Footprint" ""
+		(property "Footprint" "Capacitor_SMD:C_0603_1608Metric"
 			(at 121.92 264.16 0)
 			(effects
@@
 			)
 		)
-		(property "Footprint" ""
+		(property "Footprint" "Capacitor_SMD:C_0603_1608Metric"
 			(at 152.4 264.16 0)
 			(effects
@@
 			)
 		)
-		(property "Footprint" ""
+		(property "Footprint" "Capacitor_SMD:C_0603_1608Metric"
 			(at 182.88 264.16 0)
 			(effects
@@
 			)
 		)
-		(property "Footprint" ""
+		(property "Footprint" "Capacitor_SMD:C_0603_1608Metric"
 			(at 213.36 264.16 0)
 			(effects
@@
 			)
 		)
-		(property "Footprint" ""
+		(property "Footprint" "Capacitor_SMD:C_0603_1608Metric"
 			(at 243.84 264.16 0)
 			(effects
@@
 			)
 		)
-		(property "Footprint" ""
+		(property "Footprint" "Capacitor_SMD:C_0603_1608Metric"
 			(at 274.32 264.16 0)
 			(effects
@@
 			)
 		)
-		(property "Footprint" ""
+		(property "Footprint" "Capacitor_SMD:C_0603_1608Metric"
 			(at 304.8 264.16 0)
 			(effects
@@
 			)
 		)
-		(property "Footprint" ""
+		(property "Footprint" "Capacitor_SMD:C_0603_1608Metric"
 			(at 335.28 264.16 0)
 			(effects
@@
 			)
 		)
-		(property "Footprint" ""
+		(property "Footprint" "Capacitor_SMD:C_0603_1608Metric"
 			(at 365.76 264.16 0)
 			(effects
@@
 			)
 		)
-		(property "Footprint" ""
+		(property "Footprint" "Capacitor_SMD:C_0603_1608Metric"
 			(at 396.24 264.16 0)
 			(effects
@@
 			)
 		)
-		(property "Footprint" ""
+		(property "Footprint" "Capacitor_SMD:C_0805_2012Metric"
 			(at 30.48 238.76 0)
 			(effects

Commit message: com/network/storage/parallel: 3.3V; TL16C550CPT soldered; LVC at external connectors
com_port: PLCC-44 16550 socket -> soldered TL16C550PT (LQFP-48) at +3V3,
rewired signal-for-signal from pins.py (RD/WR split renamed RD1/RD2/WR1/WR2,
INTR->INTRPT, GND->VSS, 8 new NC pins). Decode glue -> HC-grade, IRQ buffer
-> LVC125A, all +3V3. MAX3241 untouched (+5V, spec: already 3.3V-compatible).

network: only U3 (IRQ/AEN gate) moves, to LVC125A @ +3V3 -- RTL8019AS and
its EEPROM stay +5V (datasheet-verified 5V-only part, same treatment as
MAX3241), deviating from a literal reading of the brief's "power sweep"
instruction in favor of its own MAX3241 precedent.

storage: full brief table applied, all +3V3 except the CompactFlash
socket's own VCC power-feed pins (real CF-spec requirement, not a logic
signal).

parallel: brief's swap table only named 8 of 13 chips; traced the DB25
connector's actual net fan-out to fill the gap (U5, U9 also need
5V-tolerant inputs; U6/U7/U8/U12 are purely internal decode -> HC-grade).
U9 reuses the already-bound 74AHC14 value (no bare LVC04A entry exists).

Decisions logged in hardware/notes/questions-{com_port,network,storage,parallel}.md.

Co-Authored-By: Claude Fable 5 <noreply@anthropic.com>
Parts:
- U1, U2: value 74HCT574 -> 74LVC574A; footprint Package_SO:SOIC-20W_7.5x12.8mm_P1.27mm -> Package_SO:TSSOP-20_4.4x6.5mm_P0.65mm; LCSC Part Num C6001 -> C842658
- U10, U11: value 74HCT32 -> 74HC32; LCSC Part Num C5985 -> C52140395
- U12: value 74HCT00 -> 74HC00; LCSC Part Num C282337 -> C699445
- U13: value 74HCT125 -> 74LVC125A; LCSC Part Num C5962 -> C6057
- U3, U5: value 74HCT244 -> 74LVC244A; footprint Package_SO:SOIC-20W_7.5x12.8mm_P1.27mm -> Package_SO:TSSOP-20_4.4x6.5mm_P0.65mm; LCSC Part Num C5978 -> C6079
- U4: value 74HCT245 -> 74LVC245A; footprint Package_SO:SOIC-20W_7.5x12.8mm_P1.27mm -> Package_SO:TSSOP-20_4.4x6.5mm_P0.65mm; LCSC Part Num C5979 -> C6082
- U6: value 74HCT138 -> 74HC138; LCSC Part Num C5965 -> C5602
- U7, U8: value 74HCT08 -> 74HC08; LCSC Part Num C5959 -> C5593
- U9: value 74HCT04 -> 74AHC14; footprint Package_SO:SOIC-14_3.9x8.7mm_P1.27mm -> Package_SO:TSSOP-14_4.4x5mm_P0.65mm; LCSC Part Num C672096 -> C54561786
Connections:
- net +5V renamed +3V3

Commit message: addr_decode: central I/O decode, IRQ mapping + disable jumpers; UART -> TL16C550CPFBR
New addr_decode sheet owns the discrete peripherals' bus plumbing:
'138+'00+'32 windowed decode exports ~COM1/~COM2/~LPT/~IDE chip selects
(0x3F8/0x2F8/0x378 share one A5.A4.A3 fine term); one shared 74LVC125A
maps the peripherals' private IRQ requests onto IRQ4/3/7/14 (COM keeps
~OUT2 gating), replacing the three per-sheet '125s; base straps (JP1/JP2,
pulled-high commons) and per-peripheral disable jumpers JP3-JP6 (enabled
by default, fit to disable via a second '32 rank on the CS) live here.
com_port/parallel/storage lose their decode gates, IRQ drivers and
enable jumpers; board drops 97 -> 93 ICs. Docs reframed per feedback:
PRIV_CS/PRIV_IRQREQ are shared logic factored out, not isolation breaks.

UART rebound to the active TL16C550CPFBR (TQFP-48, LCSC C882798, thin
stock) -- pinout verified identical to the symbol via jlc_get_pinout;
parts.py-only swap, sourcing notes updated.

Co-Authored-By: Claude Fable 5 <noreply@anthropic.com>
Parts:
- removed C11, C12, C13: 100nF, Capacitor_SMD:C_0603_1608Metric, symbol Device:C
- removed JP1: BASE 378/278, Connector_PinHeader_2.54mm:PinHeader_1x03_P2.54mm_Vertical, symbol Connector_Generic:Conn_01x03
- removed JP2: LPT_EN, Connector_PinHeader_2.54mm:PinHeader_1x02_P2.54mm_Vertical, symbol Connector_Generic:Conn_01x02
- removed R6: 10k, Resistor_SMD:R_0603_1608Metric, symbol Device:R
- removed U13: 74LVC125A, Package_SO:SOIC-14_3.9x8.7mm_P1.27mm, symbol mini-xt:74HCT125
- removed U7, U8: 74HC08, Package_SO:SOIC-14_3.9x8.7mm_P1.27mm, symbol mini-xt:74HCT08
Connections:
- net A7 is gone; now on net GND: U9.1 (P1)
- net A8 is gone; now on net GND: U12.4 (P4), U12.5 (P5)
- net ADDR_MATCH is gone; now on net +3V3: U6.6 (E2)
- net ~{LPT_EN} is gone; now on net GND: U6.5 (~{E1})
- net AEN renamed ~{LPT_CS}
- net NA7: no longer names the net of U9.2 (P2)
- net NA8: no longer names the net of U12.6 (P6)
- net ~{IRQ7_OE} renamed ~{IRQ_LPT}
- no-connect marks 21 -> 18
Other:
- note added: "Base strap + disable jumper: addr_decode JP1/JP5; IRQ7 hardwired via its '125"
- note removed: "JP1: base 0x378/0x278; JP2: open=port disabled (frees IRQ7); IRQ7 hardwired"

Commit message: bus_mcu: delete U17 (74LVC04A, 1/6 gates) -- HLDA inverter moves to parallel's spare gate
The HLDA -> ~{HLDA} inversion for the counter '244s now lives on the
parallel sheet's spare 74AHC14 Schmitt gate (U9.1, freed by the decode
centralization) -- the board's only spare 5V-tolerant inverter, which is
what HLDA (raw 5V V20 output) requires. ~{HLDA} joins mxbus.PRIV_CPU and
crosses as an interface net; park-safety unchanged (R18 parks HLDA low,
~{HLDA} idles high, '244s off during MCU-Hi-Z). U17 + its decoupler
deleted; the orphaned 74LVC04A parts.py line (C282341) removed. Board
454 comps / 92 ICs. Also sweeps stale JP-number refs left in the
parallel/storage/com_port docstrings from the jumper renumber.

Co-Authored-By: Claude Fable 5 <noreply@anthropic.com>
Connections:
- net GND: no longer U9.1 (P1)
- net ~{HLDA}: now reaches U9.2 (P2)
- new net HLDA: U9.1 (P1)
- no-connect marks 18 -> 17
Other:
- note added: "Base hardwired 0x378; disable: addr_decode JP3; IRQ7 hardwired via its '125; U9.1 hosts the HLDA inverter"
- note removed: "Base strap + disable jumper: addr_decode JP1/JP5; IRQ7 hardwired via its '125"
Changed lines of the file:
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@@
 	(wire
 		(pts
+			(xy 22.86 63.5)
+			(xy 25.4 63.5)
+		)
+		(stroke
+			(width 0)
+			(type default)
+		)
+	)
+	(label "HLDA"
+		(at 22.86 63.5 180)
+		(effects
+			(font
+				(size 1.27 1.27)
+			)
+			(justify right)
+		)
+	)
+	(hierarchical_label "HLDA"
+		(shape input)
+		(at 25.4 63.5 0)
+		(effects
+			(font
+				(size 1.27 1.27)
+			)
+		)
+	)
+	(wire
+		(pts
+			(xy 22.86 66.04)
+			(xy 25.4 66.04)
+		)
+		(stroke
+			(width 0)
+			(type default)
+		)
+	)
+	(label "~{HLDA}"
+		(at 22.86 66.04 180)
+		(effects
+			(font
+				(size 1.27 1.27)
+			)
+			(justify right)
+		)
+	)
+	(hierarchical_label "~{HLDA}"
+		(shape output)
+		(at 25.4 66.04 0)
+		(effects
+			(font
+				(size 1.27 1.27)
+			)
+		)
+	)
+	(wire
+		(pts
 			(xy 76.2 165.1)
 			(xy 76.2 162.56)
@@
 		)
 	)
-	(global_label "GND"
-		(shape input)
+	(label "HLDA"
 		(at 59.69 171.45 180)
 		(effects
@@
 		)
 	)
-	(no_connect
-		(at 90.17 171.45)
+	(wire
+		(pts
+			(xy 90.17 171.45)
+			(xy 92.71 171.45)
+		)
+		(stroke
+			(width 0)
+			(type default)
+		)
+	)
+	(label "~{HLDA}"
+		(at 92.71 171.45 0)
+		(effects
+			(font
+				(size 1.27 1.27)
+			)
+		)
 	)
 	(wire
@@
 		)
 	)
-	(text "Base strap + disable jumper: addr_decode JP1/JP5; IRQ7 hardwired via its '125"
+	(text "Base hardwired 0x378; disable: addr_decode JP3; IRQ7 hardwired via its '125; U9.1 hosts the HLDA inverter"
 		(at 299.72 187.96 0)
 		(effects
@@
 		(instances
 			(project "mini-xt"
-				(path "/26736c46-8b40-5460-874f-03596d17270c/99b9ac7c-ce6d-5291-b48a-bf88e0661a04"
+				(path "/26736c46-8b40-5460-874f-03596d17270c/e70e4f43-b519-598d-b449-edcea257db69"
 					(reference "U609")
 					(unit 1)
@@
 		(instances
 			(project "mini-xt"
-				(path "/26736c46-8b40-5460-874f-03596d17270c/99b9ac7c-ce6d-5291-b48a-bf88e0661a04"
+				(path "/26736c46-8b40-5460-874f-03596d17270c/e70e4f43-b519-598d-b449-edcea257db69"
 					(reference "U612")
 					(unit 1)
@@
 		(instances
 			(project "mini-xt"
-				(path "/26736c46-8b40-5460-874f-03596d17270c/99b9ac7c-ce6d-5291-b48a-bf88e0661a04"
+				(path "/26736c46-8b40-5460-874f-03596d17270c/e70e4f43-b519-598d-b449-edcea257db69"
 					(reference "U606")
 					(unit 1)
@@
 		(instances
 			(project "mini-xt"
-				(path "/26736c46-8b40-5460-874f-03596d17270c/99b9ac7c-ce6d-5291-b48a-bf88e0661a04"
+				(path "/26736c46-8b40-5460-874f-03596d17270c/e70e4f43-b519-598d-b449-edcea257db69"
 					(reference "U610")
 					(unit 1)
@@
 		(instances
 			(project "mini-xt"
-				(path "/26736c46-8b40-5460-874f-03596d17270c/99b9ac7c-ce6d-5291-b48a-bf88e0661a04"
+				(path "/26736c46-8b40-5460-874f-03596d17270c/e70e4f43-b519-598d-b449-edcea257db69"
 					(reference "U611")
 					(unit 1)
@@
 		(instances
 			(project "mini-xt"
-				(path "/26736c46-8b40-5460-874f-03596d17270c/99b9ac7c-ce6d-5291-b48a-bf88e0661a04"
+				(path "/26736c46-8b40-5460-874f-03596d17270c/e70e4f43-b519-598d-b449-edcea257db69"
 					(reference "U601")
 					(unit 1)
@@
 		(instances
 			(project "mini-xt"
-				(path "/26736c46-8b40-5460-874f-03596d17270c/99b9ac7c-ce6d-5291-b48a-bf88e0661a04"
+				(path "/26736c46-8b40-5460-874f-03596d17270c/e70e4f43-b519-598d-b449-edcea257db69"
 					(reference "U604")
 					(unit 1)
@@
 		(instances
 			(project "mini-xt"
-				(path "/26736c46-8b40-5460-874f-03596d17270c/99b9ac7c-ce6d-5291-b48a-bf88e0661a04"
+				(path "/26736c46-8b40-5460-874f-03596d17270c/e70e4f43-b519-598d-b449-edcea257db69"
 					(reference "U602")
 					(unit 1)
@@
 		(instances
 			(project "mini-xt"
-				(path "/26736c46-8b40-5460-874f-03596d17270c/99b9ac7c-ce6d-5291-b48a-bf88e0661a04"
+				(path "/26736c46-8b40-5460-874f-03596d17270c/e70e4f43-b519-598d-b449-edcea257db69"
 					(reference "U605")
 					(unit 1)
@@
 		(instances
 			(project "mini-xt"
-				(path "/26736c46-8b40-5460-874f-03596d17270c/99b9ac7c-ce6d-5291-b48a-bf88e0661a04"
+				(path "/26736c46-8b40-5460-874f-03596d17270c/e70e4f43-b519-598d-b449-edcea257db69"
 					(reference "U603")
 					(unit 1)
@@
 		(instances
 			(project "mini-xt"
-				(path "/26736c46-8b40-5460-874f-03596d17270c/99b9ac7c-ce6d-5291-b48a-bf88e0661a04"
+				(path "/26736c46-8b40-5460-874f-03596d17270c/e70e4f43-b519-598d-b449-edcea257db69"
 					(reference "J601")
 					(unit 1)
@@
 		(instances
 			(project "mini-xt"
-				(path "/26736c46-8b40-5460-874f-03596d17270c/99b9ac7c-ce6d-5291-b48a-bf88e0661a04"
+				(path "/26736c46-8b40-5460-874f-03596d17270c/e70e4f43-b519-598d-b449-edcea257db69"
 					(reference "R601")
 					(unit 1)
@@
 		(instances
 			(project "mini-xt"
-				(path "/26736c46-8b40-5460-874f-03596d17270c/99b9ac7c-ce6d-5291-b48a-bf88e0661a04"
+				(path "/26736c46-8b40-5460-874f-03596d17270c/e70e4f43-b519-598d-b449-edcea257db69"
 					(reference "R602")
 					(unit 1)
@@
 		(instances
 			(project "mini-xt"
-				(path "/26736c46-8b40-5460-874f-03596d17270c/99b9ac7c-ce6d-5291-b48a-bf88e0661a04"
+				(path "/26736c46-8b40-5460-874f-03596d17270c/e70e4f43-b519-598d-b449-edcea257db69"
 					(reference "R603")
 					(unit 1)
@@
 		(instances
 			(project "mini-xt"
-				(path "/26736c46-8b40-5460-874f-03596d17270c/99b9ac7c-ce6d-5291-b48a-bf88e0661a04"
+				(path "/26736c46-8b40-5460-874f-03596d17270c/e70e4f43-b519-598d-b449-edcea257db69"
 					(reference "R604")
 					(unit 1)
@@
 		(instances
 			(project "mini-xt"
-				(path "/26736c46-8b40-5460-874f-03596d17270c/99b9ac7c-ce6d-5291-b48a-bf88e0661a04"
+				(path "/26736c46-8b40-5460-874f-03596d17270c/e70e4f43-b519-598d-b449-edcea257db69"
 					(reference "R605")
 					(unit 1)
@@
 		(instances
 			(project "mini-xt"
-				(path "/26736c46-8b40-5460-874f-03596d17270c/99b9ac7c-ce6d-5291-b48a-bf88e0661a04"
+				(path "/26736c46-8b40-5460-874f-03596d17270c/e70e4f43-b519-598d-b449-edcea257db69"
 					(reference "C601")
 					(unit 1)
@@
 		(instances
 			(project "mini-xt"
-				(path "/26736c46-8b40-5460-874f-03596d17270c/99b9ac7c-ce6d-5291-b48a-bf88e0661a04"
+				(path "/26736c46-8b40-5460-874f-03596d17270c/e70e4f43-b519-598d-b449-edcea257db69"
 					(reference "C602")
 					(unit 1)
@@
 		(instances
 			(project "mini-xt"
-				(path "/26736c46-8b40-5460-874f-03596d17270c/99b9ac7c-ce6d-5291-b48a-bf88e0661a04"
+				(path "/26736c46-8b40-5460-874f-03596d17270c/e70e4f43-b519-598d-b449-edcea257db69"
 					(reference "C603")
 					(unit 1)
@@
 		(instances
 			(project "mini-xt"
-				(path "/26736c46-8b40-5460-874f-03596d17270c/99b9ac7c-ce6d-5291-b48a-bf88e0661a04"
+				(path "/26736c46-8b40-5460-874f-03596d17270c/e70e4f43-b519-598d-b449-edcea257db69"
 					(reference "C604")
 					(unit 1)
@@
 		(instances
 			(project "mini-xt"
-				(path "/26736c46-8b40-5460-874f-03596d17270c/99b9ac7c-ce6d-5291-b48a-bf88e0661a04"
+				(path "/26736c46-8b40-5460-874f-03596d17270c/e70e4f43-b519-598d-b449-edcea257db69"
 					(reference "C605")
 					(unit 1)
@@
 		(instances
 			(project "mini-xt"
-				(path "/26736c46-8b40-5460-874f-03596d17270c/99b9ac7c-ce6d-5291-b48a-bf88e0661a04"
+				(path "/26736c46-8b40-5460-874f-03596d17270c/e70e4f43-b519-598d-b449-edcea257db69"
 					(reference "C606")
 					(unit 1)
@@
 		(instances
 			(project "mini-xt"
-				(path "/26736c46-8b40-5460-874f-03596d17270c/99b9ac7c-ce6d-5291-b48a-bf88e0661a04"
+				(path "/26736c46-8b40-5460-874f-03596d17270c/e70e4f43-b519-598d-b449-edcea257db69"
 					(reference "C607")
 					(unit 1)
@@
 		(instances
 			(project "mini-xt"
-				(path "/26736c46-8b40-5460-874f-03596d17270c/99b9ac7c-ce6d-5291-b48a-bf88e0661a04"
+				(path "/26736c46-8b40-5460-874f-03596d17270c/e70e4f43-b519-598d-b449-edcea257db69"
 					(reference "C608")
 					(unit 1)
@@
 		(instances
 			(project "mini-xt"
-				(path "/26736c46-8b40-5460-874f-03596d17270c/99b9ac7c-ce6d-5291-b48a-bf88e0661a04"
+				(path "/26736c46-8b40-5460-874f-03596d17270c/e70e4f43-b519-598d-b449-edcea257db69"
 					(reference "C609")
 					(unit 1)
@@
 		(instances
 			(project "mini-xt"
-				(path "/26736c46-8b40-5460-874f-03596d17270c/99b9ac7c-ce6d-5291-b48a-bf88e0661a04"
+				(path "/26736c46-8b40-5460-874f-03596d17270c/e70e4f43-b519-598d-b449-edcea257db69"
 					(reference "C610")
 					(unit 1)
@@
 		(instances
 			(project "mini-xt"
-				(path "/26736c46-8b40-5460-874f-03596d17270c/99b9ac7c-ce6d-5291-b48a-bf88e0661a04"
+				(path "/26736c46-8b40-5460-874f-03596d17270c/e70e4f43-b519-598d-b449-edcea257db69"
 					(reference "C614")
 					(unit 1)
