File: hardware/sheets/power.kicad_sch (KiCad schematic)
At the start: 25 parts, among them J1 USB_C_Receptacle, U1 CH224K, U2 TPS563200

Commit message: ERC power cleanup: single flag owner, flags on series-fed rails
Full-build ERC is now just the 6 expected IRQ9-13/15 label_dangling.

- Root's duplicate PWR_FLAGs removed from build.py: power.py #FLG1-3
  own +5V/+3V3/GND; the pair made flag-vs-flag pin_to_pin errors.
- PWR_FLAGs added on the local rails ERC can't see through a series
  part: VBUS_MCU / VBUS_VID (Schottky diode-OR), VBUS_KBD / HDMI_5V
  (polyfuse), CH224_VDD (1k per WCH ref), AVDD_PGUS / AGND_PGUS
  (ferrite beads).

Net membership verified unchanged: 821 nets, node-identical to HEAD.

Co-Authored-By: Claude Fable 5 <noreply@anthropic.com>
Changed lines of the file:
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@@
+	(wire
+		(pts
+			(xy 91.44 114.3)
+			(xy 91.44 111.76)
+		)
+		(stroke
+			(width 0)
+			(type default)
+		)
+	)
+	(label "CH224_VDD"
+		(at 91.44 111.76 90)
+		(effects
+			(font
+				(size 1.27 1.27)
+			)
+		)
+	)
 	(wire
 		(pts
@@
 					(unit 1)
 				)
+			)
+		)
+	)
+	(symbol
+		(lib_id "power:PWR_FLAG")
+		(at 91.44 114.3 0)
+		(unit 1)
+		(exclude_from_sim no)
+		(in_bom yes)
+		(on_board yes)
+		(dnp no)
+		(fields_autoplaced yes)
+		(property "Reference" "#FLG5"
+			(at 91.44 109.22 0)
+			(effects
+				(font
+					(size 1.27 1.27)
+				)
+			)
+		)
+		(property "Value" "PWR_FLAG"
+			(at 91.44 119.38 0)
+			(effects
+				(font
+					(size 1.27 1.27)
+				)
+			)
+		)
+		(property "Footprint" ""
+			(at 91.44 114.3 0)
+			(effects
+				(font
+					(size 1.27 1.27)
+				)
+				(hide yes)
+			)
+		)
+		(pin "1"
+		)
+		(instances
+			(project "mini-xt"
+				(path "/26736c46-8b40-5460-874f-03596d17270c/a693f317-71cb-5d55-b841-ca6e41b33f1b"
+					(reference "#FLG905")
+					(unit 1)
+				)

Commit message: Parts: footprints for all components, close 6 LCSC map gaps, check_parts.py
- mxsch.py emits the Footprint property from component props (was
  hard-coded empty); parts.py entries now carry a verified KiCad
  footprint, applied at build time alongside the LCSC number.
- Map keys fixed to match placed values: USB_PROG, SS34, LED (PicoGUS),
  APS6404L, CB3T3257/45 -- every combo across all sheets + cards now
  resolves (130 combos, 455 netlist components, all with footprints).
- Package corrections from JLC DB re-check: RTL8019AS is QFP-100 14x20
  P0.65 (not TQFP); C2897411 female header is a 2x10 strip -- fine for
  Core2350B, Pico needs 2x 1x20 (noted in jlcpcb-sourcing.md).
- 10 mini-xt:* placeholder footprints mark parts whose land pattern is
  authored at layout from the EasyEDA data (CH224K, magnetics, RJ45,
  HDMI, CF socket, ISA slot, switches, Core2350B PGA).
- New tools/check_parts.py: fails on unmapped combos, missing fp
  fields, or footprints absent from the installed KiCad libs.

Co-Authored-By: Claude Fable 5 <noreply@anthropic.com>
Parts:
- C1, C3, C7, C9: footprint (none) -> Capacitor_SMD:C_1206_3216Metric
- C2, C4, C5, C6: footprint (none) -> Capacitor_SMD:C_0603_1608Metric
- C8: footprint (none) -> Capacitor_SMD:C_0805_2012Metric
- D1, D2: footprint (none) -> LED_SMD:LED_0603_1608Metric
- D3: footprint (none) -> Diode_SMD:D_SMB
- F1: footprint (none) -> Fuse:Fuse_1812_4532Metric
- J1: footprint (none) -> Connector_USB:USB_C_Receptacle_HRO_TYPE-C-31-M-12
- L1: footprint (none) -> Inductor_SMD:L_Taiyo-Yuden_NR-40xx
- R1, R2, R4, R5, R6, R7, R8, R9: footprint (none) -> Resistor_SMD:R_0603_1608Metric
- U1: footprint (none) -> mini-xt:ESSOP-10_150mil_P1.0mm
- U2: footprint (none) -> Package_TO_SOT_SMD:TSOT-23-6
Changed lines of the file:
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@@
 			)
 		)
-		(property "Footprint" ""
+		(property "Footprint" "Connector_USB:USB_C_Receptacle_HRO_TYPE-C-31-M-12"
 			(at 50.8 165.1 0)
 			(effects
@@
 			)
 		)
-		(property "Footprint" ""
+		(property "Footprint" "Resistor_SMD:R_0603_1608Metric"
 			(at 88.9 195.58 0)
 			(effects
@@
 			)
 		)
-		(property "Footprint" ""
+		(property "Footprint" "Resistor_SMD:R_0603_1608Metric"
 			(at 101.6 195.58 0)
 			(effects
@@
 			)
 		)
-		(property "Footprint" ""
+		(property "Footprint" "Fuse:Fuse_1812_4532Metric"
 			(at 76.2 127 0)
 			(effects
@@
 			)
 		)
-		(property "Footprint" ""
+		(property "Footprint" "Diode_SMD:D_SMB"
 			(at 91.44 127 0)
 			(effects
@@
 			)
 		)
-		(property "Footprint" ""
+		(property "Footprint" "mini-xt:ESSOP-10_150mil_P1.0mm"
 			(at 139.7 165.1 0)
 			(effects
@@
 			)
 		)
-		(property "Footprint" ""
+		(property "Footprint" "Resistor_SMD:R_0603_1608Metric"
 			(at 152.4 203.2 0)
 			(effects
@@
 			)
 		)
-		(property "Footprint" ""
+		(property "Footprint" "Resistor_SMD:R_0603_1608Metric"
 			(at 177.8 139.7 0)
 			(effects
@@
 			)
 		)
-		(property "Footprint" ""
+		(property "Footprint" "Capacitor_SMD:C_0603_1608Metric"
 			(at 165.1 190.5 0)
 			(effects
@@
 			)
 		)
-		(property "Footprint" ""
+		(property "Footprint" "Capacitor_SMD:C_1206_3216Metric"
 			(at 203.2 177.8 0)
 			(effects
@@
 			)
 		)
-		(property "Footprint" ""
+		(property "Footprint" "Capacitor_SMD:C_0603_1608Metric"
 			(at 215.9 177.8 0)
 			(effects
@@
 			)
 		)
-		(property "Footprint" ""
+		(property "Footprint" "Package_TO_SOT_SMD:TSOT-23-6"
 			(at 228.6 152.4 0)
 			(effects
@@
 			)
 		)
-		(property "Footprint" ""
+		(property "Footprint" "Capacitor_SMD:C_0603_1608Metric"
 			(at 254 165.1 0)
 			(effects
@@
 			)
 		)
-		(property "Footprint" ""
+		(property "Footprint" "Inductor_SMD:L_Taiyo-Yuden_NR-40xx"
 			(at 266.7 142.24 0)
 			(effects
@@
 			)
 		)
-		(property "Footprint" ""
+		(property "Footprint" "Resistor_SMD:R_0603_1608Metric"
 			(at 279.4 177.8 0)
 			(effects
@@
 			)
 		)
-		(property "Footprint" ""
+		(property "Footprint" "Resistor_SMD:R_0603_1608Metric"
 			(at 279.4 198.12 0)
 			(effects
@@
 			)
 		)
-		(property "Footprint" ""
+		(property "Footprint" "Capacitor_SMD:C_1206_3216Metric"
 			(at 292.1 165.1 0)
 			(effects
@@
 			)
 		)
-		(property "Footprint" ""
+		(property "Footprint" "Capacitor_SMD:C_0603_1608Metric"
 			(at 304.8 165.1 0)
 			(effects
@@
 			)
 		)
-		(property "Footprint" ""
+		(property "Footprint" "Capacitor_SMD:C_1206_3216Metric"
 			(at 317.5 165.1 0)
 			(effects
@@
 			)
 		)
-		(property "Footprint" ""
+		(property "Footprint" "Capacitor_SMD:C_0805_2012Metric"
 			(at 215.9 127 0)
 			(effects
@@
 			)
 		)
-		(property "Footprint" ""
+		(property "Footprint" "Capacitor_SMD:C_1206_3216Metric"
 			(at 190.5 177.8 0)
 			(effects
@@
 			)
 		)
-		(property "Footprint" ""
+		(property "Footprint" "Resistor_SMD:R_0603_1608Metric"
 			(at 101.6 215.9 0)
 			(effects
@@
 			)
 		)
-		(property "Footprint" ""
+		(property "Footprint" "LED_SMD:LED_0603_1608Metric"
 			(at 101.6 228.6 0)
 			(effects
@@
 			)
 		)
-		(property "Footprint" ""
+		(property "Footprint" "Resistor_SMD:R_0603_1608Metric"
 			(at 304.8 215.9 0)
 			(effects
@@
 			)
 		)
-		(property "Footprint" ""
+		(property "Footprint" "LED_SMD:LED_0603_1608Metric"
 			(at 304.8 228.6 0)
 			(effects
