File: hardware/sheets/video.kicad_sch (KiCad schematic)
At the start: 35 parts, among them J1 HDMI_A, J2 VGA HD15, M1 Core2350B (8MB PSRAM), U2 74LVC245A, U3 74LVC245A, U4 74LVC245A, U5 74LVC245A

Commit message: Retire SPEED_SEL to a cpu_core-local jumper; docs, firmware notes, 595 prune
- SPEED_SEL leaves the private-net set: speed select is now a local strap on
  cpu_core (JP1 + 10k pulldown, open = 7.16 MHz) instead of an MCU GPIO;
  mxbus/supervisor/bus_mcu/cpu_core updated and sheets regenerated
- Add the addr_decode net-by-net I/O decode chart to docs/xt-mcu-sbc-design.md
- Add docs/bus-mcu-firmware.md and docs/video-firmware.md
- parts.py: prune the dead 74HC595 binding (last card_isatest leftover)

Co-Authored-By: Claude Fable 5 <noreply@anthropic.com>
Claude-Session: https://claude.ai/code/session_01VpbEjRYKoR12pVJpBtbaZF
Parts:
- JP1: LCSC Part Num C2337 -> C492401
Changed lines of the file:
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@@
 		(instances
 			(project "mini-xt"
-				(path "/26736c46-8b40-5460-874f-03596d17270c/3f5f8bf1-0374-5032-82b0-b1b8b2670099"
+				(path "/26736c46-8b40-5460-874f-03596d17270c/62bf3472-8d2a-5fe5-91e5-6c9c6e274c27"
 					(reference "M401")
 					(unit 1)
@@
 		(instances
 			(project "mini-xt"
-				(path "/26736c46-8b40-5460-874f-03596d17270c/3f5f8bf1-0374-5032-82b0-b1b8b2670099"
+				(path "/26736c46-8b40-5460-874f-03596d17270c/62bf3472-8d2a-5fe5-91e5-6c9c6e274c27"
 					(reference "D401")
 					(unit 1)
@@
 		(instances
 			(project "mini-xt"
-				(path "/26736c46-8b40-5460-874f-03596d17270c/3f5f8bf1-0374-5032-82b0-b1b8b2670099"
+				(path "/26736c46-8b40-5460-874f-03596d17270c/62bf3472-8d2a-5fe5-91e5-6c9c6e274c27"
 					(reference "#FLG401")
 					(unit 1)
@@
 		(instances
 			(project "mini-xt"
-				(path "/26736c46-8b40-5460-874f-03596d17270c/3f5f8bf1-0374-5032-82b0-b1b8b2670099"
+				(path "/26736c46-8b40-5460-874f-03596d17270c/62bf3472-8d2a-5fe5-91e5-6c9c6e274c27"
 					(reference "#FLG402")
 					(unit 1)
@@
 		(instances
 			(project "mini-xt"
-				(path "/26736c46-8b40-5460-874f-03596d17270c/3f5f8bf1-0374-5032-82b0-b1b8b2670099"
+				(path "/26736c46-8b40-5460-874f-03596d17270c/62bf3472-8d2a-5fe5-91e5-6c9c6e274c27"
 					(reference "C401")
 					(unit 1)
@@
 		(instances
 			(project "mini-xt"
-				(path "/26736c46-8b40-5460-874f-03596d17270c/3f5f8bf1-0374-5032-82b0-b1b8b2670099"
+				(path "/26736c46-8b40-5460-874f-03596d17270c/62bf3472-8d2a-5fe5-91e5-6c9c6e274c27"
 					(reference "C402")
 					(unit 1)
@@
 		(instances
 			(project "mini-xt"
-				(path "/26736c46-8b40-5460-874f-03596d17270c/3f5f8bf1-0374-5032-82b0-b1b8b2670099"
+				(path "/26736c46-8b40-5460-874f-03596d17270c/62bf3472-8d2a-5fe5-91e5-6c9c6e274c27"
 					(reference "C403")
 					(unit 1)
@@
 		(instances
 			(project "mini-xt"
-				(path "/26736c46-8b40-5460-874f-03596d17270c/3f5f8bf1-0374-5032-82b0-b1b8b2670099"
+				(path "/26736c46-8b40-5460-874f-03596d17270c/62bf3472-8d2a-5fe5-91e5-6c9c6e274c27"
 					(reference "C404")
 					(unit 1)
@@
 		(instances
 			(project "mini-xt"
-				(path "/26736c46-8b40-5460-874f-03596d17270c/3f5f8bf1-0374-5032-82b0-b1b8b2670099"
+				(path "/26736c46-8b40-5460-874f-03596d17270c/62bf3472-8d2a-5fe5-91e5-6c9c6e274c27"
 					(reference "C405")
 					(unit 1)
@@
 		(instances
 			(project "mini-xt"
-				(path "/26736c46-8b40-5460-874f-03596d17270c/3f5f8bf1-0374-5032-82b0-b1b8b2670099"
+				(path "/26736c46-8b40-5460-874f-03596d17270c/62bf3472-8d2a-5fe5-91e5-6c9c6e274c27"
 					(reference "RN401")
 					(unit 1)
@@
 		(instances
 			(project "mini-xt"
-				(path "/26736c46-8b40-5460-874f-03596d17270c/3f5f8bf1-0374-5032-82b0-b1b8b2670099"
+				(path "/26736c46-8b40-5460-874f-03596d17270c/62bf3472-8d2a-5fe5-91e5-6c9c6e274c27"
 					(reference "RN402")
 					(unit 1)
@@
 			)
 		)
-		(property "LCSC Part Num" "C2337"
+		(property "LCSC Part Num" "C492401"
 			(at 137.16 40.64 0)
 			(effects
@@
 		(instances
 			(project "mini-xt"
-				(path "/26736c46-8b40-5460-874f-03596d17270c/3f5f8bf1-0374-5032-82b0-b1b8b2670099"
+				(path "/26736c46-8b40-5460-874f-03596d17270c/62bf3472-8d2a-5fe5-91e5-6c9c6e274c27"
 					(reference "JP401")
 					(unit 1)
@@
 		(instances
 			(project "mini-xt"
-				(path "/26736c46-8b40-5460-874f-03596d17270c/3f5f8bf1-0374-5032-82b0-b1b8b2670099"
+				(path "/26736c46-8b40-5460-874f-03596d17270c/62bf3472-8d2a-5fe5-91e5-6c9c6e274c27"
 					(reference "U402")
 					(unit 1)
@@
 		(instances
 			(project "mini-xt"
-				(path "/26736c46-8b40-5460-874f-03596d17270c/3f5f8bf1-0374-5032-82b0-b1b8b2670099"
+				(path "/26736c46-8b40-5460-874f-03596d17270c/62bf3472-8d2a-5fe5-91e5-6c9c6e274c27"
 					(reference "U403")
 					(unit 1)
@@
 		(instances
 			(project "mini-xt"
-				(path "/26736c46-8b40-5460-874f-03596d17270c/3f5f8bf1-0374-5032-82b0-b1b8b2670099"
+				(path "/26736c46-8b40-5460-874f-03596d17270c/62bf3472-8d2a-5fe5-91e5-6c9c6e274c27"
 					(reference "U404")
 					(unit 1)
@@
 		(instances
 			(project "mini-xt"
-				(path "/26736c46-8b40-5460-874f-03596d17270c/3f5f8bf1-0374-5032-82b0-b1b8b2670099"
+				(path "/26736c46-8b40-5460-874f-03596d17270c/62bf3472-8d2a-5fe5-91e5-6c9c6e274c27"
 					(reference "U405")
 					(unit 1)
@@
 		(instances
 			(project "mini-xt"
-				(path "/26736c46-8b40-5460-874f-03596d17270c/3f5f8bf1-0374-5032-82b0-b1b8b2670099"
+				(path "/26736c46-8b40-5460-874f-03596d17270c/62bf3472-8d2a-5fe5-91e5-6c9c6e274c27"
 					(reference "F401")
 					(unit 1)
@@
 		(instances
 			(project "mini-xt"
-				(path "/26736c46-8b40-5460-874f-03596d17270c/3f5f8bf1-0374-5032-82b0-b1b8b2670099"
+				(path "/26736c46-8b40-5460-874f-03596d17270c/62bf3472-8d2a-5fe5-91e5-6c9c6e274c27"
 					(reference "J401")
 					(unit 1)
@@
 		(instances
 			(project "mini-xt"
-				(path "/26736c46-8b40-5460-874f-03596d17270c/3f5f8bf1-0374-5032-82b0-b1b8b2670099"
+				(path "/26736c46-8b40-5460-874f-03596d17270c/62bf3472-8d2a-5fe5-91e5-6c9c6e274c27"
 					(reference "R410")
 					(unit 1)
@@
 		(instances
 			(project "mini-xt"
-				(path "/26736c46-8b40-5460-874f-03596d17270c/3f5f8bf1-0374-5032-82b0-b1b8b2670099"
+				(path "/26736c46-8b40-5460-874f-03596d17270c/62bf3472-8d2a-5fe5-91e5-6c9c6e274c27"
 					(reference "R411")
 					(unit 1)
@@
 		(instances
 			(project "mini-xt"
-				(path "/26736c46-8b40-5460-874f-03596d17270c/3f5f8bf1-0374-5032-82b0-b1b8b2670099"
+				(path "/26736c46-8b40-5460-874f-03596d17270c/62bf3472-8d2a-5fe5-91e5-6c9c6e274c27"
 					(reference "R412")
 					(unit 1)
@@
 		(instances
 			(project "mini-xt"
-				(path "/26736c46-8b40-5460-874f-03596d17270c/3f5f8bf1-0374-5032-82b0-b1b8b2670099"
+				(path "/26736c46-8b40-5460-874f-03596d17270c/62bf3472-8d2a-5fe5-91e5-6c9c6e274c27"
 					(reference "R413")
 					(unit 1)
@@
 		(instances
 			(project "mini-xt"
-				(path "/26736c46-8b40-5460-874f-03596d17270c/3f5f8bf1-0374-5032-82b0-b1b8b2670099"
+				(path "/26736c46-8b40-5460-874f-03596d17270c/62bf3472-8d2a-5fe5-91e5-6c9c6e274c27"
 					(reference "R414")
 					(unit 1)
@@
 		(instances
 			(project "mini-xt"
-				(path "/26736c46-8b40-5460-874f-03596d17270c/3f5f8bf1-0374-5032-82b0-b1b8b2670099"
+				(path "/26736c46-8b40-5460-874f-03596d17270c/62bf3472-8d2a-5fe5-91e5-6c9c6e274c27"
 					(reference "R415")
 					(unit 1)
@@
 		(instances
 			(project "mini-xt"
-				(path "/26736c46-8b40-5460-874f-03596d17270c/3f5f8bf1-0374-5032-82b0-b1b8b2670099"
+				(path "/26736c46-8b40-5460-874f-03596d17270c/62bf3472-8d2a-5fe5-91e5-6c9c6e274c27"
 					(reference "R416")
 					(unit 1)
@@
 		(instances
 			(project "mini-xt"
-				(path "/26736c46-8b40-5460-874f-03596d17270c/3f5f8bf1-0374-5032-82b0-b1b8b2670099"
+				(path "/26736c46-8b40-5460-874f-03596d17270c/62bf3472-8d2a-5fe5-91e5-6c9c6e274c27"
 					(reference "R417")
 					(unit 1)
@@
 		(instances
 			(project "mini-xt"
-				(path "/26736c46-8b40-5460-874f-03596d17270c/3f5f8bf1-0374-5032-82b0-b1b8b2670099"
+				(path "/26736c46-8b40-5460-874f-03596d17270c/62bf3472-8d2a-5fe5-91e5-6c9c6e274c27"
 					(reference "R420")
 					(unit 1)
@@
 		(instances
 			(project "mini-xt"
-				(path "/26736c46-8b40-5460-874f-03596d17270c/3f5f8bf1-0374-5032-82b0-b1b8b2670099"
+				(path "/26736c46-8b40-5460-874f-03596d17270c/62bf3472-8d2a-5fe5-91e5-6c9c6e274c27"
 					(reference "R421")
 					(unit 1)
@@
 		(instances
 			(project "mini-xt"
-				(path "/26736c46-8b40-5460-874f-03596d17270c/3f5f8bf1-0374-5032-82b0-b1b8b2670099"
+				(path "/26736c46-8b40-5460-874f-03596d17270c/62bf3472-8d2a-5fe5-91e5-6c9c6e274c27"
 					(reference "R422")
 					(unit 1)
@@
 		(instances
 			(project "mini-xt"
-				(path "/26736c46-8b40-5460-874f-03596d17270c/3f5f8bf1-0374-5032-82b0-b1b8b2670099"
+				(path "/26736c46-8b40-5460-874f-03596d17270c/62bf3472-8d2a-5fe5-91e5-6c9c6e274c27"
 					(reference "R423")
 					(unit 1)
@@
 		(instances
 			(project "mini-xt"
-				(path "/26736c46-8b40-5460-874f-03596d17270c/3f5f8bf1-0374-5032-82b0-b1b8b2670099"
+				(path "/26736c46-8b40-5460-874f-03596d17270c/62bf3472-8d2a-5fe5-91e5-6c9c6e274c27"
 					(reference "R424")
 					(unit 1)
@@
 		(instances
 			(project "mini-xt"
-				(path "/26736c46-8b40-5460-874f-03596d17270c/3f5f8bf1-0374-5032-82b0-b1b8b2670099"
+				(path "/26736c46-8b40-5460-874f-03596d17270c/62bf3472-8d2a-5fe5-91e5-6c9c6e274c27"
 					(reference "R425")
 					(unit 1)
@@
 		(instances
 			(project "mini-xt"
-				(path "/26736c46-8b40-5460-874f-03596d17270c/3f5f8bf1-0374-5032-82b0-b1b8b2670099"
+				(path "/26736c46-8b40-5460-874f-03596d17270c/62bf3472-8d2a-5fe5-91e5-6c9c6e274c27"
 					(reference "R426")
 					(unit 1)
@@
 		(instances
 			(project "mini-xt"
-				(path "/26736c46-8b40-5460-874f-03596d17270c/3f5f8bf1-0374-5032-82b0-b1b8b2670099"
+				(path "/26736c46-8b40-5460-874f-03596d17270c/62bf3472-8d2a-5fe5-91e5-6c9c6e274c27"
 					(reference "R427")
 					(unit 1)
@@
 		(instances
 			(project "mini-xt"
-				(path "/26736c46-8b40-5460-874f-03596d17270c/3f5f8bf1-0374-5032-82b0-b1b8b2670099"
+				(path "/26736c46-8b40-5460-874f-03596d17270c/62bf3472-8d2a-5fe5-91e5-6c9c6e274c27"
 					(reference "R428")
 					(unit 1)
@@
 		(instances
 			(project "mini-xt"
-				(path "/26736c46-8b40-5460-874f-03596d17270c/3f5f8bf1-0374-5032-82b0-b1b8b2670099"
+				(path "/26736c46-8b40-5460-874f-03596d17270c/62bf3472-8d2a-5fe5-91e5-6c9c6e274c27"
 					(reference "R429")
 					(unit 1)
@@
 		(instances
 			(project "mini-xt"
-				(path "/26736c46-8b40-5460-874f-03596d17270c/3f5f8bf1-0374-5032-82b0-b1b8b2670099"
+				(path "/26736c46-8b40-5460-874f-03596d17270c/62bf3472-8d2a-5fe5-91e5-6c9c6e274c27"
 					(reference "J402")
 					(unit 1)
